Commit message: New omni wheels.

File: summit_xl_description/robots/summit_xl_omni.urdf.xacro (robot description, xacro)
@@ -30,5 +30,5 @@
   <xacro:ros_control/>
   <!-- Gazebo omni steering plugin -->
-	<xacro:omni_steering/>
+  <xacro:omni_steering/>
 	<!-- WHEELS -->
 	<xacro:omni_wheel name="front_right" parent="base_link" reflect="false" hq="true">

File: summit_xl_description/urdf/wheels/omni_wheel.urdf.xacro (robot description, xacro)
@@ -33,5 +33,5 @@
               <mesh filename="package://summit_xl_description/meshes/wheels/omni_wheel_2.dae" />
             </geometry>
-					</xacro:unless>
+		  s</xacro:unless>
         </xacro:if>
         <xacro:unless value="${hq}">
@@ -79,11 +79,10 @@
     </transmission>
     <gazebo reference="${name}_wheel">
-		<mu1 value="5.0"/>
-		<mu2 value="0.5"/>
+		<mu1 value="1.0"/>
+		<mu2 value="1.0"/>
 		<kp value="10000000.0" />
 		<kd value="1.0" />
 		<fdir1 value="1 0 0"/>
-      <material>Gazebo/Grey</material>
-      <turnGravityOff>false</turnGravityOff>
+        <turnGravityOff>false</turnGravityOff>
     </gazebo>
   </xacro:macro>

Commit message: Removed old rubber wheel STL's.

File: summit_xl_description/robots/summit_xl_omni.urdf.xacro (robot description, xacro)
@@ -16,6 +16,6 @@
 	<xacro:property name="PI" value="3.1415926535897931"/>
 	<!-- Wheel parameters -->
-	<xacro:property name="wheel_offset_x" value="0.229" />    <!-- x,y,z in translation from base_link to the center of the wheel -->
-	<xacro:property name="wheel_offset_y" value="0.234" />
+	<xacro:property name="wheel_offset_x" value="0.22911" />    <!-- x,y,z in translation from base_link to the center of the wheel -->
+	<xacro:property name="wheel_offset_y" value="0.24070" />
 	<xacro:property name="wheel_offset_z" value="0.0" />
 	<!-- Flag to select the high or low quality model -->

File: summit_xl_description/urdf/wheels/omni_wheel.urdf.xacro (robot description, xacro)
@@ -3,6 +3,6 @@
   <xacro:property name="M_PI" value="3.1415926535897931" />
   <!-- Wheels -->
-  <property name="wheel_radius" value="0.117" />
-  <property name="wheel_height" value="0.14" />
+  <property name="wheel_radius" value="0.127" />
+  <property name="wheel_height" value="0.087" />
   <property name="wheel_mass" value="6.5" /> <!-- in kg-->
   <macro name="cylinder_inertia" params="m r h">
