Commit message: changed dev names to have same joint names in real and sim

File: summit_xl_description/robots/summit_xl_hls_omni.urdf (robot description, URDF)
Before this commit: robot summit_xl, 38 links, 37 joints
Links:
- removed link xtion1_cam_depth_frame
- removed link xtion1_cam_depth_optical_frame
- removed link xtion1_cam_link
- removed link xtion1_cam_rgb_frame
- removed link xtion1_cam_rgb_optical_frame
- removed link xtion2_cam_depth_frame
- removed link xtion2_cam_depth_optical_frame
- removed link xtion2_cam_link
- removed link xtion2_cam_rgb_frame
- removed link xtion2_cam_rgb_optical_frame
- added link camera_front_depth_optical_frame, mass 0.001
- added link camera_rear_depth_optical_frame, mass 0.001
- added link ptu1_cam_depth_frame, mass 0.01
- added link ptu1_cam_depth_optical_frame, mass 0.001
- added link ptu1_cam_link, mass 0.01; collision box size=0.0730 .2760 0.0720; visual mesh filename=package://robotnik_sensors/meshes/asus_xtion_pro_live.dae scale=0.001 0.001 0.001
- added link ptu1_cam_rgb_frame, mass 0.001
- added link ptu1_cam_rgb_optical_frame, mass 0.001
- added link ptu2_cam_depth_frame, mass 0.01
- added link ptu2_cam_depth_optical_frame, mass 0.001
- added link ptu2_cam_link, mass 0.01; collision box size=0.0730 .2760 0.0720; visual mesh filename=package://robotnik_sensors/meshes/asus_xtion_pro_live.dae scale=0.001 0.001 0.001
- added link ptu2_cam_rgb_frame, mass 0.001
- added link ptu2_cam_rgb_optical_frame, mass 0.001
Joints:
- removed joint xtion1_cam_depth_joint
- removed joint xtion1_cam_depth_optical_joint
- removed joint xtion1_cam_joint
- removed joint xtion1_cam_rgb_joint
- removed joint xtion1_cam_rgb_optical_joint
- removed joint xtion2_cam_depth_joint
- removed joint xtion2_cam_depth_optical_joint
- removed joint xtion2_cam_joint
- removed joint xtion2_cam_rgb_joint
- removed joint xtion2_cam_rgb_optical_joint
- added joint camera_front_depth_optical_joint: type fixed, parent camera_front_link, child camera_front_depth_optical_frame, origin xyz=0 0 0 rpy=-1.57079632679 0 -1.57079632679
- added joint camera_rear_depth_optical_joint: type fixed, parent camera_rear_link, child camera_rear_depth_optical_frame, origin xyz=0 0 0 rpy=-1.57079632679 0 -1.57079632679
- added joint ptu1_cam_depth_joint: type fixed, parent ptu1_cam_rgb_frame, child ptu1_cam_depth_frame, origin xyz=0 0.027 0 rpy=0 0 0
- added joint ptu1_cam_depth_optical_joint: type fixed, parent ptu1_cam_depth_frame, child ptu1_cam_depth_optical_frame, origin xyz=0 0 0 rpy=-1.57079632679 0 -1.57079632679
- added joint ptu1_cam_joint: type fixed, parent ptu1_cam_rgb_frame, child ptu1_cam_link, origin xyz=0 -0.022 0 rpy=0 0 0
- added joint ptu1_cam_rgb_joint: type fixed, parent ptu1_link_2, child ptu1_cam_rgb_frame, origin xyz=0.015 0.020 0.045 rpy=0 0 0
- added joint ptu1_cam_rgb_optical_joint: type fixed, parent ptu1_cam_rgb_frame, child ptu1_cam_rgb_optical_frame, origin xyz=0 0 0 rpy=-1.57079632679 0 -1.57079632679
- added joint ptu2_cam_depth_joint: type fixed, parent ptu2_cam_rgb_frame, child ptu2_cam_depth_frame, origin xyz=0 0.027 0 rpy=0 0 0
- added joint ptu2_cam_depth_optical_joint: type fixed, parent ptu2_cam_depth_frame, child ptu2_cam_depth_optical_frame, origin xyz=0 0 0 rpy=-1.57079632679 0 -1.57079632679
- added joint ptu2_cam_joint: type fixed, parent ptu2_cam_rgb_frame, child ptu2_cam_link, origin xyz=0 -0.022 0 rpy=0 0 0
- added joint ptu2_cam_rgb_joint: type fixed, parent ptu2_link_2, child ptu2_cam_rgb_frame, origin xyz=0.015 0.020 0.045 rpy=0 0 0
- added joint ptu2_cam_rgb_optical_joint: type fixed, parent ptu2_cam_rgb_frame, child ptu2_cam_rgb_optical_frame, origin xyz=0 0 0 rpy=-1.57079632679 0 -1.57079632679

File: summit_xl_description/robots/summit_xl_hls_omni.urdf.xacro (robot description, xacro)
@@ -85,8 +85,8 @@
 		<origin xyz="0.438 -0.117 1.375" rpy="0 0 0"/>
     </xacro:pan_tilt>
-    <xacro:sensor_asus_xtion_pro name="xtion1" parent="ptu1_link_2">
+    <xacro:sensor_asus_xtion_pro name="ptu1" parent="ptu1_link_2">
 		<origin xyz="0.015 0.020 0.045" rpy="0 0 0"/>
     </xacro:sensor_asus_xtion_pro>
-    <xacro:sensor_asus_xtion_pro name="xtion2" parent="ptu2_link_2">
+    <xacro:sensor_asus_xtion_pro name="ptu2" parent="ptu2_link_2">
 		<origin xyz="0.015 0.020 0.045" rpy="0 0 0"/>
     </xacro:sensor_asus_xtion_pro>
