Commit message: added pan-tilt units to description

File: summit_xl_description/robots/summit_xl_hls_omni.urdf.xacro (robot description, xacro)
@@ -11,4 +11,7 @@
 	<!-- Import strucutres, holders -->
 	<xacro:include filename="$(find summit_xl_description)/urdf/structures/structure_hokuyo.urdf.xacro" />
+	<xacro:include filename="$(find summit_xl_description)/urdf/structures/structure_masts.urdf.xacro" />
+	<!-- Import pan-tilt unit -->
+	<xacro:include filename="$(find summit_xl_description)/urdf/pan_tilt/pan_tilt.urdf.xacro" />
 	<!-- Import all available sensors -->
 	<xacro:include filename="$(find robotnik_sensors)/urdf/all_sensors.urdf.xacro" />
@@ -40,4 +43,7 @@
        <origin xyz="-0.2225 0.105 0.001" rpy="0 0 3.1416"/>
     </xacro:structure>
+    <xacro:structure_masts name="structure_masts" parent="base_link">
+       <origin xyz="0.0 0.0 0.0" rpy="0 0 0"/>
+    </xacro:structure_masts>
 	<!-- WHEELS -->
 	<xacro:omni_wheel name="front_right" parent="base_link" reflect="false" hq="true">
@@ -55,8 +61,8 @@
 	<!-- SENSORS -->
 	<xacro:sensor_hokuyo_ust10lx name="hokuyo_front" parent="base_link">
-		<origin xyz="0.403 -0.256 -0.050" rpy="3.1416 0 -0.7854"/>
+		<origin xyz="0.403 -0.256 -0.045" rpy="3.1416 0 -0.7854"/>
 	</xacro:sensor_hokuyo_ust10lx>
 	<xacro:sensor_hokuyo_ust10lx name="hokuyo_rear" parent="base_link">
-		<origin xyz="-0.403 0.256 -0.050" rpy="3.1416 0 2.3562"/>
+		<origin xyz="-0.403 0.256 -0.045" rpy="3.1416 0 2.3562"/>
 	</xacro:sensor_hokuyo_ust10lx>
 	<xacro:sensor_axis_m5013 name="camera_front" parent="base_link">
@@ -69,4 +75,17 @@
 		<origin xyz="-0.18 0.0 0.170" rpy="0 0 0"/>
 	</xacro:sensor_imu>
+	<!-- PAN TILT UNITS -->
+    <xacro:pan_tilt name="ptu1" parent="base_link" hq="true">
+		<origin xyz="0.438 0.113 0.675" rpy="0 0 0"/>
+    </xacro:pan_tilt>
+    <xacro:pan_tilt name="ptu2" parent="base_link" hq="true">
+		<origin xyz="0.438 -0.117 1.375" rpy="0 0 0"/>
+    </xacro:pan_tilt>
+    <xacro:sensor_asus_xtion_pro name="xtion1" parent="ptu1_link_2">
+		<origin xyz="0.0 0.0 0.033" rpy="0 0 0"/>
+    </xacro:sensor_asus_xtion_pro>
+    <xacro:sensor_asus_xtion_pro name="xtion2" parent="ptu2_link_2">
+		<origin xyz="0.0 0.0 0.033" rpy="0 0 0"/>
+    </xacro:sensor_asus_xtion_pro>
 <!-- xacro:sensor_gps name="gps" parent="base_link">
 		<origin xyz="-0.22 0 0.275" rpy="0 0 0"/>

Commit message: corrected pos of xtions

File: summit_xl_description/robots/summit_xl_hls_omni.urdf.xacro (robot description, xacro)
@@ -61,8 +61,8 @@
 	<!-- SENSORS -->
 	<xacro:sensor_hokuyo_ust10lx name="hokuyo_front" parent="base_link">
-		<origin xyz="0.403 -0.256 -0.045" rpy="3.1416 0 -0.7854"/>
+		<origin xyz="0.403 -0.256 0.045" rpy="3.1416 0 -0.7854"/>
 	</xacro:sensor_hokuyo_ust10lx>
 	<xacro:sensor_hokuyo_ust10lx name="hokuyo_rear" parent="base_link">
-		<origin xyz="-0.403 0.256 -0.045" rpy="3.1416 0 2.3562"/>
+		<origin xyz="-0.403 0.256 0.025" rpy="3.1416 0 2.3562"/>
 	</xacro:sensor_hokuyo_ust10lx>
 	<xacro:sensor_axis_m5013 name="camera_front" parent="base_link">
@@ -83,8 +83,8 @@
     </xacro:pan_tilt>
     <xacro:sensor_asus_xtion_pro name="xtion1" parent="ptu1_link_2">
-		<origin xyz="0.0 0.0 0.033" rpy="0 0 0"/>
+		<origin xyz="0.015 0.020 0.045" rpy="0 0 0"/>
     </xacro:sensor_asus_xtion_pro>
     <xacro:sensor_asus_xtion_pro name="xtion2" parent="ptu2_link_2">
-		<origin xyz="0.0 0.0 0.033" rpy="0 0 0"/>
+		<origin xyz="0.015 0.020 0.045" rpy="0 0 0"/>
     </xacro:sensor_asus_xtion_pro>
 <!-- xacro:sensor_gps name="gps" parent="base_link">

Commit message: minor pos changes in urdf xacro

File: summit_xl_description/robots/summit_xl_hls_omni.urdf.xacro (robot description, xacro)
@@ -60,9 +60,12 @@
 	</xacro:omni_wheel>
 	<!-- SENSORS -->
+	<!-- xacro:sensor_hokuyo_ust10lx name="hokuyo_front" parent="base_link">
+		<origin xyz="0.403 -0.256 0.045" rpy="3.1416 0 -0.7854"/>
+	</xacro:sensor_hokuyo_ust10lx -->
+	<xacro:sensor_hokuyo_ust10lx name="hokuyo_rear" parent="base_link">
+		<origin xyz="-0.403 0.256 -0.045" rpy="3.1416 0 2.3562"/>
+	</xacro:sensor_hokuyo_ust10lx>
 	<xacro:sensor_hokuyo_ust10lx name="hokuyo_front" parent="base_link">
-		<origin xyz="0.403 -0.256 0.045" rpy="3.1416 0 -0.7854"/>
-	</xacro:sensor_hokuyo_ust10lx>
-	<xacro:sensor_hokuyo_ust10lx name="hokuyo_rear" parent="base_link">
-		<origin xyz="-0.403 0.256 0.025" rpy="3.1416 0 2.3562"/>
+		<origin xyz="0.403 -0.256 -0.045" rpy="3.1416 0 -0.7854"/>
 	</xacro:sensor_hokuyo_ust10lx>
 	<xacro:sensor_axis_m5013 name="camera_front" parent="base_link">

Commit message: description: corrected ptz cameras position

File: summit_xl_description/robots/summit_xl_hls_omni.urdf.xacro (robot description, xacro)
@@ -70,8 +70,15 @@
 	</xacro:sensor_hokuyo_ust10lx>
 	<xacro:sensor_axis_m5013 name="camera_front" parent="base_link">
-		<origin xyz="0.370 -0.234 0.148" rpy="0 0 0"/>
+<!--
+		<origin xyz="0.370 -0.234 0.148" rpy="0 0 -0.2837"/>
+-->
+		<!-- modified axis position to correct ar_marker error -->
+		<origin xyz="0.370 -0.180 0.148" rpy="0 0 -0.2837"/>
 	</xacro:sensor_axis_m5013>
 	<xacro:sensor_axis_m5013 name="camera_rear" parent="base_link">
+<!--
 		<origin xyz="-0.370 0.234 0.148" rpy="0 0 3.1416"/>
+-->
+		<origin xyz="-0.370 0.234 0.148" rpy="0 0 2.8578"/>
 	</xacro:sensor_axis_m5013>
 	<xacro:sensor_imu name="imu" parent="base_link">

Commit message: description: connecting rgbd links with the pantilts

File: summit_xl_description/robots/summit_xl_hls_omni.urdf.xacro (robot description, xacro)
@@ -86,4 +86,5 @@
 	</xacro:sensor_imu>
 	<!-- PAN TILT UNITS -->
+<!-- Original, edited to solve ptu1vsptu2 exchange and parent _link_2 not existing
     <xacro:pan_tilt name="ptu1" parent="base_link" hq="true">
 		<origin xyz="0.438 0.113 0.675" rpy="0 0 0"/>
@@ -97,4 +98,17 @@
     <xacro:sensor_asus_xtion_pro name="ptu2" parent="ptu2_link_2">
 		<origin xyz="0.015 0.020 0.045" rpy="0 0 0"/>
+    </xacro:sensor_asus_xtion_pro>
+-->
+    <xacro:pan_tilt name="ptu2" parent="base_link" hq="true">
+                <origin xyz="0.438 0.113 0.675" rpy="0 0 0"/>
+    </xacro:pan_tilt>
+    <xacro:pan_tilt name="ptu1" parent="base_link" hq="true">
+                <origin xyz="0.438 -0.117 1.375" rpy="0 0 0"/>
+    </xacro:pan_tilt>
+    <xacro:sensor_asus_xtion_pro name="ptu1" parent="ptu1_link_2">
+                <origin xyz="0.015 0.020 0.045" rpy="0 0 0"/>
+    </xacro:sensor_asus_xtion_pro>
+    <xacro:sensor_asus_xtion_pro name="ptu2" parent="ptu2_link_2">
+                <origin xyz="0.015 0.020 0.045" rpy="0 0 0"/>
     </xacro:sensor_asus_xtion_pro>
 <!-- xacro:sensor_gps name="gps" parent="base_link">

Commit message: changed to hector imu

File: summit_xl_description/robots/summit_xl_hls_omni.urdf.xacro (robot description, xacro)
@@ -82,7 +82,11 @@
 		<origin xyz="-0.370 0.234 0.148" rpy="0 0 2.8578"/>
 	</xacro:sensor_axis_m5013>
-	<xacro:sensor_imu name="imu" parent="base_link">
+	<!-- xacro:sensor_imu name="imu" parent="base_link">
 		<origin xyz="-0.18 0.0 0.170" rpy="0 0 0"/>
-	</xacro:sensor_imu>
+	</xacro:sensor_imu -->
+	<!-- Imu with hector plugin -->
+	<xacro:sensor_imu_hector name="imu" parent="base_link">
+		<origin xyz="-0.18 0.0 0.170" rpy="0 0 0"/>
+	</xacro:sensor_imu_hector>
 	<!-- PAN TILT UNITS -->
 <!-- Original, edited to solve ptu1vsptu2 exchange and parent _link_2 not existing

Commit message: updated robot models

File: summit_xl_description/robots/summit_xl_hls_omni.urdf.xacro (robot description, xacro)
@@ -1,4 +1,5 @@
 <?xml version="1.0"?>
 <robot name="summit_xl" xmlns:xacro="http://www.ros.org/wiki/xacro">
+	<!-- Version 1.0 -->
 	<!-- ***************** -->
 	<!-- Imported elements -->
@@ -34,10 +35,4 @@
     <xacro:omni_steering/>
     <!-- HOLDERS, STRUCTURES -->
-    <xacro:structure name="structure_hokuyo_front" parent="base_link">
-       <origin xyz="0.2225 -0.105 0.001" rpy="0 0 0"/>
-    </xacro:structure>
-    <xacro:structure name="structure_hokuyo_rear" parent="base_link">
-       <origin xyz="-0.2225 0.105 0.001" rpy="0 0 3.1416"/>
-    </xacro:structure>
 	<!-- WHEELS -->
 	<xacro:omni_wheel name="front_right" parent="base_link" reflect="false" hq="true">
@@ -55,18 +50,21 @@
 	<!-- SENSORS -->
 	<xacro:sensor_hokuyo_ust10lx name="hokuyo_front" parent="base_link">
-		<origin xyz="0.403 -0.256 -0.050" rpy="3.1416 0 -0.7854"/>
+		<origin xyz="0.377 -0.20957 0.2024" rpy="0 0 ${-PI/4.0}"/>
 	</xacro:sensor_hokuyo_ust10lx>
 	<xacro:sensor_hokuyo_ust10lx name="hokuyo_rear" parent="base_link">
-		<origin xyz="-0.403 0.256 -0.050" rpy="3.1416 0 2.3562"/>
+		<origin xyz="-0.377 0.20957 0.2024" rpy="0 0 ${3.0*PI/4.0}"/>
 	</xacro:sensor_hokuyo_ust10lx>
-	<xacro:sensor_axis_m5013 name="camera_front" parent="base_link">
-		<origin xyz="0.370 -0.234 0.148" rpy="0 0 0"/>
+	<!--xacro:sensor_axis_m5013 name="camera_front" parent="base_link">
+		<origin xyz="0.370 0.234 0.148" rpy="0 0 0"/>
 	</xacro:sensor_axis_m5013>
 	<xacro:sensor_axis_m5013 name="camera_rear" parent="base_link">
-		<origin xyz="-0.370 0.234 0.148" rpy="0 0 3.1416"/>
+		<origin xyz="-0.370 -0.234 0.148" rpy="0 0 3.1416"/>
 	</xacro:sensor_axis_m5013>
 	<xacro:sensor_imu name="imu" parent="base_link">
 		<origin xyz="-0.18 0.0 0.170" rpy="0 0 0"/>
-	</xacro:sensor_imu>
+	</xacro:sensor_imu-->
+	<xacro:sensor_orbbec_astra name="orbbec_astra" parent="base_link">
+		<origin xyz="0.324 0.012 0.230" rpy="0 0 0"/>
+	</xacro:sensor_orbbec_astra>
 <!-- xacro:sensor_gps name="gps" parent="base_link">
 		<origin xyz="-0.22 0 0.275" rpy="0 0 0"/>

File: summit_xl_description/urdf/bases/summit_xl_base.gazebo.xacro (robot description, xacro)
@@ -6,5 +6,4 @@
       <plugin name="ros_control" filename="libgazebo_ros_control.so">
         <!--<robotNamespace>/summit_xl</robotNamespace>-->
-        <robotNamespace>/summit_xl</robotNamespace>
         <robotParam>robot_description</robotParam>
         <controlPeriod>0.001</controlPeriod>

File: summit_xl_description/urdf/bases/summit_xl_hls_base.urdf.xacro (robot description, xacro)
@@ -52,4 +52,12 @@
     </collision>
   </link>
+   <!-- DOCKING CONTACT -->
+    <link name="base_docking_contact">
+    </link>
+    <joint name="base_docking_joint" type="fixed">
+      <origin xyz="0.30 0 0.09" rpy="0 0 0" />
+      <parent link="base_link"/>
+      <child link="base_docking_contact" />
+    </joint>
   </xacro:macro>
 </robot>

Commit message: description: HLS omni modifications

File: summit_xl_description/robots/summit_xl_hls_omni.urdf.xacro (robot description, xacro)
@@ -2,4 +2,35 @@
 <robot name="summit_xl" xmlns:xacro="http://www.ros.org/wiki/xacro">
 	<!-- Version 1.0 -->
+	<!-- ***************** -->
+	<!-- Global parameters -->
+	<!-- ***************** -->
+	<xacro:property name="PI" value="3.1415926535897931"/>
+	<!-- Wheel parameters -->
+	<xacro:property name="wheel_offset_x" value="0.2225" />    <!-- x,y,z in translation from base_link to the center of the wheel -->
+	<xacro:property name="wheel_offset_y" value="0.2045" />
+	<xacro:property name="wheel_offset_z" value="0.0" />
+	<xacro:property name="front_laser_offset_x" value="0.377"/>
+	<xacro:property name="front_laser_offset_y" value="-0.20957"/>
+	<xacro:property name="front_laser_offset_z" value="0.2024"/>
+	<xacro:property name="rear_laser_offset_x" value="-0.377"/>
+	<xacro:property name="rear_laser_offset_y" value="0.20957"/>
+	<xacro:property name="rear_laser_offset_z" value="0.2024"/>
+	<xacro:property name="front_camera_offset_x" value="0.308"/>
+	<xacro:property name="front_camera_offset_y" value="0.141"/>
+	<xacro:property name="front_camera_offset_z" value="0.195"/>
+	<xacro:property name="rear_camera_offset_x" value="-0.308"/>
+	<xacro:property name="rear_camera_offset_y" value="-0.141"/>
+	<xacro:property name="rear_camera_offset_z" value="0.195"/>
+	<xacro:property name="imu_offset_x" value="0.25"/>
+	<xacro:property name="imu_offset_y" value="-0.15"/>
+	<xacro:property name="imu_offset_z" value="0.18"/>
+	<xacro:property name="front_rgbd_camera_offset_x" value="0.324"/>
+	<xacro:property name="front_rgbd_camera_offset_y" value="0.012"/>
+	<xacro:property name="front_rgbd_camera_offset_z" value="0.230"/>
+	<xacro:property name="gps_offset_x" value="-0.365"/>
+	<xacro:property name="gps_offset_y" value="-0.167"/>
+	<xacro:property name="gps_offset_z" value="0.302"/>
+	<!-- Flag to select the high or low quality model -->
+	<xacro:property name="hq" value="true" />
 	<!-- ***************** -->
 	<!-- Imported elements -->
@@ -14,14 +45,4 @@
 	<!-- Import all available sensors -->
 	<xacro:include filename="$(find robotnik_sensors)/urdf/all_sensors.urdf.xacro" />
-	<!-- ***************** -->
-	<!-- Global parameters -->
-	<!-- ***************** -->
-	<xacro:property name="PI" value="3.1415926535897931"/>
-	<!-- Wheel parameters -->
-	<xacro:property name="wheel_offset_x" value="0.2225" />    <!-- x,y,z in translation from base_link to the center of the wheel -->
-	<xacro:property name="wheel_offset_y" value="0.2045" />
-	<xacro:property name="wheel_offset_z" value="0.0" />
-	<!-- Flag to select the high or low quality model -->
-	<xacro:property name="hq" value="true" />
 	<!-- *************** -->
 	<!-- Robots Elements -->
@@ -29,10 +50,9 @@
 	<!-- Here we create the robot elements using the xacro:macros imported at the beggining of this file -->
 	<!-- Summit XL base -->
-    <xacro:summit_xl_hls_base name="summit_xl" publish_bf="true" hq="${hq}"/>
-    <!-- Gazebo ros control pluggins -->
-    <xacro:ros_control/>
-    <!-- Gazebo omni steering plugin -->
-    <xacro:omni_steering/>
-    <!-- HOLDERS, STRUCTURES -->
+	<xacro:summit_xl_hls_base name="summit_xl" publish_bf="true" hq="${hq}"/>
+	<!-- Gazebo ros control pluggins -->
+	<xacro:ros_control/>
+	<!-- Gazebo omni steering plugin -->
+	<xacro:omni_steering/>
 	<!-- WHEELS -->
 	<xacro:omni_wheel name="front_right" parent="base_link" reflect="false" hq="true">
@@ -49,34 +69,24 @@
 	</xacro:omni_wheel>
 	<!-- SENSORS -->
-	<xacro:sensor_hokuyo_ust10lx name="hokuyo_front" parent="base_link">
-		<origin xyz="0.377 -0.20957 0.2024" rpy="0 0 ${-PI/4.0}"/>
+	<xacro:sensor_hokuyo_ust10lx name="laser_front" parent="base_link">
+		<origin xyz="${front_laser_offset_x} ${front_laser_offset_y} ${front_laser_offset_z}" rpy="0 0 ${-PI/4.0}"/>
 	</xacro:sensor_hokuyo_ust10lx>
-	<xacro:sensor_hokuyo_ust10lx name="hokuyo_rear" parent="base_link">
-		<origin xyz="-0.377 0.20957 0.2024" rpy="0 0 ${3.0*PI/4.0}"/>
+	<xacro:sensor_hokuyo_ust10lx name="laser_rear" parent="base_link">
+		<origin xyz="${rear_laser_offset_x} ${rear_laser_offset_y} ${rear_laser_offset_z}" rpy="0 0 ${3.0*PI/4.0}"/>
 	</xacro:sensor_hokuyo_ust10lx>
-	<!--xacro:sensor_axis_m5013 name="camera_front" parent="base_link">
-		<origin xyz="0.370 0.234 0.148" rpy="0 0 0"/>
+	<xacro:sensor_axis_m5013 name="camera_front" parent="base_link">
+		<origin xyz="${front_camera_offset_x} ${front_camera_offset_y} ${front_camera_offset_z}" rpy="${-PI/2} 0 0"/>
 	</xacro:sensor_axis_m5013>
 	<xacro:sensor_axis_m5013 name="camera_rear" parent="base_link">
-		<origin xyz="-0.370 -0.234 0.148" rpy="0 0 3.1416"/>
+		<origin xyz="${rear_camera_offset_x} ${rear_camera_offset_y} ${rear_camera_offset_z}" rpy="${-PI/2} 0 ${PI}"/>
 	</xacro:sensor_axis_m5013>
 	<xacro:sensor_imu name="imu" parent="base_link">
-		<origin xyz="-0.18 0.0 0.170" rpy="0 0 0"/>
-	</xacro:sensor_imu-->
-	<xacro:sensor_orbbec_astra name="orbbec_astra" parent="base_link">
-		<origin xyz="0.324 0.012 0.230" rpy="0 0 0"/>
+		<origin xyz="${imu_offset_x} ${imu_offset_y} ${imu_offset_z}" rpy="0 0 0"/>
+	</xacro:sensor_imu>
+	<xacro:sensor_orbbec_astra name="rgbd_front" parent="base_link">
+		<origin xyz="${front_rgbd_camera_offset_x} ${front_rgbd_camera_offset_y} ${front_rgbd_camera_offset_z}" rpy="0 0 0"/>
 	</xacro:sensor_orbbec_astra>
-<!-- xacro:sensor_gps name="gps" parent="base_link">
-		<origin xyz="-0.22 0 0.275" rpy="0 0 0"/>
-	</xacro:sensor_gps -->
-<!--
-	<xacro:sensor_kinect name="kinect" parent="base_link">
-		<origin xyz="0.325 0.0 0.16" rpy="0 0 0"/>
-	</xacro:sensor_kinect>
--->
-<!--
-	<xacro:sensor_fotonic name="fotonic" parent="base_link">
-		<origin xyz="0.3 0.0 0.24" rpy="0 0 0"/>
-	</xacro:sensor_fotonic>
--->
+	<xacro:sensor_gps name="gps" parent="base_link">
+		<origin xyz="${gps_offset_x} ${gps_offset_y} ${gps_offset_z}" rpy="0 0 0"/>
+	</xacro:sensor_gps>
 </robot>

Commit message: Updated Summit XL Steel urdfs and meshes to current robot mechanical standard configuration

File: summit_xl_description/robots/summit_xl_hls_omni.urdf.xacro (robot description, xacro)
@@ -42,5 +42,5 @@
 	<xacro:include filename="$(find summit_xl_description)/urdf/wheels/omni_wheel.urdf.xacro" />
 	<!-- Import strucutres, holders -->
-	<xacro:include filename="$(find summit_xl_description)/urdf/structures/structure_hokuyo.urdf.xacro" />
+	<xacro:include filename="$(find summit_xl_description)/urdf/structures/structure_hokuyo_ust.urdf.xacro" />
 	<!-- Import all available sensors -->
 	<xacro:include filename="$(find robotnik_sensors)/urdf/all_sensors.urdf.xacro" />
@@ -68,4 +68,11 @@
 		<origin xyz="-${wheel_offset_x} -${wheel_offset_y} ${wheel_offset_z}" rpy="0 0 0"/>
 	</xacro:omni_wheel>
+	<!-- Structures -->
+	<xacro:structure_ust name="structure_front" parent="base_link">
+		<origin xyz="0.303 -0.160 0.155" rpy="0 0 0" />
+	</xacro:structure_ust>
+	<xacro:structure_ust name="structure_rear" parent="base_link">
+		<origin xyz="-0.303 0.160 0.155" rpy="0 0 ${PI}" />
+	</xacro:structure_ust>
 	<!-- SENSORS -->
 	<xacro:sensor_hokuyo_ust10lx name="laser_front" parent="base_link">

File: summit_xl_description/urdf/bases/summit_xl_hls_base.urdf.xacro (robot description, xacro)
@@ -33,10 +33,10 @@
        <xacro:if value="${hq}">
        <geometry>
-	     <mesh filename="package://summit_xl_description/meshes/bases/hls/summit_xl_hls.stl"/>
+	     <mesh filename="package://summit_xl_description/meshes/bases/hls/v2017/lateral_plates.stl"/>
        </geometry>
        </xacro:if>
        <xacro:unless value="${hq}">
        <geometry>
-	     <mesh filename="package://summit_xl_description/meshes/bases/hls/summit_xl_hls.dae"/>
+	     <mesh filename="package://summit_xl_description/meshes/bases/hls/v2017/lateral_plates.dae"/>
        </geometry>
        </xacro:unless>
@@ -48,11 +48,114 @@
        <origin xyz="0 0 0" rpy="0 0 0 " />
        <geometry>
-         <mesh filename="package://summit_xl_description/meshes/bases/hls/summit_xl_hls.dae"/>
+         <mesh filename="package://summit_xl_description/meshes/bases/hls/v2017/lateral_plates.dae"/>
        </geometry>
     </collision>
   </link>
-   <!-- DOCKING CONTACT -->
-    <link name="base_docking_contact">
-    </link>
+  <joint name="base_back_plate_joint" type="fixed">
+     <origin xyz="0 0 0" rpy="0 0 0" />
+     <parent link="base_link"/>
+     <child link="back_plate_link" />
+  </joint>
+  <link name="back_plate_link">
+    <inertial>
+      <mass value="5.0" />
+      <origin xyz="0 0 0" />
+      <inertia  ixx="0.139" ixy="0.004"  ixz="0.0"  iyy="0.685"  iyz="0.0"  izz="0.613" />
+    </inertial>
+    <visual>
+       <origin xyz="0 0 0" rpy="0 0 0" />
+       <xacro:if value="${hq}">
+       <geometry>
+	     <mesh filename="package://summit_xl_description/meshes/bases/hls/v2017/back_plate.stl"/>
+       </geometry>
+       </xacro:if>
+       <xacro:unless value="${hq}">
+       <geometry>
+	     <mesh filename="package://summit_xl_description/meshes/bases/hls/v2017/back_plate.dae"/>
+       </geometry>
+       </xacro:unless>
+       <material name="darkgrey">
+         <color rgba="0.1 0.1 0.1 1"/>
+       </material>
+    </visual>
+    <collision>
+       <origin xyz="0 0 0" rpy="0 0 0 " />
+       <geometry>
+         <mesh filename="package://summit_xl_description/meshes/bases/hls/v2017/back_plate.dae"/>
+       </geometry>
+    </collision>
+  </link>
+  <joint name="base_chassis_box_joint" type="fixed">
+     <origin xyz="0 0 0.043" rpy="0 0 0" />
+     <parent link="base_link"/>
+     <child link="chassis_box_link" />
+  </joint>
+  <!-- Chassis box -->
+  <link name="chassis_box_link">
+    <inertial>
+      <mass value="5.0" />
+      <origin xyz="0 0 0" />
+      <inertia  ixx="0.139" ixy="0.004"  ixz="0.0"  iyy="0.685"  iyz="0.0"  izz="0.613" />
+    </inertial>
+    <visual>
+       <origin xyz="0 0 0" rpy="0 0 0" />
+       <xacro:if value="${hq}">
+       <geometry>
+	     <mesh filename="package://summit_xl_description/meshes/bases/hls/v2017/chassis_box.stl"/>
+       </geometry>
+       </xacro:if>
+       <xacro:unless value="${hq}">
+       <geometry>
+	     <mesh filename="package://summit_xl_description/meshes/bases/hls/v2017/chassis_box.dae"/>
+       </geometry>
+       </xacro:unless>
+       <material name="darkgrey">
+         <color rgba="0.1 0.1 0.1 1"/>
+       </material>
+    </visual>
+    <collision>
+       <origin xyz="0 0 0" rpy="0 0 0 " />
+       <geometry>
+         <mesh filename="package://summit_xl_description/meshes/bases/hls/v2017/chassis_box.dae"/>
+       </geometry>
+    </collision>
+  </link>
+  <joint name="base_top_plate_joint" type="fixed">
+     <origin xyz="0 0 0.288" rpy="0 0 0" />
+     <parent link="base_link"/>
+     <child link="top_plate_link" />
+  </joint>
+  <link name="top_plate_link">
+    <inertial>
+      <mass value="5.0" />
+      <origin xyz="0 0 0" />
+      <inertia  ixx="0.139" ixy="0.004"  ixz="0.0"  iyy="0.685"  iyz="0.0"  izz="0.613" />
+    </inertial>
+    <visual>
+       <origin xyz="0 0 0" rpy="0 0 0" />
+       <xacro:if value="${hq}">
+       <geometry>
+	     <mesh filename="package://summit_xl_description/meshes/bases/hls/v2017/top_plate.stl"/>
+       </geometry>
+       </xacro:if>
+       <xacro:unless value="${hq}">
+       <geometry>
+	     <mesh filename="package://summit_xl_description/meshes/bases/hls/v2017/top_plate.dae"/>
+       </geometry>
+       </xacro:unless>
+       <material name="darkgrey">
+         <color rgba="0.1 0.1 0.1 1"/>
+       </material>
+    </visual>
+    <collision>
+       <origin xyz="0 0 0" rpy="0 0 0 " />
+       <geometry>
+         <mesh filename="package://summit_xl_description/meshes/bases/hls/v2017/top_plate.dae"/>
+       </geometry>
+    </collision>
+  </link>
+  <!-- DOCKING CONTACT -->
+  <link name="base_docking_contact">
+  </link>
     <joint name="base_docking_joint" type="fixed">
       <origin xyz="0.30 0 0.09" rpy="0 0 0" />
