Commit message: updated to new standard

File: summit_xl_description/robots/summit_xl_hls_omni.urdf.xacro (robot description, xacro)
@@ -30,5 +30,5 @@
     <xacro:summit_xl_hls_base name="summit_xl" publish_bf="true" hq="${hq}"/>
     <!-- Gazebo ros control pluggins -->
-    <xacro:ros_control/>
+	<xacro:ros_control prefix=""/>
     <!-- Gazebo omni steering plugin -->
     <xacro:omni_steering/>
@@ -54,8 +54,8 @@
 	</xacro:omni_wheel>
 	<!-- SENSORS -->
-	<xacro:sensor_hokuyo_ust10lx name="hokuyo_front" parent="base_link">
+	<xacro:sensor_hokuyo_ust10lx name="laser_front" parent="base_link">
 		<origin xyz="0.403 -0.256 -0.050" rpy="3.1416 0 -0.7854"/>
 	</xacro:sensor_hokuyo_ust10lx>
-	<xacro:sensor_hokuyo_ust10lx name="hokuyo_rear" parent="base_link">
+	<xacro:sensor_hokuyo_ust10lx name="laser_rear" parent="base_link">
 		<origin xyz="-0.403 0.256 -0.050" rpy="3.1416 0 2.3562"/>
 	</xacro:sensor_hokuyo_ust10lx>

File: summit_xl_description/urdf/wheels/omni_wheel.urdf.xacro (robot description, xacro)
@@ -12,5 +12,5 @@
   </xacro:macro>
   <xacro:macro name="omni_wheel" params="name parent *origin reflect hq">
-    <joint name="joint_${name}_wheel" type="continuous">
+    <joint name="${name}_wheel_joint" type="continuous">
       <parent link="${parent}"/>
       <child link="${name}_wheel"/>
