Commit message: summit_xl_description: adding new params to hokuyo sensors in robots

File: summit_xl_description/robots/summit_xl.urdf.xacro (robot description, xacro)
@@ -45,11 +45,16 @@
 	</xacro:rubber_wheel>
 	<!-- SENSORS -->
-	<xacro:sensor_hokuyo_utm30lx name="hokuyo_base" parent="base_link">
+	<xacro:sensor_hokuyo_utm30lx name="hokuyo_base" parent="base_link" min_angle="2.35" max_angle="-2.35">
 		<origin xyz="0.0 0.0 0.33" rpy="0 0 0"/>
 	</xacro:sensor_hokuyo_utm30lx>
 <!--
-	<xacro:sensor_hokuyo_urg04lx name="hokuyo1" parent="base_link">
+	<xacro:sensor_hokuyo_urg04lx name="hokuyo1" parent="base_link" min_angle="2.0943" max_angle="-2.0943">
 		<origin xyz="-0.1 0.0 0.33" rpy="0 0 0"/>
 	</xacro:sensor_hokuyo_urg04lx>
+-->
+<!--
+  <xacro:sensor_hokuyo_ust10lx name="hokuyo_base" parent="base_link" min_angle="2.35" max_angle="-2.35">
+		<origin xyz="0.0 0.0 0.33" rpy="0 0 0"/>
+	</xacro:sensor_hokuyo_ust10lx>
 -->
 	<xacro:sensor_axis name="camera" parent="base_link">

File: summit_xl_description/robots/summit_xl_hl.urdf.xacro (robot description, xacro)
@@ -45,11 +45,16 @@
 	</xacro:rubber_wheel>
 	<!-- SENSORS -->
-	<xacro:sensor_hokuyo_utm30lx name="hokuyo" parent="base_link">
+	<xacro:sensor_hokuyo_utm30lx name="hokuyo_base" parent="base_link" min_angle="2.35" max_angle="-2.35">
 		<origin xyz="0.0 0.0 0.33" rpy="0 0 0"/>
 	</xacro:sensor_hokuyo_utm30lx>
 <!--
-	<xacro:sensor_hokuyo_urg04lx name="hokuyo1" parent="base_link">
+	<xacro:sensor_hokuyo_urg04lx name="hokuyo1" parent="base_link" min_angle="2.0943" max_angle="-2.0943">
 		<origin xyz="-0.1 0.0 0.33" rpy="0 0 0"/>
 	</xacro:sensor_hokuyo_urg04lx>
+-->
+<!--
+  <xacro:sensor_hokuyo_ust10lx name="hokuyo_base" parent="base_link" min_angle="2.35" max_angle="-2.35">
+		<origin xyz="0.0 0.0 0.33" rpy="0 0 0"/>
+	</xacro:sensor_hokuyo_ust10lx>
 -->
 	<xacro:sensor_axis name="camera" parent="base_link">

File: summit_xl_description/robots/summit_xl_hl_omni.urdf.xacro (robot description, xacro)
@@ -45,11 +45,16 @@
 	</xacro:omni_wheel>
 	<!-- SENSORS -->
-	<xacro:sensor_hokuyo_utm30lx name="hokuyo" parent="base_link">
+	<xacro:sensor_hokuyo_utm30lx name="hokuyo_base" parent="base_link" min_angle="2.35" max_angle="-2.35">
 		<origin xyz="0.0 0.0 0.33" rpy="0 0 0"/>
 	</xacro:sensor_hokuyo_utm30lx>
 <!--
-	<xacro:sensor_hokuyo_urg04lx name="hokuyo1" parent="base_link">
+	<xacro:sensor_hokuyo_urg04lx name="hokuyo1" parent="base_link" min_angle="2.0943" max_angle="-2.0943">
 		<origin xyz="-0.1 0.0 0.33" rpy="0 0 0"/>
 	</xacro:sensor_hokuyo_urg04lx>
+-->
+<!--
+  <xacro:sensor_hokuyo_ust10lx name="hokuyo_base" parent="base_link" min_angle="2.35" max_angle="-2.35">
+		<origin xyz="0.0 0.0 0.33" rpy="0 0 0"/>
+	</xacro:sensor_hokuyo_ust10lx>
 -->
 	<xacro:sensor_axis name="camera" parent="base_link">

File: summit_xl_description/robots/summit_xl_omni.urdf.xacro (robot description, xacro)
@@ -45,11 +45,16 @@
 	</xacro:omni_wheel>
 	<!-- SENSORS -->
-	<xacro:sensor_hokuyo_utm30lx name="hokuyo" parent="base_link">
+	<xacro:sensor_hokuyo_utm30lx name="hokuyo_base" parent="base_link" min_angle="2.35" max_angle="-2.35">
 		<origin xyz="0.0 0.0 0.33" rpy="0 0 0"/>
 	</xacro:sensor_hokuyo_utm30lx>
 <!--
-	<xacro:sensor_hokuyo_urg04lx name="hokuyo1" parent="base_link">
+	<xacro:sensor_hokuyo_urg04lx name="hokuyo1" parent="base_link" min_angle="2.0943" max_angle="-2.0943">
 		<origin xyz="-0.1 0.0 0.33" rpy="0 0 0"/>
 	</xacro:sensor_hokuyo_urg04lx>
+-->
+<!--
+  <xacro:sensor_hokuyo_ust10lx name="hokuyo_base" parent="base_link" min_angle="2.35" max_angle="-2.35">
+		<origin xyz="0.0 0.0 0.33" rpy="0 0 0"/>
+	</xacro:sensor_hokuyo_ust10lx>
 -->
 	<xacro:sensor_axis name="camera" parent="base_link">

Commit message: added summit_xl_description from robotnik_robots

File: summit_xl_description/robots/summit_xl.urdf.xacro (robot description, xacro)
@@ -10,5 +10,5 @@
 	<xacro:include filename="$(find summit_xl_description)/urdf/wheels/rubber_wheel.urdf.xacro" />
 	<!-- Import all available sensors -->
-	<xacro:include filename="$(find robotnik_sensors)/urdf/all_sensors.urdf.xacro" />
+	<xacro:include filename="$(find summit_xl_description)/urdf/sensors/all_sensors.urdf.xacro" />
 	<!-- ***************** -->
 	<!-- Global parameters -->
@@ -45,7 +45,5 @@
 	</xacro:rubber_wheel>
 	<!-- SENSORS -->
-  <!-- Hokuyo laser sensors can be parametized with min_angle and max_angle e.g: -->
-  <!--xacro:sensor_hokuyo_utm30lx name="hokuyo_base" parent="base_link" min_angle="2.35" max_angle="-2.35"-->
-	<xacro:sensor_hokuyo_utm30lx name="hokuyo_base" parent="base_link">
+	<xacro:sensor_hokuyo_utm30lx name="hokuyo" parent="base_link">
 		<origin xyz="0.0 0.0 0.33" rpy="0 0 0"/>
 	</xacro:sensor_hokuyo_utm30lx>
@@ -54,9 +52,4 @@
 		<origin xyz="-0.1 0.0 0.33" rpy="0 0 0"/>
 	</xacro:sensor_hokuyo_urg04lx>
--->
-<!--
-  <xacro:sensor_hokuyo_ust10lx name="hokuyo_base" parent="base_link">
-		<origin xyz="0.0 0.0 0.33" rpy="0 0 0"/>
-	</xacro:sensor_hokuyo_ust10lx>
 -->
 	<xacro:sensor_axis name="camera" parent="base_link">
@@ -76,5 +69,5 @@
 <!--
 	<xacro:sensor_kinect name="kinect" parent="base_link">
-		<origin xyz="0.325 0.0 0.16" rpy="0 0 0"/>
+		<origin xyz="0.3 0.0 0.16" rpy="0 0 0"/>
 	</xacro:sensor_kinect>
 -->

File: summit_xl_description/robots/summit_xl_omni.urdf.xacro (robot description, xacro)
@@ -10,5 +10,5 @@
 	<xacro:include filename="$(find summit_xl_description)/urdf/wheels/omni_wheel.urdf.xacro" />
 	<!-- Import all available sensors -->
-	<xacro:include filename="$(find robotnik_sensors)/urdf/all_sensors.urdf.xacro" />
+	<xacro:include filename="$(find summit_xl_description)/urdf/sensors/all_sensors.urdf.xacro" />
 	<!-- ***************** -->
 	<!-- Global parameters -->
@@ -16,6 +16,6 @@
 	<xacro:property name="PI" value="3.1415926535897931"/>
 	<!-- Wheel parameters -->
-	<xacro:property name="wheel_offset_x" value="0.22911" />    <!-- x,y,z in translation from base_link to the center of the wheel -->
-	<xacro:property name="wheel_offset_y" value="0.24070" />
+	<xacro:property name="wheel_offset_x" value="0.229" />    <!-- x,y,z in translation from base_link to the center of the wheel -->
+	<xacro:property name="wheel_offset_y" value="0.234" />
 	<xacro:property name="wheel_offset_z" value="0.0" />
 	<!-- Flag to select the high or low quality model -->
@@ -30,5 +30,5 @@
   <xacro:ros_control/>
   <!-- Gazebo omni steering plugin -->
-  <xacro:omni_steering/>
+	<xacro:omni_steering/>
 	<!-- WHEELS -->
 	<xacro:omni_wheel name="front_right" parent="base_link" reflect="false" hq="true">
@@ -45,7 +45,5 @@
 	</xacro:omni_wheel>
 	<!-- SENSORS -->
-  <!-- Hokuyo laser sensors can be parametized with min_angle and max_angle e.g: -->
-  <!--xacro:sensor_hokuyo_utm30lx name="hokuyo_base" parent="base_link" min_angle="2.35" max_angle="-2.35"-->
-	<xacro:sensor_hokuyo_utm30lx name="hokuyo_base" parent="base_link">
+	<xacro:sensor_hokuyo_utm30lx name="hokuyo" parent="base_link">
 		<origin xyz="0.0 0.0 0.33" rpy="0 0 0"/>
 	</xacro:sensor_hokuyo_utm30lx>
@@ -54,9 +52,4 @@
 		<origin xyz="-0.1 0.0 0.33" rpy="0 0 0"/>
 	</xacro:sensor_hokuyo_urg04lx>
--->
-<!--
-  <xacro:sensor_hokuyo_ust10lx name="hokuyo_base" parent="base_link">
-		<origin xyz="0.0 0.0 0.33" rpy="0 0 0"/>
-	</xacro:sensor_hokuyo_ust10lx>
 -->
 	<xacro:sensor_axis name="camera" parent="base_link">
@@ -71,5 +64,5 @@
 <!--
 	<xacro:sensor_kinect name="kinect" parent="base_link">
-		<origin xyz="0.325 0.0 0.16" rpy="0 0 0"/>
+		<origin xyz="0.3 0.0 0.16" rpy="0 0 0"/>
 	</xacro:sensor_kinect>
 -->

File: summit_xl_description/urdf/bases/summit_xl_base.urdf.xacro (robot description, xacro)
@@ -1,5 +1,5 @@
 <?xml version="1.0"?>
 <robot name="summit_xl" xmlns:xacro="http://www.ros.org/wiki/xacro">
-  <xacro:include filename="$(find summit_xl_description)/urdf/bases/summit_xl_base.gazebo.xacro" />
+	<xacro:include filename="$(find summit_xl_description)/urdf/bases/summit_xl_base.gazebo.xacro" />
   <xacro:macro name="summit_xl_base" params="name publish_bf hq">
   <!-- Robot mechanical and motor parameters -->
@@ -15,4 +15,12 @@
           </geometry>
       </visual>
+<!--
+      <collision>
+          <origin xyz="0 0 0" rpy="0 0 0" />
+          <geometry>
+            <box size="0.001 0.001 0.001" />
+          </geometry>
+      </collision>
+-->
     </link>
     <joint name="base_footprint_joint" type="fixed">
@@ -52,4 +60,46 @@
     </collision>
   </link>
+  <!-- COVERS AND SUSPENSIONS -->
+<!--
+  <xacro:if value="${hq}">
+  <joint name="covers_joint" type="fixed">
+     <origin xyz="0 0 0" rpy="0 0 0" />
+     <parent link="base_link"/>
+     <child link="covers_link" />
+  </joint>
+  <link name="covers_link">
+    <visual>
+       <origin xyz="0 0 0" rpy="0 0 0" />
+       <geometry>
+	     <mesh filename="package://summit_xl_description/meshes/bases/summit_xl_covers.stl"/>
+       </geometry>
+       <material name="silver">
+         <color rgba="0.6 0.6 0.6 1"/>
+       </material>
+    </visual>
+  </link>
+  </xacro:if>
+-->
+  <!-- LOGOS -->
+<!--
+  <joint name="logos_joint" type="fixed">
+     <origin xyz="0 0 0" rpy="0 0 0" />
+     <parent link="base_link"/>
+     <child link="logos_link" />
+  </joint>
+-->
+<!--
+  <link name="logos_link">
+    <visual>
+       <origin xyz="0 0 0" rpy="0 0 0" />
+       <geometry>
+	     <mesh filename="package://summit_xl_description/meshes/bases/summit_xl_logos.stl" scale="1.001 1.001 1.001"/>
+       </geometry>
+       <material name="red">
+         <color rgba="0.8 0.1 0.1 1"/>
+       </material>
+    </visual>
+  </link>
+-->
   </xacro:macro>
 </robot>

File: summit_xl_description/urdf/wheels/omni_wheel.urdf.xacro (robot description, xacro)
@@ -3,6 +3,6 @@
   <xacro:property name="M_PI" value="3.1415926535897931" />
   <!-- Wheels -->
-  <property name="wheel_radius" value="0.127" />
-  <property name="wheel_height" value="0.087" />
+  <property name="wheel_radius" value="0.117" />
+  <property name="wheel_height" value="0.14" />
   <property name="wheel_mass" value="6.5" /> <!-- in kg-->
   <macro name="cylinder_inertia" params="m r h">
@@ -33,5 +33,5 @@
               <mesh filename="package://summit_xl_description/meshes/wheels/omni_wheel_2.dae" />
             </geometry>
-		  s</xacro:unless>
+					</xacro:unless>
         </xacro:if>
         <xacro:unless value="${hq}">
@@ -71,18 +71,18 @@
     <transmission name="${name}_wheel_joint_trans">
       <type>transmission_interface/SimpleTransmission</type>
-      <joint name="joint_${name}_wheel" >
-         <hardwareInterface>EffortJointInterface</hardwareInterface>
-      </joint>
+      <joint name="joint_${name}_wheel" />
       <actuator name="${name}_wheel_joint_motor">
-         <mechanicalReduction>1</mechanicalReduction>
+        <hardwareInterface>EffortJointInterface</hardwareInterface>
+        <mechanicalReduction>1</mechanicalReduction>
       </actuator>
     </transmission>
     <gazebo reference="${name}_wheel">
-		<mu1 value="1.0"/>
-		<mu2 value="1.0"/>
+		<mu1 value="5.0"/>
+		<mu2 value="0.5"/>
 		<kp value="10000000.0" />
 		<kd value="1.0" />
 		<fdir1 value="1 0 0"/>
-        <turnGravityOff>false</turnGravityOff>
+      <material>Gazebo/Grey</material>
+      <turnGravityOff>false</turnGravityOff>
     </gazebo>
   </xacro:macro>

File: summit_xl_description/urdf/wheels/rubber_wheel.urdf.xacro (robot description, xacro)
@@ -58,14 +58,13 @@
     <transmission name="${name}_wheel_joint_trans">
       <type>transmission_interface/SimpleTransmission</type>
-      <joint name="joint_${name}_wheel">
-		<hardwareInterface>EffortJointInterface</hardwareInterface>
-      </joint>
+      <joint name="joint_${name}_wheel" />
       <actuator name="${name}_wheel_joint_motor">
+        <hardwareInterface>EffortJointInterface</hardwareInterface>
         <mechanicalReduction>1</mechanicalReduction>
       </actuator>
-     </transmission>
+    </transmission>
     <gazebo reference="${name}_wheel">
-			<mu1 value="1.0"/>
-			<mu2 value="1.0"/>
+			<mu1 value="5.0"/>
+			<mu2 value="0.5"/>
 			<kp value="10000000.0" />
 			<kd value="1.0" />

Commit message: added plugin option ros_force_based_move from hector_plugins

File: summit_xl_description/robots/summit_xl.urdf.xacro (robot description, xacro)
@@ -30,4 +30,5 @@
 	<xacro:ros_control/>
 	<!-- Gazebo skid steering pluggins -->
+	<!-- xacro:ros_force_based_move broadcastOdomTF="1"/ -->
 	<xacro:skid_steering broadcastOdomTF="1"/>
 	<!-- WHEELS -->

File: summit_xl_description/urdf/bases/summit_xl_base.gazebo.xacro (robot description, xacro)
@@ -45,4 +45,20 @@
 	  </gazebo>
   </xacro:macro>
+  <xacro:macro name="ros_force_based_move" params="broadcastOdomTF">
+	  <gazebo>
+		 <plugin name="ros_force_based_move" filename="libgazebo_ros_force_based_move.so">
+			 <robotNamespace>/summit_xl</robotNamespace>
+			 <commandTopic>/summit_xl_control/cmd_vel</commandTopic>
+			 <odometryTopic>/summit_xl/odom</odometryTopic>
+	         <odometryFrame>odom</odometryFrame>
+			 <yaw_velocity_p_gain>10000.0</yaw_velocity_p_gain>
+			 <x_velocity_p_gain>10000.0</x_velocity_p_gain>
+			 <y_velocity_p_gain>10000.0</y_velocity_p_gain>
+			 <robotBaseFrame>base_footprint</robotBaseFrame>
+			 <odometryRate>20.0</odometryRate>
+			 <publishOdometryTf>${broadcastOdomTF}</publishOdometryTf>
+		 </plugin>
+	  </gazebo>
+  </xacro:macro>
   <gazebo reference="base_footprint">
     <material>Gazebo/Green</material>

Commit message: summit_xl_description: updated urdf parameters for simulation

File: summit_xl_description/robots/summit_xl.urdf.xacro (robot description, xacro)
@@ -30,6 +30,7 @@
 	<xacro:ros_control/>
 	<!-- Gazebo skid steering pluggins -->
-	<!-- xacro:ros_force_based_move broadcastOdomTF="1"/ -->
-	<xacro:skid_steering broadcastOdomTF="0"/>
+    <!-- Simulation now uses a set of ros_control controllers and a node called summit_xl_robot_control -->
+    <!--xacro:ros_force_based_move broadcastOdomTF="0"/-->
+    <!--xacro:skid_steering broadcastOdomTF="0"/>-->
 	<!-- WHEELS -->
 	<xacro:rubber_wheel name="front_right" parent="base_link" reflect="false" hq="${hq}">
@@ -59,8 +60,8 @@
 	</xacro:sensor_hokuyo_ust10lx>
 -->
-	<!--xacro:sensor_axis name="camera" parent="base_link">
-		<origin xyz="0.19 0 0.17" rpy="0 ${15*PI/180} 0"/>
-	</xacro:sensor_axis-->
-	<xacro:sensor_imu_hector name="imu" parent="base_link">
+	<xacro:sensor_axis name="camera" parent="base_link">
+		<origin xyz="0.19 0 0.17" rpy="0 ${-75*PI/180} 0"/>
+	</xacro:sensor_axis>
+	<xacro:sensor_imu_hector name="imu" parent="base_link" >
 		<origin xyz="-0.18 0.0 0.170" rpy="0 0 0"/>
 	</xacro:sensor_imu_hector>
@@ -68,7 +69,7 @@
 		<origin xyz="-0.22 0 0.275" rpy="0 0 0"/>
 	</xacro:sensor_gps>
-	<xacro:sensor_orbbec_astra name="orbbec_astra" parent="base_link">
-		<origin xyz="0.324 0.012 0.172" rpy="0 0 0"/>
-	</xacro:sensor_orbbec_astra>
+	<!--<xacro:sensor_orbbec_astra name="orbbec_astra" parent="base_link">-->
+		<!--<origin xyz="0.324 0.012 0.172" rpy="0 0 0"/> -->
+	<!--</xacro:sensor_orbbec_astra>  -->
 <!--
 	<xacro:sensor_kinect name="kinect" parent="base_link">

File: summit_xl_description/robots/summit_xl_omni.urdf.xacro (robot description, xacro)
@@ -61,5 +61,5 @@
 -->
 	<xacro:sensor_axis name="camera" parent="base_link">
-		<origin xyz="0.19 0 0.17" rpy="0 ${15*PI/180} 0"/>
+		<origin xyz="0.19 0 0.17" rpy="0 ${-75*PI/180} 0"/>
 	</xacro:sensor_axis>
 	<xacro:sensor_imu name="imu" parent="base_link">

File: summit_xl_description/urdf/bases/summit_xl_base.gazebo.xacro (robot description, xacro)
@@ -5,5 +5,5 @@
     <gazebo>
       <plugin name="ros_control" filename="libgazebo_ros_control.so">
-        <robotNamespace>/summit_xl</robotNamespace>
+        <!--<robotNamespace>/summit_xl</robotNamespace>-->
         <robotParam>robot_description</robotParam>
         <controlPeriod>0.001</controlPeriod>
@@ -16,5 +16,5 @@
     <gazebo>
       <plugin name="skid_steer_drive_controller" filename="libgazebo_ros_skid_steer_drive.so">
-			<robotNamespace>/summit_xl</robotNamespace>
+			<!--<robotNamespace>/summit_xl</robotNamespace>-->
 		    <updateRate>100.0</updateRate>
 		    <leftFrontJoint>joint_front_left_wheel</leftFrontJoint>
@@ -38,5 +38,5 @@
 	    <plugin name="omni_steering" filename="libgazebo_ros_planar_move.so">
 	      <commandTopic>/summit_xl_control/cmd_vel</commandTopic>
-	      <odometryTopic>/summit_xl/odom</odometryTopic>
+	      <odometryTopic>/odom</odometryTopic>
 	      <odometryFrame>odom</odometryFrame>
 	      <odometryRate>20.0</odometryRate>
@@ -48,5 +48,5 @@
 	  <gazebo>
 		 <plugin name="ros_force_based_move" filename="libgazebo_ros_force_based_move.so">
-			 <robotNamespace>/summit_xl</robotNamespace>
+			 <!--<robotNamespace>/summit_xl</robotNamespace>-->
 			 <commandTopic>/summit_xl_control/cmd_vel</commandTopic>
 			 <odometryTopic>/summit_xl/odom</odometryTopic>

File: summit_xl_description/urdf/wheels/omni_wheel.urdf.xacro (robot description, xacro)
@@ -8,6 +8,6 @@
   <xacro:macro name="cylinder_inertia" params="m r h">
     <inertia  ixx="${m*(3*r*r+h*h)/12}" ixy = "0" ixz = "0"
-              iyy="${m*(3*r*r+h*h)/12}" iyz = "0"
-              izz="${m*r*r/2}" />
+              iyy="${m*r*r/2}" iyz = "0"
+              izz="${m*(3*r*r+h*h)/12}" />
   </xacro:macro>
   <xacro:macro name="omni_wheel" params="name parent *origin reflect hq">
@@ -33,5 +33,5 @@
               <mesh filename="package://summit_xl_description/meshes/wheels/omni_wheel_2.dae" />
             </geometry>
-		  s</xacro:unless>
+		  </xacro:unless>
         </xacro:if>
         <xacro:unless value="${hq}">
@@ -72,5 +72,5 @@
       <type>transmission_interface/SimpleTransmission</type>
       <joint name="joint_${name}_wheel" >
-         <hardwareInterface>EffortJointInterface</hardwareInterface>
+        <hardwareInterface>VelocityJointInterface</hardwareInterface>
       </joint>
       <actuator name="${name}_wheel_joint_motor">

File: summit_xl_description/urdf/wheels/rubber_wheel.urdf.xacro (robot description, xacro)
@@ -3,11 +3,11 @@
   <xacro:property name="M_PI" value="3.1415926535897931" />
   <!-- Wheels -->
-  <xacro:property name="wheel_radius" value="0.117" />
-  <xacro:property name="wheel_height" value="0.14" />
+  <xacro:property name="wheel_radius" value="0.125" />
+  <xacro:property name="wheel_height" value="0.14" /> <!-- really is the wheel width -->
   <xacro:property name="wheel_mass" value="6.5" /> <!-- in kg-->
   <xacro:macro name="cylinder_inertia" params="m r h">
     <inertia  ixx="${m*(3*r*r+h*h)/12}" ixy = "0" ixz = "0"
-              iyy="${m*(3*r*r+h*h)/12}" iyz = "0"
-              izz="${m*r*r/2}" />
+              iyy="${m*r*r/2}" iyz = "0"
+              izz="${m*(3*r*r+h*h)/12}" />
   </xacro:macro>
   <xacro:macro name="rubber_wheel" params="name parent *origin reflect hq">
@@ -59,5 +59,5 @@
       <type>transmission_interface/SimpleTransmission</type>
       <joint name="joint_${name}_wheel">
-		<hardwareInterface>EffortJointInterface</hardwareInterface>
+        <hardwareInterface>VelocityJointInterface</hardwareInterface>
       </joint>
       <actuator name="${name}_wheel_joint_motor">

Commit message: Modifying models to work with several robots

File: summit_xl_description/robots/summit_xl.urdf.xacro (robot description, xacro)
@@ -26,7 +26,7 @@
 	<!-- Here we create the robot elements using the xacro:macros imported at the beggining of this file -->
 	<!-- Summit XL base -->
-	<xacro:summit_xl_base name="summit_xl" publish_bf="true" hq="${hq}" />
+	<xacro:summit_xl_base prefix="" publish_bf="true" hq="${hq}" />
 	<!-- Gazebo ros control pluggins -->
-	<xacro:ros_control/>
+	<xacro:ros_control prefix=""/>
 	<!-- Gazebo skid steering pluggins -->
     <!-- Simulation now uses a set of ros_control controllers and a node called summit_xl_robot_control -->
@@ -52,7 +52,7 @@
 		<origin xyz="0.0 0.0 0.33" rpy="0 0 0"/>
 	</xacro:sensor_hokuyo_utm30lx-->
-	<xacro:sensor_hokuyo_urg04lx name="hokuyo_base" parent="base_link">
+	<!--xacro:sensor_hokuyo_urg04lx name="hokuyo_base" parent="base_link">
 		<origin xyz="-0.0 0.0 0.33" rpy="0 0 0"/>
-	</xacro:sensor_hokuyo_urg04lx>
+	</xacro:sensor_hokuyo_urg04lx-->
 <!--
   <xacro:sensor_hokuyo_ust10lx name="hokuyo_base" parent="base_link">
@@ -60,13 +60,13 @@
 	</xacro:sensor_hokuyo_ust10lx>
 -->
-	<xacro:sensor_axis name="camera" parent="base_link">
+	<!--xacro:sensor_axis name="camera" parent="base_link">
 		<origin xyz="0.19 0 0.17" rpy="0 ${-75*PI/180} 0"/>
-	</xacro:sensor_axis>
-	<xacro:sensor_imu_hector name="imu" parent="base_link" >
+	</xacro:sensor_axis-->
+	<!--xacro:sensor_imu_hector name="imu" parent="base_link" >
 		<origin xyz="-0.18 0.0 0.170" rpy="0 0 0"/>
-	</xacro:sensor_imu_hector>
-	<xacro:sensor_gps name="gps" parent="base_link">
+	</xacro:sensor_imu_hector-->
+	<!--xacro:sensor_gps name="gps" parent="base_link">
 		<origin xyz="-0.22 0 0.275" rpy="0 0 0"/>
-	</xacro:sensor_gps>
+	</xacro:sensor_gps-->
 	<!--<xacro:sensor_orbbec_astra name="orbbec_astra" parent="base_link">-->
 		<!--<origin xyz="0.324 0.012 0.172" rpy="0 0 0"/> -->

File: summit_xl_description/urdf/bases/summit_xl_base.gazebo.xacro (robot description, xacro)
@@ -2,9 +2,9 @@
 <robot xmlns:xacro="http://www.ros.org/wiki/xacro">
   <!-- ros control plugin -->
-  <xacro:macro name="ros_control">
+  <xacro:macro name="ros_control" params="prefix">
     <gazebo>
       <plugin name="ros_control" filename="libgazebo_ros_control.so">
         <!--<robotNamespace>/summit_xl</robotNamespace>-->
-        <robotNamespace>/summit_xl</robotNamespace>
+        <robotNamespace>${prefix}</robotNamespace>
         <robotParam>robot_description</robotParam>
         <controlPeriod>0.001</controlPeriod>

File: summit_xl_description/urdf/wheels/rubber_wheel.urdf.xacro (robot description, xacro)
@@ -13,5 +13,5 @@
   <xacro:macro name="rubber_wheel" params="name parent *origin reflect hq">
 <!--WHEEL TIRE -->
-    <joint name="joint_${name}_wheel" type="continuous">
+    <joint name="${name}_wheel_joint" type="continuous">
       <parent link="${parent}"/>
       <child link="${name}_wheel"/>
@@ -58,5 +58,5 @@
     <transmission name="${name}_wheel_joint_trans">
       <type>transmission_interface/SimpleTransmission</type>
-      <joint name="joint_${name}_wheel">
+      <joint name="${name}_wheel_joint">
         <hardwareInterface>VelocityJointInterface</hardwareInterface>
       </joint>

Commit message: description: setting name of the xacro without prefix 'multi'

File: summit_xl_description/robots/summit_xl.urdf.xacro (robot description, xacro)
@@ -19,5 +19,5 @@
 	<xacro:property name="hq" value="true" />
 	<xacro:arg name="prefix" default="summit_xl_"/>
-    <xacro:macro name="summit_xl_multi" params="prefix publish_bf hq">
+    <xacro:macro name="summit_xl" params="prefix publish_bf hq">
 		<!-- *************** -->
 		<!-- Robots Elements -->
@@ -50,4 +50,4 @@
    <!-- Gazebo ros control pluggins -->
    <xacro:ros_control/>
-   <xacro:summit_xl_multi prefix="$(arg prefix)" publish_bf="true" hq="true"/>
+   <xacro:summit_xl prefix="$(arg prefix)" publish_bf="true" hq="true"/>
 </robot>
