Commit message: replacing name by prefix in the urdf

File: summit_xl_description/robots/summit_xl.urdf.xacro (robot description, xacro)
@@ -34,51 +34,41 @@
     <!--xacro:skid_steering broadcastOdomTF="0"/>-->
 	<!-- WHEELS -->
-	<xacro:rubber_wheel name="front_right" parent="base_link" reflect="false" hq="${hq}">
+	<xacro:rubber_wheel prefix="front_right" parent="base_link" reflect="false" hq="${hq}">
 		<origin xyz="${wheel_offset_x} -${wheel_offset_y} ${wheel_offset_z}" rpy="0 0 0"/>
 	</xacro:rubber_wheel>
-	<xacro:rubber_wheel name="front_left" parent="base_link" reflect="true" hq="${hq}">
+	<xacro:rubber_wheel prefix="front_left" parent="base_link" reflect="true" hq="${hq}">
 		<origin xyz="${wheel_offset_x} ${wheel_offset_y} ${wheel_offset_z}" rpy="0 0 0"/>
 	</xacro:rubber_wheel>
-	<xacro:rubber_wheel name="back_left" parent="base_link" reflect="true" hq="${hq}">
+	<xacro:rubber_wheel prefix="back_left" parent="base_link" reflect="true" hq="${hq}">
 		<origin xyz="-${wheel_offset_x} ${wheel_offset_y} ${wheel_offset_z}" rpy="0 0 0"/>
 	</xacro:rubber_wheel>
-	<xacro:rubber_wheel name="back_right" parent="base_link" reflect="false" hq="${hq}">
+	<xacro:rubber_wheel prefix="back_right" parent="base_link" reflect="false" hq="${hq}">
 		<origin xyz="-${wheel_offset_x} -${wheel_offset_y} ${wheel_offset_z}" rpy="0 0 0"/>
 	</xacro:rubber_wheel>
 	<!-- SENSORS -->
-  <!-- Hokuyo laser sensors can be parametized with min_angle and max_angle e.g: -->
-  <!--xacro:sensor_hokuyo_utm30lx name="hokuyo_base" parent="base_link" min_angle="2.35" max_angle="-2.35"-->
+	<!-- Hokuyo laser sensors can be parametized with min_angle and max_angle e.g: -->
 	<!--xacro:sensor_hokuyo_utm30lx name="hokuyo_base" parent="base_link">
 		<origin xyz="0.0 0.0 0.33" rpy="0 0 0"/>
 	</xacro:sensor_hokuyo_utm30lx-->
-	<xacro:sensor_hokuyo_urg04lx name="hokuyo_base" parent="base_link">
+	<!--xacro:sensor_hokuyo_urg04lx prefix="hokuyo_base" parent="base_link">
 		<origin xyz="-0.0 0.0 0.33" rpy="0 0 0"/>
-	</xacro:sensor_hokuyo_urg04lx>
-<!--
-  <xacro:sensor_hokuyo_ust10lx name="hokuyo_base" parent="base_link">
+	</xacro:sensor_hokuyo_urg04lx-->
+	<xacro:sensor_hokuyo_ust10lx prefix="hokuyo_base" parent="base_link">
 		<origin xyz="0.0 0.0 0.33" rpy="0 0 0"/>
 	</xacro:sensor_hokuyo_ust10lx>
--->
-	<xacro:sensor_axis name="camera" parent="base_link">
+	<xacro:sensor_axis prefix="camera" parent="base_link">
 		<origin xyz="0.19 0 0.17" rpy="0 ${-75*PI/180} 0"/>
 	</xacro:sensor_axis>
-	<xacro:sensor_imu_hector name="imu" parent="base_link" >
+	<xacro:sensor_imu_hector prefix="imu" parent="base_link" >
 		<origin xyz="-0.18 0.0 0.170" rpy="0 0 0"/>
 	</xacro:sensor_imu_hector>
-	<xacro:sensor_gps name="gps" parent="base_link">
+	<xacro:sensor_gps prefix="gps" parent="base_link">
 		<origin xyz="-0.22 0 0.275" rpy="0 0 0"/>
 	</xacro:sensor_gps>
-	<!--<xacro:sensor_orbbec_astra name="orbbec_astra" parent="base_link">-->
-		<!--<origin xyz="0.324 0.012 0.172" rpy="0 0 0"/> -->
-	<!--</xacro:sensor_orbbec_astra>  -->
-<!--
-	<xacro:sensor_kinect name="kinect" parent="base_link">
-		<origin xyz="0.325 0.0 0.16" rpy="0 0 0"/>
-	</xacro:sensor_kinect>
--->
-<!--
-	<xacro:sensor_fotonic name="fotonic" parent="base_link">
+	<!--xacro:sensor_orbbec_astra prefix="orbbec_astra" parent="base_link">
+		<origin xyz="0.324 0.012 0.172" rpy="0 0 0"/>
+	</xacro:sensor_orbbec_astra-->
+	<!--xacro:sensor_fotonic prefix="fotonic" parent="base_link">
 		<origin xyz="0.3 0.0 0.24" rpy="0 0 0"/>
-	</xacro:sensor_fotonic>
--->
+	</xacro:sensor_fotonic-->
 </robot>

File: summit_xl_description/urdf/wheels/omni_wheel.urdf.xacro (robot description, xacro)
@@ -11,8 +11,8 @@
               izz="${m*(3*r*r+h*h)/12}" />
   </xacro:macro>
-  <xacro:macro name="omni_wheel" params="name parent *origin reflect hq">
-    <joint name="joint_${name}_wheel" type="continuous">
+  <xacro:macro name="omni_wheel" params="prefix parent *origin reflect hq">
+    <joint name="joint_${prefix}_wheel" type="continuous">
       <parent link="${parent}"/>
-      <child link="${name}_wheel"/>
+      <child link="${prefix}_wheel"/>
       <xacro:insert_block name="origin" />
       <axis xyz="0 1 0" rpy="0 0 0" />
@@ -20,5 +20,5 @@
       <joint_properties damping="0.0" friction="0.0"/>
     </joint>
-    <link name="${name}_wheel">
+    <link name="${prefix}_wheel">
       <visual>
         <xacro:if value="${hq}">
@@ -69,14 +69,14 @@
     </link>
     <!-- Transmission is important to link the joints and the controller (see summit_xl_control/config/summit_xl_control.yaml)-->
-    <transmission name="${name}_wheel_joint_trans">
+    <transmission name="${prefix}_wheel_joint_trans">
       <type>transmission_interface/SimpleTransmission</type>
-      <joint name="joint_${name}_wheel" >
+      <joint name="joint_${prefix}_wheel" >
         <hardwareInterface>VelocityJointInterface</hardwareInterface>
       </joint>
-      <actuator name="${name}_wheel_joint_motor">
+      <actuator name="${prefix}_wheel_joint_motor">
          <mechanicalReduction>1</mechanicalReduction>
       </actuator>
     </transmission>
-    <gazebo reference="${name}_wheel">
+    <gazebo reference="${prefix}_wheel">
 		<mu1 value="1.0"/>
 		<mu2 value="1.0"/>

File: summit_xl_description/urdf/wheels/rubber_wheel.urdf.xacro (robot description, xacro)
@@ -11,9 +11,9 @@
               izz="${m*(3*r*r+h*h)/12}" />
   </xacro:macro>
-  <xacro:macro name="rubber_wheel" params="name parent *origin reflect hq">
+  <xacro:macro name="rubber_wheel" params="prefix parent *origin reflect hq">
 <!--WHEEL TIRE -->
-    <joint name="joint_${name}_wheel" type="continuous">
+    <joint name="joint_${prefix}_wheel" type="continuous">
       <parent link="${parent}"/>
-      <child link="${name}_wheel"/>
+      <child link="${prefix}_wheel"/>
       <xacro:insert_block name="origin" />
       <axis xyz="0 1 0" rpy="0 0 0" />
@@ -21,5 +21,5 @@
       <joint_properties damping="0.0" friction="0.0"/>
     </joint>
-    <link name="${name}_wheel">
+    <link name="${prefix}_wheel">
       <visual>
         <!-- HIGH RESOLUTION WHEELS -->
@@ -56,15 +56,15 @@
     </link>
     <!-- Transmission is important to link the joints and the controller (see summit_xl_control/config/summit_xl_control.yaml)-->
-    <transmission name="${name}_wheel_joint_trans">
+    <transmission name="${prefix}_wheel_joint_trans">
       <type>transmission_interface/SimpleTransmission</type>
-      <joint name="joint_${name}_wheel">
+      <joint name="joint_${prefix}_wheel">
         <hardwareInterface>VelocityJointInterface</hardwareInterface>
       </joint>
-      <actuator name="${name}_wheel_joint_motor">
+      <actuator name="${prefix}_wheel_joint_motor">
         <mechanicalReduction>1</mechanicalReduction>
         <motorTorqueConstant>20</motorTorqueConstant>
       </actuator>
      </transmission>
-    <gazebo reference="${name}_wheel">
+    <gazebo reference="${prefix}_wheel">
 			<mu1 value="1.0"/>
 			<mu2 value="1.0"/>

Commit message: description: setting the ptz position correctly

File: summit_xl_description/robots/summit_xl.urdf.xacro (robot description, xacro)
@@ -58,5 +58,5 @@
 	</xacro:sensor_hokuyo_ust10lx>
 	<xacro:sensor_axis prefix="camera" parent="base_link">
-		<origin xyz="0.19 0 0.3" rpy="0 ${15*PI/180} 0"/>
+		<origin xyz="0.19 0 0.26" rpy="0 ${15*PI/180} 0"/>
 	</xacro:sensor_axis>
 	<xacro:sensor_imu_hector prefix="imu" parent="base_link" >

Commit message: description: adjusting z value of ptz camera

File: summit_xl_description/robots/summit_xl.urdf.xacro (robot description, xacro)
@@ -47,5 +47,5 @@
 		<!-- ptz camera -->
 		<!--xacro:sensor_axis prefix="$(arg prefix)front_ptz_camera" parent="$(arg prefix)base_link">
-			<origin xyz="0.19 0 0.3" rpy="0 ${15*PI/180} 0"/>
+			<origin xyz="0.19 0 0.26" rpy="0 ${15*PI/180} 0"/>
 		</xacro:sensor_axis-->
 	    <!-- RGBD -->

File: summit_xl_description/robots/summit_xl_std.urdf.xacro (robot description, xacro)
@@ -48,5 +48,5 @@
 		<!-- ptz camera -->
 		<xacro:sensor_axis prefix="$(arg prefix)front_ptz_camera" parent="$(arg prefix)base_link">
-			<origin xyz="0.19 0 0.3" rpy="0 ${15*PI/180} 0"/>
+			<origin xyz="0.19 0 0.26" rpy="0 ${15*PI/180} 0"/>
 		</xacro:sensor_axis>
 	    <!-- RGBD -->
