Commit message: added cameras of steel in correct pos

File: summit_xl_description/robots/summit_xl_steel_omni.urdf.xacro (robot description, xacro)
@@ -51,10 +51,10 @@
 		<origin xyz="-0.373 0.210 0.205" rpy="0 0 2.3562"/>
 	</xacro:sensor_hokuyo_ust10lx>
-	<!-- xacro:sensor_axis_m5013 name="camera_front" parent="base_link">
-		<origin xyz="0.370 -0.234 0.148" rpy="0 0 0"/>
+	<xacro:sensor_axis_m5013 name="camera_front" parent="base_link">
+		<origin xyz="0.308 0.140 0.195" rpy="0 0 0"/>
 	</xacro:sensor_axis_m5013>
 	<xacro:sensor_axis_m5013 name="camera_rear" parent="base_link">
-		<origin xyz="-0.370 0.234 0.148" rpy="0 0 3.1416"/>
-	</xacro:sensor_axis_m5013 -->
+		<origin xyz="-0.308 -0.140 0.195" rpy="0 0 3.1416"/>
+	</xacro:sensor_axis_m5013>
 	<xacro:sensor_imu name="imu" parent="base_link">
 		<origin xyz="-0.18 0.0 0.170" rpy="0 0 0"/>

Commit message: files added and modified for steel multi control via gazebo planar plugin

File: summit_xl_description/robots/summit_xl_steel_omni.urdf.xacro (robot description, xacro)
@@ -16,5 +16,5 @@
 	<xacro:property name="PI" value="3.1415926535897931"/>
 	<!-- Wheel parameters -->
-	<xacro:property name="wheel_offset_x" value="0.2225" />    <!-- x,y,z in translation from base_link to the center of the wheel -->
+	<xacro:property name="wheel_offset_x" value="0.223" />    <!-- x,y,z in translation from base_link to the center of the wheel -->
 	<xacro:property name="wheel_offset_y" value="0.205" />
 	<xacro:property name="wheel_offset_z" value="0.0" />
@@ -26,9 +26,9 @@
 	<!-- Here we create the robot elements using the xacro:macros imported at the beggining of this file -->
 	<!-- Summit XL base -->
-    <xacro:summit_xl_steel_base name="summit_xl" publish_bf="true" hq="${hq}"/>
+    <xacro:summit_xl_steel_base name="" publish_bf="true" hq="${hq}"/>
     <!-- Gazebo ros control pluggins -->
 	<xacro:ros_control prefix=""/>
     <!-- Gazebo omni steering plugin -->
-    <xacro:omni_steering/>
+    <xacro:omni_steering prefix=""/>
 	<!-- WHEELS -->
 	<xacro:omni_wheel name="front_right" parent="base_link" reflect="false" hq="true">

File: summit_xl_description/urdf/bases/summit_xl_base.gazebo.xacro (robot description, xacro)
@@ -35,5 +35,16 @@
     </gazebo>
   </xacro:macro>
-  <xacro:macro name="omni_steering">
+  <xacro:macro name="omni_steering" params="prefix">
+		<gazebo>
+	    <plugin name="omni_steering" filename="libgazebo_ros_planar_move.so">
+	      <commandTopic>${prefix}/summit_xl_control/cmd_vel</commandTopic>
+	      <odometryTopic>${prefix}/odom</odometryTopic>
+	      <odometryFrame>${prefix}odom</odometryFrame>
+	      <odometryRate>20.0</odometryRate>
+	      <robotBaseFrame>${prefix}base_footprint</robotBaseFrame>
+	    </plugin>
+	  </gazebo>
+  </xacro:macro>
+  <!-- xacro:macro name="omni_steering">
 		<gazebo>
 	    <plugin name="omni_steering" filename="libgazebo_ros_planar_move.so">
@@ -45,5 +56,5 @@
 	    </plugin>
 	  </gazebo>
-  </xacro:macro>
+  </xacro:macro -->
   <xacro:macro name="ros_force_based_move" params="broadcastOdomTF">
 	  <gazebo>

File: summit_xl_description/urdf/bases/summit_xl_steel_base.urdf.xacro (robot description, xacro)
@@ -8,5 +8,5 @@
   <!-- BASE FOOTPRINT -->
   <xacro:if value="${publish_bf}">
-    <link name="base_footprint">
+    <link name="${name}base_footprint">
       <visual>
           <origin xyz="0 0 0" rpy="0 0 0" />
@@ -16,12 +16,12 @@
       </visual>
     </link>
-    <joint name="base_footprint_joint" type="fixed">
+    <joint name="${name}base_footprint_joint" type="fixed">
       <origin xyz="0 0 ${wheel_radius}" rpy="0 0 0" /> <!-- ${wheel_radius} property must be defined inside wheel description -->
-      <parent link="base_footprint"/>
-      <child link="base_link" />
+      <parent link="${name}base_footprint"/>
+      <child link="${name}base_link" />
     </joint>
   </xacro:if>
   <!-- BASE_LINK -->
-  <link name="base_link">
+  <link name="${name}base_link">
     <inertial>
       <mass value="25.0" />
@@ -53,10 +53,10 @@
   </link>
    <!-- DOCKING CONTACT -->
-    <link name="base_docking_contact">
+    <link name="${name}base_docking_contact">
     </link>
-    <joint name="base_docking_joint" type="fixed">
+    <joint name="${name}base_docking_joint" type="fixed">
       <origin xyz="0.30 0 0.09" rpy="0 0 0" />
-      <parent link="base_link"/>
-      <child link="base_docking_contact" />
+      <parent link="${name}base_link"/>
+      <child link="${name}base_docking_contact" />
     </joint>
   </xacro:macro>
