Commit message: yaml,launch and xacro modified to multirobot

File: summit_xl_description/robots/summit_xl_multi.urdf.xacro (robot description, xacro)
@@ -11,5 +11,5 @@
 	<!-- Import all available sensors -->
 	<xacro:include filename="$(find robotnik_sensors)/urdf/all_sensors.urdf.xacro" />
-    <xacro:property name="PI" value="3.1415926535897931"/>
+	<xacro:property name="PI" value="3.1415926535897931"/>
 	<!-- Wheel parameters -->
 	<xacro:property name="wheel_offset_x" value="0.229" />    <!-- x,y,z in translation from base_link to the center of the wheel -->
@@ -18,6 +18,7 @@
 	<!-- Flag to select the high or low quality model -->
 	<xacro:property name="hq" value="true" />
-	<xacro:arg name="prefix" default="summit_xl"/>
-    <xacro:macro name="summit_xl_multi" params="prefix publish_bf hq">
+	<xacro:arg name="prefix_topic" default=""/>
+	<xacro:arg name="prefix_frame" default="summit_xl"/>
+    	<xacro:macro name="summit_xl_multi" params="prefix_frame prefix_topic publish_bf hq">
 		<!-- *************** -->
 		<!-- Robots Elements -->
@@ -25,26 +26,29 @@
 		<!-- Here we create the robot elements using the xacro:macros imported at the beggining of this file -->
 		<!-- Summit XL base -->
-		<xacro:summit_xl_base prefix="$(arg prefix)" publish_bf="true" hq="${hq}" />
-		<xacro:rubber_wheel name="$(arg prefix)front_right" parent="$(arg prefix)base_link" reflect="false" hq="${hq}">
+		<xacro:summit_xl_base prefix_frame="$(arg prefix_frame)" prefix_topic="$(arg prefix_topic)" publish_bf="true" hq="${hq}" />
+		<xacro:rubber_wheel name="$(arg prefix_frame)front_right" parent="$(arg prefix_frame)base_link" reflect="false" hq="${hq}">
 			<origin xyz="${wheel_offset_x} -${wheel_offset_y} ${wheel_offset_z}" rpy="0 0 0"/>
 		</xacro:rubber_wheel>
-		<xacro:rubber_wheel name="$(arg prefix)front_left" parent="$(arg prefix)base_link" reflect="true" hq="${hq}">
+		<xacro:rubber_wheel name="$(arg prefix_frame)front_left" parent="$(arg prefix_frame)base_link" reflect="true" hq="${hq}">
 			<origin xyz="${wheel_offset_x} ${wheel_offset_y} ${wheel_offset_z}" rpy="0 0 0"/>
 		</xacro:rubber_wheel>
-		<xacro:rubber_wheel name="$(arg prefix)back_left" parent="$(arg prefix)base_link" reflect="true" hq="${hq}">
+		<xacro:rubber_wheel name="$(arg prefix_frame)back_left" parent="$(arg prefix_frame)base_link" reflect="true" hq="${hq}">
 			<origin xyz="-${wheel_offset_x} ${wheel_offset_y} ${wheel_offset_z}" rpy="0 0 0"/>
 		</xacro:rubber_wheel>
-		<xacro:rubber_wheel name="$(arg prefix)back_right" parent="$(arg prefix)base_link" reflect="false" hq="${hq}">
+		<xacro:rubber_wheel name="$(arg prefix_frame)back_right" parent="$(arg prefix_frame)base_link" reflect="false" hq="${hq}">
 			<origin xyz="-${wheel_offset_x} -${wheel_offset_y} ${wheel_offset_z}" rpy="0 0 0"/>
 		</xacro:rubber_wheel>
-		<xacro:sensor_imu_hector name="$(arg prefix)imu" parent="$(arg prefix)base_link" >
+		<xacro:sensor_imu_hector prefix_frame="$(arg prefix_frame)imu" parent="$(arg prefix_frame)base_link" prefix_topic="$(arg prefix_topic)" >
 			<origin xyz="-0.18 0.0 0.170" rpy="0 0 0"/>
 		</xacro:sensor_imu_hector>
-		<xacro:sensor_hokuyo_ust10lx name="$(arg prefix)hokuyo_base" parent="$(arg prefix)base_link">
+		<xacro:sensor_hokuyo_ust10lx parent="$(arg prefix_frame)base_link" prefix_frame="$(arg prefix_frame)hokuyo_base" prefix_topic="$(arg prefix_topic)">
 			<origin xyz="0.0 0.0 0.33" rpy="0 0 0"/>
 		</xacro:sensor_hokuyo_ust10lx>
+		<!--xacro:sensor_hokuyo_ust10lx name="$(arg prefix_frame)hokuyo_base" parent="$(arg prefix_frame)base_link" prefix_frame="$(arg prefix_frame)" prefix_topic="$(arg prefix_topic)">
+                        <origin xyz="0.0 0.0 0.33" rpy="0 0 0"/>
+                </xacro:sensor_hokuyo_ust10lx-->
 		<!-- Gazebo ros control pluggins -->
-		<xacro:ros_control prefix="$(arg prefix)"/>
+		<xacro:ros_control prefix_topic="$(arg prefix_topic)" prefix_frame="$(arg prefix_frame)"/>
    </xacro:macro>
-   <xacro:summit_xl_multi prefix="$(arg prefix)" publish_bf="true" hq="true"/>
+   <xacro:summit_xl_multi prefix_frame="$(arg prefix_frame)" prefix_topic="$(arg prefix_topic)" publish_bf="true" hq="true"/>
 </robot>

File: summit_xl_description/urdf/bases/summit_xl_base.gazebo.xacro (robot description, xacro)
@@ -2,10 +2,11 @@
 <robot xmlns:xacro="http://www.ros.org/wiki/xacro">
   <!-- ros control plugin -->
-  <xacro:macro name="ros_control" params="prefix">
+  <xacro:macro name="ros_control" params="prefix_frame prefix_topic">
     <gazebo>
       <plugin name="ros_control" filename="libgazebo_ros_control.so">
         <!--<robotNamespace>/summit_xl</robotNamespace>-->
-        <robotNamespace>${prefix}</robotNamespace>
-        <robotParam>robot_description</robotParam>
+        <!--robotNamespace>${prefix_frame}/</robotNamespace-->
+        <!--robotNamespace>summit_xl_a</robotNamespace-->
+	<robotParam>robot_description</robotParam>
         <controlPeriod>0.001</controlPeriod>
 	    <robotSimType>gazebo_ros_control/DefaultRobotHWSim</robotSimType>
@@ -19,16 +20,17 @@
 			<!--<robotNamespace>/summit_xl</robotNamespace>-->
 		    <updateRate>100.0</updateRate>
-		    <leftFrontJoint>joint_front_left_wheel</leftFrontJoint>
-		    <rightFrontJoint>joint_front_right_wheel</rightFrontJoint>
-		    <leftRearJoint>joint_back_left_wheel</leftRearJoint>
-		    <rightRearJoint>joint_back_right_wheel</rightRearJoint>
+		    <leftFrontJoint>$(prefix_frame)joint_front_left_wheel</leftFrontJoint>
+		    <rightFrontJoint>$(prefix_frame)joint_front_right_wheel</rightFrontJoint>
+		    <leftRearJoint>$(prefix_frame)joint_back_left_wheel</leftRearJoint>
+		    <rightRearJoint>$(prefix_frame)joint_back_right_wheel</rightRearJoint>
 		    <!-- wheelSeparation>0.566</wheelSeparation --> <!-- real parameter value -->
 		    <wheelSeparation>1.5</wheelSeparation> <!-- works a bit better in Gazebo -->
 		    <wheelDiameter>0.234</wheelDiameter>
-		    <robotBaseFrame>base_footprint</robotBaseFrame>
+		    <robotBaseFrame>$(prefix_frame)base_footprint</robotBaseFrame>
 		    <torque>50</torque>
 		    <commandTopic>/summit_xl_control/cmd_vel</commandTopic>
 		    <odometryTopic>odom</odometryTopic>
-		    <odometryFrame>/odom</odometryFrame>
+		    <!--odometryFrame>/odom</odometryFrame-->
+		    <odometryFrame>$(prefix_frame)odom</odometryFrame>
 		    <broadcastTF>${broadcastOdomTF}</broadcastTF>
       </plugin>
@@ -42,5 +44,5 @@
 	      <odometryFrame>odom</odometryFrame>
 	      <odometryRate>20.0</odometryRate>
-	      <robotBaseFrame>base_footprint</robotBaseFrame>
+	      <robotBaseFrame>$(prefix_frame)base_footprint</robotBaseFrame>
 	    </plugin>
 	  </gazebo>
@@ -56,5 +58,5 @@
 			 <x_velocity_p_gain>10000.0</x_velocity_p_gain>
 			 <y_velocity_p_gain>10000.0</y_velocity_p_gain>
-			 <robotBaseFrame>base_footprint</robotBaseFrame>
+			 <robotBaseFrame>$(prefix_frame)base_footprint</robotBaseFrame>
 			 <odometryRate>20.0</odometryRate>
 			 <publishOdometryTf>${broadcastOdomTF}</publishOdometryTf>

File: summit_xl_description/urdf/bases/summit_xl_base.urdf.xacro (robot description, xacro)
@@ -2,5 +2,5 @@
 <robot name="summit_xl" xmlns:xacro="http://www.ros.org/wiki/xacro">
   <xacro:include filename="$(find summit_xl_description)/urdf/bases/summit_xl_base.gazebo.xacro" />
-  <xacro:macro name="summit_xl_base" params="prefix publish_bf hq">
+  <xacro:macro name="summit_xl_base" params="prefix_frame prefix_topic publish_bf hq">
 	  <!-- Robot mechanical and motor parameters -->
 	  <xacro:property name="PI" value="3.1415926535897931"/>
@@ -8,5 +8,5 @@
 	  <!-- BASE FOOTPRINT -->
 	  <xacro:if value="${publish_bf}">
-		<link name="${prefix}base_footprint">
+		<link name="${prefix_frame}base_footprint">
 		  <visual>
 			  <origin xyz="0 0 0" rpy="0 0 0" />
@@ -16,12 +16,12 @@
 		  </visual>
 		</link>
-		<joint name="${prefix}base_footprint_joint" type="fixed">
+		<joint name="${prefix_frame}base_footprint_joint" type="fixed">
 		  <origin xyz="0 0 ${wheel_radius}" rpy="0 0 0" /> <!-- ${wheel_radius} property must be defined inside wheel description -->
-		  <parent link="${prefix}base_footprint"/>
-		  <child link="${prefix}base_link" />
+		  <parent link="${prefix_frame}base_footprint"/>
+		  <child link="${prefix_frame}base_link" />
 		</joint>
 	  </xacro:if>
 	  <!-- BASE_LINK -->
-	  <link name="${prefix}base_link">
+	  <link name="${prefix_frame}base_link">
 		<inertial>
 		  <mass value="25.0" />

File: summit_xl_description/urdf/wheels/rubber_wheel.urdf.xacro (robot description, xacro)
@@ -59,5 +59,5 @@
       <type>transmission_interface/SimpleTransmission</type>
       <joint name="${name}_wheel_joint">
-        <hardwareInterface>VelocityJointInterface</hardwareInterface>
+        <hardwareInterface>hardware_interface/VelocityJointInterface</hardwareInterface>
       </joint>
       <actuator name="${name}_wheel_joint_motor">
