Commit message: xacro updated to multirobot

File: summit_xl_description/robots/summit_xl_multi.urdf.xacro (robot description, xacro)
@@ -18,7 +18,6 @@
 	<!-- Flag to select the high or low quality model -->
 	<xacro:property name="hq" value="true" />
-	<xacro:arg name="prefix_topic" default=""/>
-	<xacro:arg name="prefix_frame" default="summit_xl"/>
-    	<xacro:macro name="summit_xl_multi" params="prefix_frame prefix_topic publish_bf hq">
+	<xacro:arg name="prefix" default="summit_xl"/>
+    <xacro:macro name="summit_xl_multi" params="prefix publish_bf hq">
 		<!-- *************** -->
 		<!-- Robots Elements -->
@@ -26,29 +25,29 @@
 		<!-- Here we create the robot elements using the xacro:macros imported at the beggining of this file -->
 		<!-- Summit XL base -->
-		<xacro:summit_xl_base prefix_frame="$(arg prefix_frame)" prefix_topic="$(arg prefix_topic)" publish_bf="true" hq="${hq}" />
-		<xacro:rubber_wheel name="$(arg prefix_frame)front_right" parent="$(arg prefix_frame)base_link" reflect="false" hq="${hq}">
+		<xacro:summit_xl_base prefix="$(arg prefix)" publish_bf="true" hq="${hq}" />
+		<xacro:rubber_wheel prefix="$(arg prefix)front_right" parent="$(arg prefix)base_link" reflect="false" hq="${hq}">
 			<origin xyz="${wheel_offset_x} -${wheel_offset_y} ${wheel_offset_z}" rpy="0 0 0"/>
 		</xacro:rubber_wheel>
-		<xacro:rubber_wheel name="$(arg prefix_frame)front_left" parent="$(arg prefix_frame)base_link" reflect="true" hq="${hq}">
+		<xacro:rubber_wheel prefix="$(arg prefix)front_left" parent="$(arg prefix)base_link" reflect="true" hq="${hq}">
 			<origin xyz="${wheel_offset_x} ${wheel_offset_y} ${wheel_offset_z}" rpy="0 0 0"/>
 		</xacro:rubber_wheel>
-		<xacro:rubber_wheel name="$(arg prefix_frame)back_left" parent="$(arg prefix_frame)base_link" reflect="true" hq="${hq}">
+		<xacro:rubber_wheel prefix="$(arg prefix)back_left" parent="$(arg prefix)base_link" reflect="true" hq="${hq}">
 			<origin xyz="-${wheel_offset_x} ${wheel_offset_y} ${wheel_offset_z}" rpy="0 0 0"/>
 		</xacro:rubber_wheel>
-		<xacro:rubber_wheel name="$(arg prefix_frame)back_right" parent="$(arg prefix_frame)base_link" reflect="false" hq="${hq}">
+		<xacro:rubber_wheel prefix="$(arg prefix)back_right" parent="$(arg prefix)base_link" reflect="false" hq="${hq}">
 			<origin xyz="-${wheel_offset_x} -${wheel_offset_y} ${wheel_offset_z}" rpy="0 0 0"/>
 		</xacro:rubber_wheel>
-		<xacro:sensor_imu_hector prefix_frame="$(arg prefix_frame)imu" parent="$(arg prefix_frame)base_link" prefix_topic="$(arg prefix_topic)" >
+		<xacro:sensor_imu_hector prefix="$(arg prefix)imu" parent="$(arg prefix)base_link">
 			<origin xyz="-0.18 0.0 0.170" rpy="0 0 0"/>
 		</xacro:sensor_imu_hector>
-		<xacro:sensor_hokuyo_ust10lx name="hokuyo_base" parent="$(arg prefix_frame)base_link" prefix_frame="$(arg prefix_frame)" prefix_topic="$(arg prefix_topic)">
+		<xacro:sensor_hokuyo_ust10lx prefix="$(arg prefix)front_laser" parent="$(arg prefix)base_link">
 			<origin xyz="0.0 0.0 0.33" rpy="0 0 0"/>
 		</xacro:sensor_hokuyo_ust10lx>
-		<!--xacro:sensor_hokuyo_ust10lx name="$(arg prefix_frame)hokuyo_base" parent="$(arg prefix_frame)base_link" prefix_frame="$(arg prefix_frame)" prefix_topic="$(arg prefix_topic)">
+		<!--xacro:sensor_hokuyo_ust10lx prefix="$(arg prefix)hokuyo_base" parent="$(arg prefix)base_link">
                         <origin xyz="0.0 0.0 0.33" rpy="0 0 0"/>
                 </xacro:sensor_hokuyo_ust10lx-->
-		<!-- Gazebo ros control pluggins -->
-		<xacro:ros_control prefix_topic="$(arg prefix_topic)" prefix_frame="$(arg prefix_frame)"/>
    </xacro:macro>
-   <xacro:summit_xl_multi prefix_frame="$(arg prefix_frame)" prefix_topic="$(arg prefix_topic)" publish_bf="true" hq="true"/>
+   <!-- Gazebo ros control pluggins -->
+   <xacro:ros_control/>
+   <xacro:summit_xl_multi prefix="$(arg prefix)" publish_bf="true" hq="true"/>
 </robot>

File: summit_xl_description/robots/summit_xl_omni.urdf.xacro (robot description, xacro)
@@ -25,21 +25,22 @@
 	<!-- *************** -->
 	<!-- Here we create the robot elements using the xacro:macros imported at the beggining of this file -->
+	<xacro:arg name="prefix" default="summit_xl"/>
 	<!-- Summit XL base -->
-  <xacro:summit_xl_base name="summit_xl" publish_bf="true" hq="${hq}"/>
+  <xacro:summit_xl_base prefix="$(arg prefix)" publish_bf="true" hq="${hq}"/>
   <!-- Gazebo ros control pluggins -->
   <xacro:ros_control/>
   <!-- Gazebo omni steering plugin -->
-  <xacro:omni_steering/>
+  <xacro:omni_steering prefix="$(arg prefix)"/>
 	<!-- WHEELS -->
-	<xacro:omni_wheel name="front_right" parent="base_link" reflect="false" hq="true">
+	<xacro:omni_wheel prefix="$(arg prefix)front_right" parent="$(arg prefix)base_link" reflect="false" hq="true">
 		<origin xyz="${wheel_offset_x} -${wheel_offset_y} ${wheel_offset_z}" rpy="0 0 0"/>
 	</xacro:omni_wheel>
-	<xacro:omni_wheel name="front_left" parent="base_link" reflect="true" hq="true">
+	<xacro:omni_wheel prefix="$(arg prefix)front_left" parent="$(arg prefix)base_link" reflect="true" hq="true">
 		<origin xyz="${wheel_offset_x} ${wheel_offset_y} ${wheel_offset_z}" rpy="0 0 0"/>
 	</xacro:omni_wheel>
-	<xacro:omni_wheel name="back_left" parent="base_link" reflect="false" hq="true">
+	<xacro:omni_wheel prefix="$(arg prefix)back_left" parent="$(arg prefix)base_link" reflect="false" hq="true">
 		<origin xyz="-${wheel_offset_x} ${wheel_offset_y} ${wheel_offset_z}" rpy="0 0 0"/>
 	</xacro:omni_wheel>
-	<xacro:omni_wheel name="back_right" parent="base_link" reflect="true" hq="true">
+	<xacro:omni_wheel prefix="$(arg prefix)back_right" parent="$(arg prefix)base_link" reflect="true" hq="true">
 		<origin xyz="-${wheel_offset_x} -${wheel_offset_y} ${wheel_offset_z}" rpy="0 0 0"/>
 	</xacro:omni_wheel>
@@ -47,5 +48,5 @@
   <!-- Hokuyo laser sensors can be parametized with min_angle and max_angle e.g: -->
   <!--xacro:sensor_hokuyo_utm30lx name="hokuyo_base" parent="base_link" min_angle="2.35" max_angle="-2.35"-->
-	<xacro:sensor_hokuyo_utm30lx name="hokuyo_base" parent="base_link">
+	<xacro:sensor_hokuyo_utm30lx prefix="$(arg prefix)hokuyo_base" parent="$(arg prefix)base_link">
 		<origin xyz="0.0 0.0 0.33" rpy="0 0 0"/>
 	</xacro:sensor_hokuyo_utm30lx>
@@ -60,11 +61,11 @@
 	</xacro:sensor_hokuyo_ust10lx>
 -->
-	<xacro:sensor_axis name="camera" parent="base_link">
+	<xacro:sensor_axis prefix="$(arg prefix)camera" parent="$(arg prefix)base_link">
 		<origin xyz="0.19 0 0.17" rpy="0 ${-75*PI/180} 0"/>
 	</xacro:sensor_axis>
-	<xacro:sensor_imu name="imu" parent="base_link">
+	<xacro:sensor_imu prefix="$(arg prefix)imu" parent="$(arg prefix)base_link">
 		<origin xyz="-0.18 0.0 0.170" rpy="0 0 0"/>
 	</xacro:sensor_imu>
-	<xacro:sensor_gps name="gps" parent="base_link">
+	<xacro:sensor_gps prefix="$(arg prefix)gps" parent="$(arg prefix)base_link">
 		<origin xyz="-0.22 0 0.275" rpy="0 0 0"/>
 	</xacro:sensor_gps>

File: summit_xl_description/urdf/bases/summit_xl_base.gazebo.xacro (robot description, xacro)
@@ -2,9 +2,9 @@
 <robot xmlns:xacro="http://www.ros.org/wiki/xacro">
   <!-- ros control plugin -->
-  <xacro:macro name="ros_control" params="prefix_frame prefix_topic">
+  <xacro:macro name="ros_control">
     <gazebo>
       <plugin name="ros_control" filename="libgazebo_ros_control.so">
         <!--<robotNamespace>/summit_xl</robotNamespace>-->
-	<robotParam>robot_description</robotParam>
+		<robotParam>robot_description</robotParam>
         <controlPeriod>0.001</controlPeriod>
 	    <robotSimType>gazebo_ros_control/DefaultRobotHWSim</robotSimType>
@@ -13,48 +13,48 @@
 	</xacro:macro>
 	<!-- skid steering plugin -->
-	<xacro:macro name="skid_steering" params="broadcastOdomTF">
+	<xacro:macro name="skid_steering" params="broadcastOdomTF prefix">
     <gazebo>
       <plugin name="skid_steer_drive_controller" filename="libgazebo_ros_skid_steer_drive.so">
 			<!--<robotNamespace>/summit_xl</robotNamespace>-->
 		    <updateRate>100.0</updateRate>
-		    <leftFrontJoint>$(prefix_frame)joint_front_left_wheel</leftFrontJoint>
-		    <rightFrontJoint>$(prefix_frame)joint_front_right_wheel</rightFrontJoint>
-		    <leftRearJoint>$(prefix_frame)joint_back_left_wheel</leftRearJoint>
-		    <rightRearJoint>$(prefix_frame)joint_back_right_wheel</rightRearJoint>
+		    <leftFrontJoint>${prefix}joint_front_left_wheel</leftFrontJoint>
+		    <rightFrontJoint>${prefix}joint_front_right_wheel</rightFrontJoint>
+		    <leftRearJoint>${prefix}joint_back_left_wheel</leftRearJoint>
+		    <rightRearJoint>${prefix}joint_back_right_wheel</rightRearJoint>
 		    <!-- wheelSeparation>0.566</wheelSeparation --> <!-- real parameter value -->
 		    <wheelSeparation>1.5</wheelSeparation> <!-- works a bit better in Gazebo -->
 		    <wheelDiameter>0.234</wheelDiameter>
-		    <robotBaseFrame>$(prefix_frame)base_footprint</robotBaseFrame>
+		    <robotBaseFrame>${prefix}base_footprint</robotBaseFrame>
 		    <torque>50</torque>
-		    <commandTopic>/summit_xl_control/cmd_vel</commandTopic>
+		    <commandTopic>summit_xl_control/cmd_vel</commandTopic>
 		    <odometryTopic>odom</odometryTopic>
 		    <!--odometryFrame>/odom</odometryFrame-->
-		    <odometryFrame>$(prefix_frame)odom</odometryFrame>
+		    <odometryFrame>${prefix}odom</odometryFrame>
 		    <broadcastTF>${broadcastOdomTF}</broadcastTF>
       </plugin>
     </gazebo>
   </xacro:macro>
-  <xacro:macro name="omni_steering">
+  <xacro:macro name="omni_steering" params="prefix">
 		<gazebo>
 	    <plugin name="omni_steering" filename="libgazebo_ros_planar_move.so">
-	      <commandTopic>/summit_xl_control/cmd_vel</commandTopic>
-	      <odometryTopic>/odom</odometryTopic>
-	      <odometryFrame>odom</odometryFrame>
+	      <commandTopic>summit_xl_control/cmd_vel</commandTopic>
+	      <odometryTopic>odom</odometryTopic>
+	      <odometryFrame>${prefix}odom</odometryFrame>
 	      <odometryRate>20.0</odometryRate>
-	      <robotBaseFrame>$(prefix_frame)base_footprint</robotBaseFrame>
+	      <robotBaseFrame>${prefix}base_footprint</robotBaseFrame>
 	    </plugin>
 	  </gazebo>
   </xacro:macro>
-  <xacro:macro name="ros_force_based_move" params="broadcastOdomTF">
+  <xacro:macro name="ros_force_based_move" params="broadcastOdomTF prefix">
 	  <gazebo>
 		 <plugin name="ros_force_based_move" filename="libgazebo_ros_force_based_move.so">
 			 <!--<robotNamespace>/summit_xl</robotNamespace>-->
-			 <commandTopic>/summit_xl_control/cmd_vel</commandTopic>
-			 <odometryTopic>/summit_xl/odom</odometryTopic>
+			 <commandTopic>summit_xl_control/cmd_vel</commandTopic>
+			 <odometryTopic>summit_xl/odom</odometryTopic>
 	         <odometryFrame>odom</odometryFrame>
 			 <yaw_velocity_p_gain>10000.0</yaw_velocity_p_gain>
 			 <x_velocity_p_gain>10000.0</x_velocity_p_gain>
 			 <y_velocity_p_gain>10000.0</y_velocity_p_gain>
-			 <robotBaseFrame>$(prefix_frame)base_footprint</robotBaseFrame>
+			 <robotBaseFrame>${prefix}base_footprint</robotBaseFrame>
 			 <odometryRate>20.0</odometryRate>
 			 <publishOdometryTf>${broadcastOdomTF}</publishOdometryTf>

File: summit_xl_description/urdf/bases/summit_xl_base.urdf.xacro (robot description, xacro)
@@ -2,5 +2,5 @@
 <robot name="summit_xl" xmlns:xacro="http://www.ros.org/wiki/xacro">
   <xacro:include filename="$(find summit_xl_description)/urdf/bases/summit_xl_base.gazebo.xacro" />
-  <xacro:macro name="summit_xl_base" params="prefix_frame prefix_topic publish_bf hq">
+  <xacro:macro name="summit_xl_base" params="prefix publish_bf hq">
 	  <!-- Robot mechanical and motor parameters -->
 	  <xacro:property name="PI" value="3.1415926535897931"/>
@@ -8,5 +8,5 @@
 	  <!-- BASE FOOTPRINT -->
 	  <xacro:if value="${publish_bf}">
-		<link name="${prefix_frame}base_footprint">
+		<link name="${prefix}base_footprint">
 		  <visual>
 			  <origin xyz="0 0 0" rpy="0 0 0" />
@@ -16,12 +16,12 @@
 		  </visual>
 		</link>
-		<joint name="${prefix_frame}base_footprint_joint" type="fixed">
+		<joint name="${prefix}base_footprint_joint" type="fixed">
 		  <origin xyz="0 0 ${wheel_radius}" rpy="0 0 0" /> <!-- ${wheel_radius} property must be defined inside wheel description -->
-		  <parent link="${prefix_frame}base_footprint"/>
-		  <child link="${prefix_frame}base_link" />
+		  <parent link="${prefix}base_footprint"/>
+		  <child link="${prefix}base_link" />
 		</joint>
 	  </xacro:if>
 	  <!-- BASE_LINK -->
-	  <link name="${prefix_frame}base_link">
+	  <link name="${prefix}base_link">
 		<inertial>
 		  <mass value="25.0" />

File: summit_xl_description/urdf/bases/summit_xl_hls_base.urdf.xacro (robot description, xacro)
@@ -2,5 +2,5 @@
 <robot name="summit_xl" xmlns:xacro="http://www.ros.org/wiki/xacro">
   <xacro:include filename="$(find summit_xl_description)/urdf/bases/summit_xl_base.gazebo.xacro" />
-  <xacro:macro name="summit_xl_hls_base" params="name publish_bf hq">
+  <xacro:macro name="summit_xl_hls_base" params="prefix publish_bf hq">
   <!-- Robot mechanical and motor parameters -->
   <xacro:property name="PI" value="3.1415926535897931"/>
@@ -8,5 +8,5 @@
   <!-- BASE FOOTPRINT -->
   <xacro:if value="${publish_bf}">
-    <link name="base_footprint">
+    <link name="${prefix}base_footprint">
       <visual>
           <origin xyz="0 0 0" rpy="0 0 0" />
@@ -16,12 +16,12 @@
       </visual>
     </link>
-    <joint name="base_footprint_joint" type="fixed">
+    <joint name="${prefix}base_footprint_joint" type="fixed">
       <origin xyz="0 0 ${wheel_radius}" rpy="0 0 0" /> <!-- ${wheel_radius} property must be defined inside wheel description -->
-      <parent link="base_footprint"/>
-      <child link="base_link" />
+      <parent link="${prefix}base_footprint"/>
+      <child link="${prefix}base_link" />
     </joint>
   </xacro:if>
   <!-- BASE_LINK -->
-  <link name="base_link">
+  <link name="${prefix}base_link">
     <inertial>
       <mass value="25.0" />
@@ -53,10 +53,10 @@
   </link>
    <!-- DOCKING CONTACT -->
-    <link name="base_docking_contact">
+    <link name="${prefix}base_docking_contact">
     </link>
-    <joint name="base_docking_joint" type="fixed">
+    <joint name="${prefix}base_docking_joint" type="fixed">
       <origin xyz="0.30 0 0.09" rpy="0 0 0" />
-      <parent link="base_link"/>
-      <child link="base_docking_contact" />
+      <parent link="${prefix}base_link"/>
+      <child link="${prefix}base_docking_contact" />
     </joint>
   </xacro:macro>

File: summit_xl_description/urdf/structures/structure_hokuyo.urdf.xacro (robot description, xacro)
@@ -1,12 +1,12 @@
 <?xml version="1.0"?>
 <robot name="structure" xmlns:xacro="http://ros.org/wiki/xacro">
-  <xacro:macro name="structure" params="name parent *origin">
-	  <joint name="${name}_joint" type="fixed">
+  <xacro:macro name="structure" params="prefix parent *origin">
+	  <joint name="${prefix}_joint" type="fixed">
 	    <axis xyz="0 1 0"/>
 	    <xacro:insert_block name="origin"/>
 	    <parent link="${parent}"/>
-	    <child link="${name}_link"/>
+	    <child link="${prefix}_link"/>
 	  </joint>
-	  <link name="${name}_link">
+	  <link name="${prefix}_link">
 	    <inertial>
 	      <mass value="0.001"/>
@@ -30,5 +30,5 @@
 	    </collision>
 	  </link>
-	  <gazebo reference="${name}_link">
+	  <gazebo reference="${prefix}_link">
 	    <material>Gazebo/White</material>
 	    <gravity>true</gravity>

File: summit_xl_description/urdf/structures/structure_ptz_rgbd_gps.urdf.xacro (robot description, xacro)
@@ -1,12 +1,12 @@
 <?xml version="1.0"?>
 <robot name="structure" xmlns:xacro="http://ros.org/wiki/xacro">
-  <xacro:macro name="structure" params="name parent *origin">
-	  <joint name="${name}_joint" type="fixed">
+  <xacro:macro name="structure" params="prefix parent *origin">
+	  <joint name="${prefix}_joint" type="fixed">
 	    <axis xyz="0 1 0"/>
 	    <xacro:insert_block name="origin"/>
 	    <parent link="${parent}"/>
-	    <child link="${name}_link"/>
+	    <child link="${prefix}_link"/>
 	  </joint>
-	  <link name="${name}_link">
+	  <link name="${prefix}_link">
 	    <inertial>
 	      <mass value="0.001"/>
@@ -30,5 +30,5 @@
 	    </collision>
 	  </link>
-	  <gazebo reference="${name}_link">
+	  <gazebo reference="${prefix}_link">
 	    <material>Gazebo/White</material>
 	    <gravity>true</gravity>

File: summit_xl_description/urdf/wheels/omni_wheel.urdf.xacro (robot description, xacro)
@@ -11,8 +11,8 @@
               izz="${m*(3*r*r+h*h)/12}" />
   </xacro:macro>
-  <xacro:macro name="omni_wheel" params="name parent *origin reflect hq">
-    <joint name="joint_${name}_wheel" type="continuous">
+  <xacro:macro name="omni_wheel" params="prefix parent *origin reflect hq">
+    <joint name="${prefix}_wheel_joint" type="continuous">
       <parent link="${parent}"/>
-      <child link="${name}_wheel"/>
+      <child link="${prefix}_wheel_link"/>
       <xacro:insert_block name="origin" />
       <axis xyz="0 1 0" rpy="0 0 0" />
@@ -20,5 +20,5 @@
       <joint_properties damping="0.0" friction="0.0"/>
     </joint>
-    <link name="${name}_wheel">
+    <link name="${prefix}_wheel_link">
       <visual>
         <xacro:if value="${hq}">
@@ -69,14 +69,14 @@
     </link>
     <!-- Transmission is important to link the joints and the controller (see summit_xl_control/config/summit_xl_control.yaml)-->
-    <transmission name="${name}_wheel_joint_trans">
+    <transmission name="${prefix}_wheel_joint_trans">
       <type>transmission_interface/SimpleTransmission</type>
-      <joint name="joint_${name}_wheel" >
+      <joint name="${prefix}_wheel_joint" >
         <hardwareInterface>VelocityJointInterface</hardwareInterface>
       </joint>
-      <actuator name="${name}_wheel_joint_motor">
+      <actuator name="${prefix}_wheel_joint_motor">
          <mechanicalReduction>1</mechanicalReduction>
       </actuator>
     </transmission>
-    <gazebo reference="${name}_wheel">
+    <gazebo reference="${prefix}_wheel_link">
 		<mu1 value="1.0"/>
 		<mu2 value="1.0"/>

File: summit_xl_description/urdf/wheels/rubber_wheel.urdf.xacro (robot description, xacro)
@@ -11,9 +11,9 @@
               izz="${m*(3*r*r+h*h)/12}" />
   </xacro:macro>
-  <xacro:macro name="rubber_wheel" params="name parent *origin reflect hq">
+  <xacro:macro name="rubber_wheel" params="prefix parent *origin reflect hq">
 <!--WHEEL TIRE -->
-    <joint name="${name}_wheel_joint" type="continuous">
+    <joint name="${prefix}_wheel_joint" type="continuous">
       <parent link="${parent}"/>
-      <child link="${name}_wheel"/>
+      <child link="${prefix}_wheel"/>
       <xacro:insert_block name="origin" />
       <axis xyz="0 1 0" rpy="0 0 0" />
@@ -21,5 +21,5 @@
       <joint_properties damping="0.0" friction="0.0"/>
     </joint>
-    <link name="${name}_wheel">
+    <link name="${prefix}_wheel">
       <visual>
         <!-- HIGH RESOLUTION WHEELS -->
@@ -56,15 +56,15 @@
     </link>
     <!-- Transmission is important to link the joints and the controller (see summit_xl_control/config/summit_xl_control.yaml)-->
-    <transmission name="${name}_wheel_joint_trans">
+    <transmission name="${prefix}_wheel_joint_trans">
       <type>transmission_interface/SimpleTransmission</type>
-      <joint name="${name}_wheel_joint">
+      <joint name="${prefix}_wheel_joint">
         <hardwareInterface>hardware_interface/VelocityJointInterface</hardwareInterface>
       </joint>
-      <actuator name="${name}_wheel_joint_motor">
+      <actuator name="${prefix}_wheel_joint_motor">
         <mechanicalReduction>1</mechanicalReduction>
         <motorTorqueConstant>20</motorTorqueConstant>
       </actuator>
      </transmission>
-    <gazebo reference="${name}_wheel">
+    <gazebo reference="${prefix}_wheel">
 			<mu1 value="1.0"/>
 			<mu2 value="1.0"/>

Commit message: rangefinders in correct pos in multi cfg

File: summit_xl_description/robots/summit_xl_multi.urdf.xacro (robot description, xacro)
@@ -41,6 +41,9 @@
 			<origin xyz="-0.18 0.0 0.170" rpy="0 0 0"/>
 		</xacro:sensor_imu_hector>
-		<xacro:sensor_hokuyo_ust10lx name="$(arg prefix)hokuyo_base" parent="$(arg prefix)base_link">
-			<origin xyz="0.0 0.0 0.33" rpy="0 0 0"/>
+		<xacro:sensor_hokuyo_ust10lx name="laser_front" parent="base_link">
+			<origin xyz="0.373 -0.210 0.205" rpy="0 0 -0.7854"/>
+		</xacro:sensor_hokuyo_ust10lx>
+		<xacro:sensor_hokuyo_ust10lx name="laser_rear" parent="base_link">
+			<origin xyz="-0.373 0.210 0.205" rpy="0 0 2.3562"/>
 		</xacro:sensor_hokuyo_ust10lx>
 		<!-- Gazebo ros control pluggins -->

Commit message: corrected urdf - 1 laser

File: summit_xl_description/robots/summit_xl_multi.urdf.xacro (robot description, xacro)
@@ -41,9 +41,6 @@
 			<origin xyz="-0.18 0.0 0.170" rpy="0 0 0"/>
 		</xacro:sensor_imu_hector>
-		<xacro:sensor_hokuyo_ust10lx name="laser_front" parent="base_link">
-			<origin xyz="0.373 -0.210 0.205" rpy="0 0 -0.7854"/>
-		</xacro:sensor_hokuyo_ust10lx>
-		<xacro:sensor_hokuyo_ust10lx name="laser_rear" parent="base_link">
-			<origin xyz="-0.373 0.210 0.205" rpy="0 0 2.3562"/>
+		<xacro:sensor_hokuyo_ust10lx name="$(arg prefix)laser_front" parent="$(arg prefix)base_link">
+			<origin xyz="0.0 0.0 0.33" rpy="0 0 0"/>
 		</xacro:sensor_hokuyo_ust10lx>
 		<!-- Gazebo ros control pluggins -->
