Commit message: corrected urdf - 2 laser and 2 cameras

File: summit_xl_description/robots/summit_xl_steel_multi.urdf.xacro (robot description, xacro)
@@ -42,7 +42,16 @@
 			<origin xyz="-0.18 0.0 0.170" rpy="0 0 0"/>
 		</xacro:sensor_imu_hector>
-		<xacro:sensor_hokuyo_ust10lx name="$(arg prefix)hokuyo_base" parent="$(arg prefix)base_link">
-			<origin xyz="0.0 0.0 0.33" rpy="0 0 0"/>
+		<xacro:sensor_hokuyo_ust10lx name="$(arg prefix)laser_front" parent="$(arg prefix)base_link">
+			<origin xyz="0.373 -0.210 0.205" rpy="0 0 -0.7854"/>
 		</xacro:sensor_hokuyo_ust10lx>
+		<xacro:sensor_hokuyo_ust10lx name="$(arg prefix)laser_rear" parent="$(arg prefix)base_link">
+			<origin xyz="-0.373 0.210 0.205" rpy="0 0 2.3562"/>
+		</xacro:sensor_hokuyo_ust10lx>
+		<xacro:sensor_axis_m5013 name="$(arg prefix)camera_front" parent="$(arg prefix)base_link">
+			<origin xyz="0.308 0.140 0.195" rpy="0 0 0"/>
+		</xacro:sensor_axis_m5013>
+		<xacro:sensor_axis_m5013 name="$(arg prefix)camera_rear" parent="$(arg prefix)base_link">
+			<origin xyz="-0.308 -0.140 0.195" rpy="0 0 3.1416"/>
+		</xacro:sensor_axis_m5013>
 		<!-- Gazebo ros control pluggins -->
 		<xacro:ros_control prefix="$(arg prefix)"/>
