Commit message: summit_xl_description:: Added summit_x. Added use_joint_state_publisher param

File: summit_xl_description/robots/summit_x_std.urdf.xacro (robot description, xacro)
@@ -52,7 +52,7 @@
 		</xacro:sensor_axis>
 	    <!-- RGBD -->
-	    <xacro:sensor_orbbec_astra prefix="$(arg prefix)front_rgbd_camera" parent="$(arg prefix)upper_base_link" prefix_topic="front_rgbd_camera">
+	    <!--xacro:sensor_orbbec_astra prefix="$(arg prefix)front_rgbd_camera" parent="$(arg prefix)upper_base_link" prefix_topic="front_rgbd_camera">
 			<origin xyz="0.13 0.0 0.1" rpy="0 0 0"/>
-		</xacro:sensor_orbbec_astra>
+		</xacro:sensor_orbbec_astra-->
 	    <!-- GPS -->
 	    <xacro:sensor_gps prefix="$(arg prefix)gps" parent="$(arg prefix)upper_base_link">

File: summit_xl_description/urdf/bases/summit_x_base.urdf.xacro (robot description, xacro)
@@ -81,4 +81,14 @@
 		<axis xyz="0 0 1"/>
 	</joint>
+	<!-- auxiliar joint that pushes the 'X' -->
+	<link name="${prefix}aux_upper_base_link">
+	</link>
+	<joint name="${prefix}aux_upper_base_joint" type="prismatic">
+		<parent link="${prefix}base_link"/>
+		<child link="${prefix}aux_upper_base_link"/>
+		<limit effort="100000.0" velocity="1000.0" lower="0.0" upper="0.5"/> <!-- lower="0.1" upper="0.5" -->
+		<origin rpy="0 ${PI/2} 0" xyz="-0.261 -0.15 0.0"/>
+		<axis xyz="0 0 1"/>
+	</joint>
 	<transmission name="${prefix}upper_base_joint_trans">
 		<type>transmission_interface/SimpleTransmission</type>
@@ -90,4 +100,13 @@
 		 </actuator>
 	</transmission>
+	<transmission name="${prefix}aux_upper_base_joint_trans">
+		<type>transmission_interface/SimpleTransmission</type>
+		<joint name="${prefix}aux_upper_base_joint">
+		  <hardwareInterface>EffortJointInterface</hardwareInterface>
+		</joint>
+		<actuator name="${prefix}aux_upper_base_motor">
+		  <mechanicalReduction>1</mechanicalReduction>
+		 </actuator>
+	</transmission>
   </xacro:macro>
 </robot>
