Commit message: Update on gazebo model for Steel

File: summit_xl_description/robots/summit_xls_std.urdf.xacro (robot description, xacro)
@@ -6,5 +6,5 @@
 	<!-- First we import all posible elements defined in the urdf.xacro files. All these elements are defined as macro:xacros -->
 	<!-- Import summit XL base elements -->
-	<xacro:include filename="$(find summit_xl_description)/urdf/bases/summit_xl_hls_base.urdf.xacro" />
+	<xacro:include filename="$(find summit_xl_description)/urdf/bases/summit_xls_base.urdf.xacro" />
 	<!-- Import summit XL wheels -->
 	<xacro:include filename="$(find summit_xl_description)/urdf/wheels/omni_wheel.urdf.xacro" />
@@ -50,5 +50,5 @@
 		<!-- Here we create the robot elements using the xacro:macros imported at the beggining of this file -->
 		<!-- Summit XL base -->
-		<xacro:summit_xl_hls_base prefix="$(arg prefix)" publish_bf="true" hq="${hq}" />
+		<xacro:summit_xls_base prefix="$(arg prefix)" publish_bf="true" hq="${hq}" />
 		<xacro:omni_wheel prefix="$(arg prefix)front_right" parent="$(arg prefix)base_link" reflect="false" hq="${hq}">
 			<origin xyz="${wheel_offset_x} -${wheel_offset_y} ${wheel_offset_z}" rpy="0 0 0"/>
@@ -75,22 +75,22 @@
 		</xacro:structure_laser-->
 		<!-- SENSORS -->
-		<xacro:sensor_hokuyo_ust10lx prefix="$(arg prefix)front_laser" parent="$(arg prefix)base_link" prefix_topic="front_laser">
+		<!--xacro:sensor_hokuyo_ust10lx prefix="$(arg prefix)front_laser" parent="$(arg prefix)base_link" prefix_topic="front_laser">
 			<origin xyz="${front_laser_offset_x} ${front_laser_offset_y} ${front_laser_offset_z}" rpy="0 0 ${-PI/4.0}"/>
-		</xacro:sensor_hokuyo_ust10lx>
-		<xacro:sensor_hokuyo_ust10lx prefix="$(arg prefix)rear_laser" parent="$(arg prefix)base_link" prefix_topic="rear_laser">
+		</xacro:sensor_hokuyo_ust10lx-->
+		<!--xacro:sensor_hokuyo_ust10lx prefix="$(arg prefix)rear_laser" parent="$(arg prefix)base_link" prefix_topic="rear_laser">
 			<origin xyz="${rear_laser_offset_x} ${rear_laser_offset_y} ${rear_laser_offset_z}" rpy="0 0 ${3.0*PI/4.0}"/>
-		</xacro:sensor_hokuyo_ust10lx>
-		<xacro:sensor_axis_m5013 prefix="$(arg prefix)front_ptz_camera" parent="$(arg prefix)base_link">
+		</xacro:sensor_hokuyo_ust10lx-->
+		<!--xacro:sensor_axis_m5013 prefix="$(arg prefix)front_ptz_camera" parent="$(arg prefix)base_link">
 			<origin xyz="${front_ptz_camera_offset_x} ${front_ptz_camera_offset_y} ${front_ptz_camera_offset_z}" rpy="${-PI/2} 0 0"/>
-		</xacro:sensor_axis_m5013>
-		<xacro:sensor_axis_m5013 prefix="$(arg prefix)rear_ptz_camera" parent="$(arg prefix)base_link">
+		</xacro:sensor_axis_m5013-->
+		<!--xacro:sensor_axis_m5013 prefix="$(arg prefix)rear_ptz_camera" parent="$(arg prefix)base_link">
 			<origin xyz="${rear_ptz_camera_offset_x} ${rear_ptz_camera_offset_y} ${rear_ptz_camera_offset_z}" rpy="${-PI/2} 0 ${PI}"/>
-		</xacro:sensor_axis_m5013>
-		<xacro:sensor_orbbec_astra prefix="$(arg prefix)front_rgbd_camera" parent="$(arg prefix)base_link" prefix_topic="front_rgbd_camera">
+		</xacro:sensor_axis_m5013-->
+		<!--xacro:sensor_orbbec_astra prefix="$(arg prefix)front_rgbd_camera" parent="$(arg prefix)base_link" prefix_topic="front_rgbd_camera">
 			<origin xyz="${front_rgbd_camera_offset_x} ${front_rgbd_camera_offset_y} ${front_rgbd_camera_offset_z}" rpy="0 0 0"/>
-		</xacro:sensor_orbbec_astra>
-		<xacro:sensor_gps prefix="$(arg prefix)gps" parent="$(arg prefix)base_link">
+		</xacro:sensor_orbbec_astra-->
+		<!--xacro:sensor_gps prefix="$(arg prefix)gps" parent="$(arg prefix)base_link">
 			<origin xyz="${gps_offset_x} ${gps_offset_y} ${gps_offset_z}" rpy="0 0 0"/>
-		</xacro:sensor_gps>
+		</xacro:sensor_gps-->
    </xacro:macro>
    <xacro:ros_control/>

File: summit_xl_description/urdf/bases/summit_xls_base.urdf.xacro (robot description, xacro)
@@ -2,8 +2,8 @@
 <robot name="summit_xl" xmlns:xacro="http://www.ros.org/wiki/xacro">
   <xacro:include filename="$(find summit_xl_description)/urdf/bases/summit_xl_base.gazebo.xacro" />
-  <xacro:macro name="summit_xl_hls_base" params="prefix publish_bf hq">
-	  <!-- Robot mechanical and motor parameters -->
-	  <xacro:property name="PI" value="3.1415926535897931"/>
-	  <xacro:property name="wheel_width" value="0.175" />
+  <xacro:macro name="summit_xls_base" params="prefix publish_bf hq">
+  <!-- Robot mechanical and motor parameters -->
+  <xacro:property name="PI" value="3.1415926535897931"/>
+  <xacro:property name="wheel_width" value="0.175" />
 	<!-- BASE FOOTPRINT -->
 	  <xacro:if value="${publish_bf}">
@@ -30,26 +30,114 @@
     </inertial>
     <visual>
-       <origin xyz="0 0 0" rpy="0 0 0" />
-       <xacro:if value="${hq}">
-       <geometry>
-	     <mesh filename="package://summit_xl_description/meshes/bases/hls/summit_xls_chassis.stl"/>
-       </geometry>
-       </xacro:if>
-       <xacro:unless value="${hq}">
-       <geometry>
-	     <mesh filename="package://summit_xl_description/meshes/bases/hls/summit_xls_chassis.dae"/>
-       </geometry>
-       </xacro:unless>
-       <material name="darkgrey">
-         <color rgba="0.1 0.1 0.1 1"/>
-       </material>
+      <origin xyz="0 0 0" rpy="0 0 0" />
+      <xacro:if value="${hq}">
+      <geometry>
+      <mesh filename="package://summit_xl_description/meshes/bases/xls/summit_xls_chassis.stl"/>
+      </geometry>
+      </xacro:if>
+      <xacro:unless value="${hq}">
+      <geometry>
+      <mesh filename="package://summit_xl_description/meshes/bases/xls/summit_xls_chassis.dae"/>
+      </geometry>
+      </xacro:unless>
+      <material name="black">
+        <color rgba="0.0 0.0 0.0 1"/>
+      </material>
     </visual>
     <collision>
        <origin xyz="0 0 0" rpy="0 0 0 " />
        <geometry>
-         <mesh filename="package://summit_xl_description/meshes/bases/hls/summit_xls_chassis.dae"/>
+         <mesh filename="package://summit_xl_description/meshes/bases/xls/summit_xls_chassis.dae"/>
        </geometry>
     </collision>
   </link>
+  <gazebo reference="${prefix}base_link">
+    <material>Gazebo/Black</material>
+  </gazebo>
+  <!-- CHAPAS INOX TAPAS -->
+  <link name="${prefix}base_chapa">
+  <visual>
+    <origin xyz="0 0 0" rpy="0 0 0" />
+    <geometry>
+    <mesh filename="package://summit_xl_description/meshes/bases/xls/summit_xls_chapas_inox_tapas.stl"/>
+    </geometry>
+    <material name="darkgrey">
+      <color rgba="0.5 0.5 0.5 1"/>
+    </material>
+    </visual>
+  </link>
+  <joint name="${prefix}base_tapa_joint" type="fixed">
+    <origin xyz="0.0 0 0.38062" rpy="0 0 0" />
+    <parent link="${prefix}base_link"/>
+    <child link="${prefix}base_chapa" />
+  </joint>
+  <!-- LOGO ROBOTNIK IZQUIERDO -->
+  <link name="${prefix}base_logo_left">
+  <visual>
+    <origin xyz="0 0 0" rpy="0 0 0" />
+    <geometry>
+    <mesh filename="package://summit_xl_description/meshes/bases/xls/robotnik_logo_chasis.stl"/>
+    </geometry>
+    <material name="darkgrey">
+      <color rgba="0.5 0.5 0.5 1"/>
+    </material>
+    </visual>
+  </link>
+  <joint name="${prefix}base_logo_left_joint" type="fixed">
+    <origin xyz="0.0 0.28931 0.29062" rpy="0 0 0" />
+    <parent link="${prefix}base_link"/>
+    <child link="${prefix}base_logo_left" />
+  </joint>
+  <!-- LOGO ROBOTNIK DERECHO -->
+  <link name="${prefix}base_logo_right">
+  <visual>
+    <origin xyz="0 0 0" rpy="0 0 0" />
+    <geometry>
+    <mesh filename="package://summit_xl_description/meshes/bases/xls/robotnik_logo_chasis.stl"/>
+    </geometry>
+    <material name="darkgrey">
+      <color rgba="0.5 0.5 0.5 1"/>
+    </material>
+    </visual>
+  </link>
+  <joint name="${prefix}base_logo_right_joint" type="fixed">
+    <origin xyz="0.0 -0.28931 0.29062" rpy="0 0 ${PI}" />
+    <parent link="${prefix}base_link"/>
+    <child link="${prefix}base_logo_right" />
+  </joint>
+  <!-- LOGO ROBOTNIK FRONTAL -->
+  <link name="${prefix}base_logo_front">
+  <visual>
+    <origin xyz="0 0 0" rpy="0 0 0" />
+    <geometry>
+    <mesh filename="package://summit_xl_description/meshes/bases/xls/robotnik_logo_chasis.stl"/>
+    </geometry>
+    <material name="darkgrey">
+      <color rgba="0.5 0.5 0.5 1"/>
+    </material>
+    </visual>
+  </link>
+  <joint name="${prefix}base_logo_front_joint" type="fixed">
+    <origin xyz="0.345 0.0 0.0" rpy="0 0 ${-PI/2}" />
+    <parent link="${prefix}base_link"/>
+    <child link="${prefix}base_logo_front" />
+  </joint>
+  <!-- LOGO ROBOTNIK TRASERO -->
+  <link name="${prefix}base_logo_rear">
+  <visual>
+    <origin xyz="0 0 0" rpy="0 0 0" />
+    <geometry>
+    <mesh filename="package://summit_xl_description/meshes/bases/xls/robotnik_logo_chasis.stl"/>
+    </geometry>
+    <material name="darkgrey">
+      <color rgba="0.5 0.5 0.5 1"/>
+    </material>
+    </visual>
+  </link>
+  <joint name="${prefix}base_logo_rear_joint" type="fixed">
+    <origin xyz="-0.345 0.0 0.0" rpy="0 0 ${PI/2}" />
+    <parent link="${prefix}base_link"/>
+    <child link="${prefix}base_logo_rear" />
+  </joint>
    <!-- DOCKING CONTACT -->
     <link name="${prefix}base_docking_contact">

Commit message: description: Update XLS model with default configuration

File: summit_xl_description/robots/summit_xls_std.urdf.xacro (robot description, xacro)
@@ -19,10 +19,10 @@
 	<xacro:property name="wheel_offset_y" value="0.2045" />
 	<xacro:property name="wheel_offset_z" value="0.0" />
-	<xacro:property name="front_laser_offset_x" value="0.377"/>
-	<xacro:property name="front_laser_offset_y" value="-0.20957"/>
-	<xacro:property name="front_laser_offset_z" value="0.2024"/>
-	<xacro:property name="rear_laser_offset_x" value="-0.377"/>
-	<xacro:property name="rear_laser_offset_y" value="0.20957"/>
-	<xacro:property name="rear_laser_offset_z" value="0.2024"/>
+	<xacro:property name="front_laser_offset_x" value="0.2865"/>
+	<xacro:property name="front_laser_offset_y" value="-0.20894"/>
+	<xacro:property name="front_laser_offset_z" value="0.2973"/>
+	<xacro:property name="rear_laser_offset_x" value="-0.2865"/>
+	<xacro:property name="rear_laser_offset_y" value="0.20894"/>
+	<xacro:property name="rear_laser_offset_z" value="0.2973"/>
 	<xacro:property name="front_ptz_camera_offset_x" value="0.308"/>
 	<xacro:property name="front_ptz_camera_offset_y" value="0.141"/>
@@ -31,10 +31,10 @@
 	<xacro:property name="rear_ptz_camera_offset_y" value="-0.141"/>
 	<xacro:property name="rear_ptz_camera_offset_z" value="0.195"/>
-	<xacro:property name="imu_offset_x" value="0.25"/>
-	<xacro:property name="imu_offset_y" value="-0.15"/>
-	<xacro:property name="imu_offset_z" value="0.18"/>
-	<xacro:property name="front_rgbd_camera_offset_x" value="0.324"/>
-	<xacro:property name="front_rgbd_camera_offset_y" value="0.012"/>
-	<xacro:property name="front_rgbd_camera_offset_z" value="0.230"/>
+	<xacro:property name="imu_offset_x" value="0.13"/>
+	<xacro:property name="imu_offset_y" value="-0.273"/>
+	<xacro:property name="imu_offset_z" value="0.066"/>
+	<xacro:property name="front_rgbd_camera_offset_x" value="0.35850"/>
+	<xacro:property name="front_rgbd_camera_offset_y" value="0.0"/>
+	<xacro:property name="front_rgbd_camera_offset_z" value="0.25062"/>
 	<xacro:property name="gps_offset_x" value="-0.365"/>
 	<xacro:property name="gps_offset_y" value="-0.167"/>
@@ -65,20 +65,13 @@
         <!-- IMU -->
 		<xacro:sensor_imu_hector prefix="$(arg prefix)imu" parent="$(arg prefix)base_link">
-			<origin xyz="-0.18 0.0 0.170" rpy="0 0 0"/>
+			<origin xyz="${imu_offset_x} ${imu_offset_y} ${imu_offset_z}" rpy="0 0 0"/>
 		</xacro:sensor_imu_hector>
-		<!-- Structures -->
-		<!--xacro:structure_laser prefix="$(arg prefix)front_laser_structure" parent="$(arg prefix)base_link">
-			<origin xyz="0.303 -0.160 0.155" rpy="0 0 0" />
-		</xacro:structure_laser>
-		<xacro:structure_laser prefix="$(arg prefix)rear_laser_structure" parent="$(arg prefix)base_link">
-			<origin xyz="-0.303 0.160 0.155" rpy="0 0 ${PI}" />
-		</xacro:structure_laser-->
 		<!-- SENSORS -->
-		<!--xacro:sensor_hokuyo_ust10lx prefix="$(arg prefix)front_laser" parent="$(arg prefix)base_link" prefix_topic="front_laser">
-			<origin xyz="${front_laser_offset_x} ${front_laser_offset_y} ${front_laser_offset_z}" rpy="0 0 ${-PI/4.0}"/>
-		</xacro:sensor_hokuyo_ust10lx-->
-		<!--xacro:sensor_hokuyo_ust10lx prefix="$(arg prefix)rear_laser" parent="$(arg prefix)base_link" prefix_topic="rear_laser">
-			<origin xyz="${rear_laser_offset_x} ${rear_laser_offset_y} ${rear_laser_offset_z}" rpy="0 0 ${3.0*PI/4.0}"/>
-		</xacro:sensor_hokuyo_ust10lx-->
+		<xacro:sensor_sick_s300 prefix="$(arg prefix)front_laser" parent="$(arg prefix)base_link" prefix_topic="front_laser">
+			<origin xyz="${front_laser_offset_x} ${front_laser_offset_y} ${front_laser_offset_z}" rpy="0 ${-PI} ${3/4*PI}" />
+		</xacro:sensor_sick_s300>
+		<xacro:sensor_sick_s300 prefix="$(arg prefix)rear_laser" parent="$(arg prefix)base_link" prefix_topic="rear_laser">
+			<origin xyz="${rear_laser_offset_x} ${rear_laser_offset_y} ${rear_laser_offset_z}" rpy="0 ${-PI} ${-1/4*PI}" />
+		</xacro:sensor_sick_s300>
 		<!--xacro:sensor_axis_m5013 prefix="$(arg prefix)front_ptz_camera" parent="$(arg prefix)base_link">
 			<origin xyz="${front_ptz_camera_offset_x} ${front_ptz_camera_offset_y} ${front_ptz_camera_offset_z}" rpy="${-PI/2} 0 0"/>
@@ -87,7 +80,7 @@
 			<origin xyz="${rear_ptz_camera_offset_x} ${rear_ptz_camera_offset_y} ${rear_ptz_camera_offset_z}" rpy="${-PI/2} 0 ${PI}"/>
 		</xacro:sensor_axis_m5013-->
-		<!--xacro:sensor_orbbec_astra prefix="$(arg prefix)front_rgbd_camera" parent="$(arg prefix)base_link" prefix_topic="front_rgbd_camera">
+		<xacro:sensor_orbbec_astra prefix="$(arg prefix)front_rgbd_camera" parent="$(arg prefix)base_link" prefix_topic="front_rgbd_camera">
 			<origin xyz="${front_rgbd_camera_offset_x} ${front_rgbd_camera_offset_y} ${front_rgbd_camera_offset_z}" rpy="0 0 0"/>
-		</xacro:sensor_orbbec_astra-->
+		</xacro:sensor_orbbec_astra>
 		<!--xacro:sensor_gps prefix="$(arg prefix)gps" parent="$(arg prefix)base_link">
 			<origin xyz="${gps_offset_x} ${gps_offset_y} ${gps_offset_z}" rpy="0 0 0"/>
