Commit message: Adjusts model parameters to a less unstable and more realistic behaviour of the rocker-bogie

File: summit_xl_description/robots/summit_xls_cobolleague.urdf.xacro (robot description, xacro)
@@ -6,5 +6,6 @@
 	<!-- First we import all posible elements defined in the urdf.xacro files. All these elements are defined as macro:xacros -->
 	<!-- Import summit XL base elements -->
-	<xacro:include filename="$(find summit_xl_description)/urdf/bases/summit_xls_base.urdf.xacro" />
+	<!-- xacro:include filename="$(find summit_xl_description)/urdf/bases/summit_xls_base.urdf.xacro" / -->
+	<xacro:include filename="$(find summit_xl_description)/urdf/bases/cobolleague_base.urdf.xacro" />
 	<!-- Import summit XL wheels -->
 	<xacro:include filename="$(find summit_xl_description)/urdf/wheels/omni_wheel.urdf.xacro" />

File: summit_xl_description/urdf/rocker/rocker.urdf.xacro (robot description, xacro)
@@ -5,5 +5,5 @@
   <xacro:property name="M_PI" value="3.1415926535897931" />
   <!-- Rocker support parameters -->
-  <xacro:property name="rocker_support_mass" value="10" /> <!-- in kg-->
+  <xacro:property name="rocker_support_mass" value="15" /> <!-- in kg-->
   <xacro:macro name="cylinder_inertia" params="m r h">
     <inertia  ixx="${m*(3*r*r+h*h)/12}" ixy = "0" ixz = "0"
@@ -17,6 +17,10 @@
       <insert_block name="origin" />
       <axis xyz="0 1 0" rpy="0 0 ${M_PI}" />
-      <limit lower="-0.5" upper="0.5" effort="100" velocity="0.5"/>
-      <joint_properties damping="5.0" friction="0.4"/>
+      <limit lower="-0.7854" upper="0.7854" effort="1" velocity="0.1"/>
+      <!-- joint_properties damping="10.0" friction="0.8"/ -->
+      <!-- joint_properties damping="10.0" friction="0.8"/ -->
+	  <!-- safety_controller k_position="100.0" k_velocity="10.0" soft_lower_limit="-0.65" soft_upper_limit="0.65"/ -->
+      <!-- dynamics damping="100" friction="0.5"/ -->
+      <joint_properties damping="10.0" friction="0.2"/>
 	</joint>
 	<!-- joint name="${prefix}joint_rsupport" type="fixed">
@@ -48,12 +52,13 @@
 	  <type>transmission_interface/SimpleTransmission</type>
 	  <joint name="${prefix}_rsupport_joint">
-		  <hardwareInterface>hardware_interface/EffortJointInterface</hardwareInterface>
+		  <hardwareInterface>hardware_interface/PositionJointInterface</hardwareInterface>
 	  </joint>
 	  <actuator name="${prefix}_rsupport_joint_motor">
-		<mechanicalReduction>1</mechanicalReduction>
-		<motorTorqueConstant>1</motorTorqueConstant>
+		<hardwareInterface>hardware_interface/PositionJointInterface</hardwareInterface>
+		<mechanicalReduction>0.1</mechanicalReduction>
+		<motorTorqueConstant>0.1</motorTorqueConstant>
 	  </actuator>
 	</transmission -->
-    <!-- transmission name="${prefix}_rsupport_joint_trans">
+    <transmission name="${prefix}_rsupport_joint_trans">
       <type>transmission_interface/SimpleTransmission</type>
       <joint name="${prefix}_rsupport_joint">
@@ -63,8 +68,9 @@
         <hardwareInterface>hardware_interface/VelocityJointInterface</hardwareInterface>
         <mechanicalReduction>1</mechanicalReduction>
+        <motorTorqueConstant>1</motorTorqueConstant>
       </actuator>
-    </transmission -->
+    </transmission>
 	<!-- Transmission is important to link the joints and the controller -->
-	<transmission name="${prefix}rsupport_joint_trans">
+	<!-- transmission name="${prefix}rsupport_joint_trans">
 	  <type>transmission_interface/SimpleTransmission</type>
 	  <joint name="${prefix}_rsupport_joint">
@@ -72,8 +78,8 @@
 	  </joint>
 	  <actuator name="${prefix}rsupport_joint_motor">
-		<mechanicalReduction>20</mechanicalReduction>
-		<motorTorqueConstant>1</motorTorqueConstant>
+		<mechanicalReduction>200</mechanicalReduction>
+		<motorTorqueConstant>0.1</motorTorqueConstant>
 	  </actuator>
-	</transmission>
+	</transmission -->
 	<!-- Flag to select the high or low quality model -->
 	<xacro:property name="hq" value="true" />
@@ -81,5 +87,5 @@
     <xacro:property name="wheel_offset_y" value="-0.075" />
     <xacro:property name="wheel_offset_z" value="-0.100" />
-	<joint name="${prefix}_joint_rsupport_front" type="fixed">
+	<!-- joint name="${prefix}_joint_rsupport_front" type="fixed">
 	  <origin xyz="${wheel_offset_x} ${wheel_offset_y} ${wheel_offset_z}" rpy="0 0 0"/>
       <parent link="${prefix}rsupport"/>
@@ -94,5 +100,5 @@
 	</joint>
 	<link name="${prefix}_rsupport_mid">
-	</link>
+	</link -->
 	<xacro:if value="${reflect}">
 		<xacro:property name="wheel_offset_y" value="0.095" />
