Commit message: summit_xl_description: Parse kinematics param inside the xacro files

File: summit_xl_description/robots/summit_xl_gen_std.urdf.xacro (robot description, xacro)
@@ -29,7 +29,7 @@
     <xacro:arg name="ros_planar_move_plugin" default="false"/>
     <xacro:arg name="ros_planar_move_plugin_force_based" default="false"/>
-    <xacro:arg name="omni_wheels" default="false"/>
+    <xacro:arg name="kinematics" default="skid"/>
     <xacro:arg name="gpu" default="false"/>
-    <xacro:macro name="summit_xl_gen" params="prefix publish_bf hq">
+    <xacro:macro name="summit_xl_gen" params="prefix publish_bf hq kinematics">
         <!-- *************** -->
         <!-- Robots Elements -->
@@ -38,5 +38,5 @@
         <!-- Summit XL base -->
         <xacro:summit_xl_base prefix="$(arg prefix)" publish_bf="true" hq="${hq}" />
-        <xacro:unless value="$(arg omni_wheels)">
+        <xacro:if value="${kinematics == 'skid' or kinematics == 'skid_4w'}">
             <xacro:rubber_wheel prefix="$(arg prefix)front_right" parent="$(arg prefix)base_link" reflect="false" hq="${hq}">
                 <origin xyz="${wheel_offset_x} -${wheel_offset_y} ${wheel_offset_z}" rpy="0 0 0"/>
@@ -51,6 +51,6 @@
                 <origin xyz="-${wheel_offset_x} -${wheel_offset_y} ${wheel_offset_z}" rpy="0 0 0"/>
             </xacro:rubber_wheel>
-        </xacro:unless>
-        <xacro:if value="$(arg omni_wheels)">
+        </xacro:if>
+        <xacro:if value="${kinematics == 'omni' or kinematics == 'omni_4w'}">
             <xacro:omni_wheel prefix="$(arg prefix)front_right" parent="$(arg prefix)base_link" reflect="false" hq="${hq}">
                 <origin xyz="${wheel_offset_x} -${wheel_offset_y} ${wheel_offset_z}" rpy="0 0 0"/>
@@ -99,15 +99,15 @@
         <link name="$(arg prefix)arm_base_link" />
         <xacro:j2s7s300 base_parent="$(arg prefix)arm_base_link" prefix="$(arg prefix)j2s7s300"/>
+        <!-- Gazebo ros control pluggins -->
+        <xacro:ros_control/>
+        <xacro:if value="$(arg ros_planar_move_plugin)">
+		    <xacro:if value="${kinematics == 'omni' or kinematics == 'omni_4w'}">
+                <xacro:omni_steering prefix="$(arg prefix)" publish_tf="true" force_based="$(arg ros_planar_move_plugin_force_based)"/>
+            </xacro:if>
+		    <xacro:if value="${kinematics == 'skid' or kinematics == 'skid_4w'}">
+                <xacro:skid_steering prefix="$(arg prefix)" publish_tf="true" force_based="$(arg ros_planar_move_plugin_force_based)"/>
+            </xacro:if>
+        </xacro:if>
     </xacro:macro>
-    <!-- Gazebo ros control pluggins -->
-    <xacro:ros_control/>
-    <xacro:if value="$(arg ros_planar_move_plugin)">
-		<xacro:if value="$(arg omni_wheels)">
-			<xacro:omni_steering prefix="$(arg prefix)" publish_tf="true" force_based="$(arg ros_planar_move_plugin_force_based)"/>
-		</xacro:if>
-		<xacro:unless value="$(arg omni_wheels)">
-			<xacro:skid_steering prefix="$(arg prefix)" publish_tf="true" force_based="$(arg ros_planar_move_plugin_force_based)"/>
-		</xacro:unless>
-    </xacro:if>
-    <xacro:summit_xl_gen prefix="$(arg prefix)" publish_bf="true" hq="true"/>
+    <xacro:summit_xl_gen prefix="$(arg prefix)" publish_bf="true" hq="true" kinematics="$(arg kinematics)"/>
 </robot>

File: summit_xl_description/robots/summit_xl_std.urdf.xacro (robot description, xacro)
@@ -14,4 +14,6 @@
 	<!-- Import antenna -->
 	<xacro:include filename="$(find summit_xl_description)/urdf/structures/structure_teltonika.urdf.xacro" />
+	<!-- Import antenna -->
+	<xacro:include filename="$(find summit_xl_description)/urdf/structures/structure_teltonika.urdf.xacro" />
 	<xacro:property name="PI" value="3.1415926535897931"/>
 	<!-- Wheel parameters -->
@@ -23,10 +25,10 @@
 	<xacro:arg name="prefix" default="summit_xl_"/>
 	<xacro:arg name="ros_planar_move_plugin" default="false"/>
-  <xacro:arg name="ros_planar_move_plugin_force_based" default="false"/>
-	<xacro:arg name="omni_wheels" default="false"/>
+    <xacro:arg name="ros_planar_move_plugin_force_based" default="false"/>
+	<xacro:arg name="kinematics" default="skid"/>
 	<xacro:arg name="gpu" default="false"/>
 	<xacro:arg name="gps_latitude" default="0"/>
 	<xacro:arg name="gps_longitude" default="0"/>
-    <xacro:macro name="summit_xl" params="prefix publish_bf hq">
+    <xacro:macro name="summit_xl" params="prefix publish_bf hq kinematics">
 		<!-- *************** -->
 		<!-- Robots Elements -->
@@ -35,5 +37,5 @@
 		<!-- Summit XL base -->
 		<xacro:summit_xl_base prefix="$(arg prefix)" publish_bf="true" hq="${hq}" />
-    <xacro:unless value="$(arg omni_wheels)">
+    <xacro:if value="${kinematics == 'skid' or kinematics == 'skid_4w'}">
   		<xacro:rubber_wheel prefix="$(arg prefix)front_right" parent="$(arg prefix)base_link" reflect="false" hq="${hq}">
   			<origin xyz="${wheel_offset_x} -${wheel_offset_y} ${wheel_offset_z}" rpy="0 0 0"/>
@@ -48,6 +50,6 @@
   			<origin xyz="-${wheel_offset_x} -${wheel_offset_y} ${wheel_offset_z}" rpy="0 0 0"/>
   		</xacro:rubber_wheel>
-    </xacro:unless>
-    <xacro:if value="$(arg omni_wheels)">
+    </xacro:if>
+    <xacro:if value="${kinematics == 'omni' or kinematics == 'omni_4w'}">
   		<xacro:omni_wheel prefix="$(arg prefix)front_right" parent="$(arg prefix)base_link" reflect="false" hq="${hq}">
   			<origin xyz="${wheel_offset_x} -${wheel_offset_y} ${wheel_offset_z}" rpy="0 0 0"/>
@@ -83,19 +85,15 @@
 			<origin xyz="-0.22528 0.095 0.275" rpy="0 0 0"/>
 		</xacro:sensor_gps_with_mast>
-	  <!--Antenna-->
-	  	<xacro:structure_mastil_teltonika prefix="$(arg prefix)antenna" parent="$(arg prefix)base_link">
-			<origin xyz="-0.22528 -0.095 0.23325" rpy="0 0 0"/>
-		</xacro:structure_mastil_teltonika>
-   </xacro:macro>
-   <!-- Gazebo ros control pluggins -->
-   <xacro:ros_control/>
-	<xacro:if value="$(arg ros_planar_move_plugin)">
-		<xacro:if value="$(arg omni_wheels)">
+	  <!-- Gazebo ros control pluggins -->
+      <xacro:ros_control/>
+	  <xacro:if value="$(arg ros_planar_move_plugin)">
+		<xacro:if value="${kinematics == 'omni' or kinematics == 'omni_4w'}">
 			<xacro:omni_steering prefix="$(arg prefix)" publish_tf="true" force_based="$(arg ros_planar_move_plugin_force_based)"/>
 		</xacro:if>
-		<xacro:unless value="$(arg omni_wheels)">
+		<xacro:if value="${kinematics == 'skid' or kinematics == 'skid_4w'}">
 			<xacro:skid_steering prefix="$(arg prefix)" publish_tf="true" force_based="$(arg ros_planar_move_plugin_force_based)"/>
-		</xacro:unless>
-	</xacro:if>
-   <xacro:summit_xl prefix="$(arg prefix)" publish_bf="true" hq="true"/>
+		</xacro:if>
+	  </xacro:if>
+   </xacro:macro>
+   <xacro:summit_xl prefix="$(arg prefix)" publish_bf="true" hq="true" kinematics="$(arg kinematics)"/>
 </robot>

File: summit_xl_description/robots/summit_xl_tix_std.urdf.xacro (robot description, xacro)
@@ -29,7 +29,7 @@
     <xacro:arg name="ros_planar_move_plugin" default="false"/>
     <xacro:arg name="ros_planar_move_plugin_force_based" default="false"/>
-    <xacro:arg name="omni_wheels" default="false"/>
+    <xacro:arg name="kinematics" default="skid"/>
     <xacro:arg name="gpu" default="false"/>
-    <xacro:macro name="summit_xl_tix" params="prefix publish_bf hq">
+    <xacro:macro name="summit_xl_tix" params="prefix publish_bf hq kinematics">
         <!-- *************** -->
         <!-- Robots Elements -->
@@ -38,5 +38,5 @@
         <!-- Summit XL base -->
         <xacro:summit_xl_base prefix="$(arg prefix)" publish_bf="true" hq="${hq}" />
-        <xacro:unless value="$(arg omni_wheels)">
+        <xacro:if value="${kinematics == 'skid' or kinematics == 'skid_4w'}">
             <xacro:rubber_wheel prefix="$(arg prefix)front_right" parent="$(arg prefix)base_link" reflect="false" hq="${hq}">
                 <origin xyz="${wheel_offset_x} -${wheel_offset_y} ${wheel_offset_z}" rpy="0 0 0"/>
@@ -51,6 +51,6 @@
                 <origin xyz="-${wheel_offset_x} -${wheel_offset_y} ${wheel_offset_z}" rpy="0 0 0"/>
             </xacro:rubber_wheel>
-        </xacro:unless>
-        <xacro:if value="$(arg omni_wheels)">
+        </xacro:if>
+        <xacro:if value="${kinematics == 'omni' or kinematics == 'omni_4w'}">
             <xacro:omni_wheel prefix="$(arg prefix)front_right" parent="$(arg prefix)base_link" reflect="false" hq="${hq}">
                 <origin xyz="${wheel_offset_x} -${wheel_offset_y} ${wheel_offset_z}" rpy="0 0 0"/>
@@ -93,15 +93,15 @@
             <origin xyz="0.0 0.0 0.05" rpy="0 0 0"/>
         </xacro:sensor_intel_d435>
+        <!-- Gazebo ros control pluggins -->
+        <xacro:ros_control/>
+        <xacro:if value="$(arg ros_planar_move_plugin)">
+		    <xacro:if value="${kinematics == 'omni' or kinematics == 'omni_4w'}">
+                <xacro:omni_steering prefix="$(arg prefix)" publish_tf="true" force_based="$(arg ros_planar_move_plugin_force_based)"/>
+            </xacro:if>
+		    <xacro:if value="${kinematics == 'skid' or kinematics == 'skid_4w'}">
+                <xacro:skid_steering prefix="$(arg prefix)" publish_tf="true" force_based="$(arg ros_planar_move_plugin_force_based)"/>
+            </xacro:if>
+        </xacro:if>
     </xacro:macro>
-    <!-- Gazebo ros control pluggins -->
-    <xacro:ros_control/>
-    <xacro:if value="$(arg ros_planar_move_plugin)">
-		<xacro:if value="$(arg omni_wheels)">
-			<xacro:omni_steering prefix="$(arg prefix)" publish_tf="true" force_based="$(arg ros_planar_move_plugin_force_based)"/>
-		</xacro:if>
-		<xacro:unless value="$(arg omni_wheels)">
-			<xacro:skid_steering prefix="$(arg prefix)" publish_tf="true" force_based="$(arg ros_planar_move_plugin_force_based)"/>
-		</xacro:unless>
-    </xacro:if>
-    <xacro:summit_xl_tix prefix="$(arg prefix)" publish_bf="true" hq="true"/>
+    <xacro:summit_xl_tix prefix="$(arg prefix)" publish_bf="true" hq="true" kinematics="$(arg kinematics)"/>
 </robot>
