Commit message: description: using gazebo_planar_move plugin for the omnidrive configuration

File: summit_xl_description/robots/summit_xl_std.urdf.xacro (robot description, xacro)
@@ -19,4 +19,5 @@
 	<xacro:property name="hq" value="true" />
 	<xacro:arg name="prefix" default="summit_xl_"/>
+	<xacro:arg name="ros_planar_move_plugin" default="false"/>
     <xacro:macro name="summit_xl" params="prefix publish_bf hq">
 		<!-- *************** -->
@@ -61,4 +62,7 @@
    <!-- Gazebo ros control pluggins -->
    <xacro:ros_control/>
+   <xacro:if value="$(arg ros_planar_move_plugin)">
+	   <xacro:omni_steering prefix="$(arg prefix)" publish_tf="false"/>
+   </xacro:if>
    <xacro:summit_xl prefix="$(arg prefix)" publish_bf="true" hq="true"/>
 </robot>

File: summit_xl_description/robots/summit_xls_std.urdf.xacro (robot description, xacro)
@@ -43,4 +43,5 @@
 	<xacro:property name="hq" value="true" />
 	<xacro:arg name="prefix" default="summit_xl_"/>
+	<xacro:arg name="ros_planar_move_plugin" default="false"/>
     <xacro:macro name="summit_xl" params="prefix publish_bf hq">
 		<!-- *************** -->
@@ -74,8 +75,8 @@
 		</xacro:structure_laser-->
 		<!-- SENSORS -->
-		<xacro:sensor_hokuyo_ust10lx prefix="$(arg prefix)front_laser" parent="$(arg prefix)base_link">
+		<xacro:sensor_hokuyo_ust10lx prefix="$(arg prefix)front_laser" parent="$(arg prefix)base_link" prefix_topic="front_laser">
 			<origin xyz="${front_laser_offset_x} ${front_laser_offset_y} ${front_laser_offset_z}" rpy="0 0 ${-PI/4.0}"/>
 		</xacro:sensor_hokuyo_ust10lx>
-		<xacro:sensor_hokuyo_ust10lx prefix="$(arg prefix)rear_laser" parent="$(arg prefix)base_link">
+		<xacro:sensor_hokuyo_ust10lx prefix="$(arg prefix)rear_laser" parent="$(arg prefix)base_link" prefix_topic="rear_laser">
 			<origin xyz="${rear_laser_offset_x} ${rear_laser_offset_y} ${rear_laser_offset_z}" rpy="0 0 ${3.0*PI/4.0}"/>
 		</xacro:sensor_hokuyo_ust10lx>
@@ -86,5 +87,5 @@
 			<origin xyz="${rear_ptz_camera_offset_x} ${rear_ptz_camera_offset_y} ${rear_ptz_camera_offset_z}" rpy="${-PI/2} 0 ${PI}"/>
 		</xacro:sensor_axis_m5013>
-		<xacro:sensor_orbbec_astra prefix="$(arg prefix)front_rgbd_camera" parent="$(arg prefix)base_link">
+		<xacro:sensor_orbbec_astra prefix="$(arg prefix)front_rgbd_camera" parent="$(arg prefix)base_link" prefix_topic="front_rgbd_camera">
 			<origin xyz="${front_rgbd_camera_offset_x} ${front_rgbd_camera_offset_y} ${front_rgbd_camera_offset_z}" rpy="0 0 0"/>
 		</xacro:sensor_orbbec_astra>
@@ -93,6 +94,8 @@
 		</xacro:sensor_gps>
    </xacro:macro>
-   <!-- Gazebo ros control pluggins -->
    <xacro:ros_control/>
+   <xacro:if value="$(arg ros_planar_move_plugin)">
+	   <xacro:omni_steering prefix="$(arg prefix)" publish_tf="false"/>
+   </xacro:if>
    <xacro:summit_xl prefix="$(arg prefix)" publish_bf="true" hq="true"/>
 </robot>

File: summit_xl_description/urdf/bases/summit_xl_base.gazebo.xacro (robot description, xacro)
@@ -35,28 +35,28 @@
     </gazebo>
   </xacro:macro>
-  <xacro:macro name="omni_steering" params="prefix">
+  <xacro:macro name="omni_steering" params="prefix publish_tf">
 		<gazebo>
 	    <plugin name="omni_steering" filename="libgazebo_ros_planar_move.so">
 	      <commandTopic>summit_xl_control/cmd_vel</commandTopic>
-	      <odometryTopic>odom</odometryTopic>
+	      <odometryTopic>summit_xl_control/odom</odometryTopic>
 	      <odometryFrame>${prefix}odom</odometryFrame>
-	      <odometryRate>20.0</odometryRate>
+	      <odometryRate>50.0</odometryRate>
 	      <robotBaseFrame>${prefix}base_footprint</robotBaseFrame>
+	      <publishTF>${publish_tf}</publishTF>
 	    </plugin>
 	  </gazebo>
   </xacro:macro>
-  <xacro:macro name="ros_force_based_move" params="broadcastOdomTF prefix">
+  <xacro:macro name="ros_force_based_move" params="publish_tf prefix">
 	  <gazebo>
 		 <plugin name="ros_force_based_move" filename="libgazebo_ros_force_based_move.so">
-			 <!--<robotNamespace>/summit_xl</robotNamespace>-->
 			 <commandTopic>summit_xl_control/cmd_vel</commandTopic>
-			 <odometryTopic>summit_xl/odom</odometryTopic>
-	         <odometryFrame>odom</odometryFrame>
+			 <odometryTopic>summit_xl_control/odom</odometryTopic>
+	         <odometryFrame>${prefix}odom</odometryFrame>
 			 <yaw_velocity_p_gain>10000.0</yaw_velocity_p_gain>
 			 <x_velocity_p_gain>10000.0</x_velocity_p_gain>
 			 <y_velocity_p_gain>10000.0</y_velocity_p_gain>
 			 <robotBaseFrame>${prefix}base_footprint</robotBaseFrame>
-			 <odometryRate>20.0</odometryRate>
-			 <publishOdometryTf>${broadcastOdomTF}</publishOdometryTf>
+			 <odometryRate>50.0</odometryRate>
+			 <publishOdometryTf>${publish_tf}</publishOdometryTf>
 		 </plugin>
 	  </gazebo>

Commit message: description: Update XL model, wheel radius property

File: summit_xl_description/robots/summit_xl_std.urdf.xacro (robot description, xacro)
@@ -15,5 +15,5 @@
 	<!-- Wheel parameters -->
 	<xacro:property name="wheel_offset_x" value="0.229" />    <!-- x,y,z in translation from base_link to the center of the wheel -->
-	<xacro:property name="wheel_offset_y" value="0.234" />
+	<xacro:property name="wheel_offset_y" value="0.235" />
 	<xacro:property name="wheel_offset_z" value="0.0" />
 	<!-- Flag to select the high or low quality model -->

File: summit_xl_description/urdf/bases/summit_xl_base.gazebo.xacro (robot description, xacro)
@@ -14,23 +14,22 @@
 	</xacro:macro>
 	<!-- skid steering plugin -->
-	<xacro:macro name="skid_steering" params="broadcastOdomTF prefix">
+	<xacro:macro name="skid_steering" params="prefix publish_tf">
     <gazebo>
       <plugin name="skid_steer_drive_controller" filename="libgazebo_ros_skid_steer_drive.so">
 			<!--<robotNamespace>/summit_xl</robotNamespace>-->
-		    <updateRate>100.0</updateRate>
-		    <leftFrontJoint>${prefix}joint_front_left_wheel</leftFrontJoint>
-		    <rightFrontJoint>${prefix}joint_front_right_wheel</rightFrontJoint>
-		    <leftRearJoint>${prefix}joint_back_left_wheel</leftRearJoint>
-		    <rightRearJoint>${prefix}joint_back_right_wheel</rightRearJoint>
+		    <updateRate>50.0</updateRate>
+		    <leftFrontJoint>${prefix}front_left_wheel_joint</leftFrontJoint>
+		    <rightFrontJoint>${prefix}front_right_wheel_joint</rightFrontJoint>
+		    <leftRearJoint>${prefix}back_left_wheel_joint</leftRearJoint>
+		    <rightRearJoint>${prefix}back_right_wheel_joint</rightRearJoint>
 		    <!-- wheelSeparation>0.566</wheelSeparation --> <!-- real parameter value -->
-		    <wheelSeparation>1.5</wheelSeparation> <!-- works a bit better in Gazebo -->
-		    <wheelDiameter>0.234</wheelDiameter>
+		    <wheelSeparation>0.462</wheelSeparation> <!-- works a bit better in Gazebo -->
+		    <wheelDiameter>0.22</wheelDiameter>
 		    <robotBaseFrame>${prefix}base_footprint</robotBaseFrame>
 		    <torque>50</torque>
 		    <commandTopic>robotnik_base_control/cmd_vel</commandTopic>
 		    <odometryTopic>robotnik_base_control/odom</odometryTopic>
-		    <!--odometryFrame>/odom</odometryFrame-->
 		    <odometryFrame>${prefix}odom</odometryFrame>
-		    <broadcastTF>${broadcastOdomTF}</broadcastTF>
+		    <broadcastTF>${publish_tf}</broadcastTF>
       </plugin>
     </gazebo>

File: summit_xl_description/urdf/bases/summit_xl_base.urdf.xacro (robot description, xacro)
@@ -5,5 +5,5 @@
 	  <!-- Robot mechanical and motor parameters -->
 	  <xacro:property name="PI" value="3.1415926535897931"/>
-	  <xacro:property name="wheel_width" value="0.175" />
+	  <xacro:property name="wheel_radius" value="0.11"/>
 	  <!-- BASE FOOTPRINT -->
 	  <xacro:if value="${publish_bf}">

File: summit_xl_description/urdf/bases/summit_xls_base.urdf.xacro (robot description, xacro)
@@ -5,5 +5,5 @@
   <!-- Robot mechanical and motor parameters -->
   <xacro:property name="PI" value="3.1415926535897931"/>
-  <xacro:property name="wheel_width" value="0.175" />
+  <xacro:property name="wheel_radius" value="0.127" />
 	<!-- BASE FOOTPRINT -->
 	  <xacro:if value="${publish_bf}">

Commit message: Update xmlns:xacro to http://wiki.ros.org/xacro
    - URL updated

File: summit_xl_description/robots/summit_xl_std.urdf.xacro (robot description, xacro)
@@ -1,4 +1,4 @@
 <?xml version="1.0"?>
-<robot name="summit_xl" xmlns:xacro="http://www.ros.org/wiki/xacro">
+<robot name="summit_xl" xmlns:xacro="http://wiki.ros.org/xacro">
 	<!-- ***************** -->
 	<!-- Imported elements -->

File: summit_xl_description/robots/summit_xls_std.urdf.xacro (robot description, xacro)
@@ -31,7 +31,7 @@
 	<xacro:property name="rear_ptz_camera_offset_y" value="-0.141"/>
 	<xacro:property name="rear_ptz_camera_offset_z" value="0.195"/>
-	<xacro:property name="imu_offset_x" value="0.13"/>
-	<xacro:property name="imu_offset_y" value="-0.273"/>
-	<xacro:property name="imu_offset_z" value="0.066"/>
+	<xacro:property name="imu_offset_x" value="0.127"/>
+	<xacro:property name="imu_offset_y" value="-0.129"/>
+	<xacro:property name="imu_offset_z" value="0.212"/>
 	<xacro:property name="front_rgbd_camera_offset_x" value="0.35850"/>
 	<xacro:property name="front_rgbd_camera_offset_y" value="0.0"/>

File: summit_xl_description/urdf/bases/summit_xl_base.gazebo.xacro (robot description, xacro)
@@ -1,4 +1,4 @@
 <?xml version="1.0"?>
-<robot xmlns:xacro="http://www.ros.org/wiki/xacro">
+<robot xmlns:xacro="http://wiki.ros.org/xacro">
   <!-- ros control plugin -->
   <xacro:macro name="ros_control">

File: summit_xl_description/urdf/bases/summit_xl_base.urdf.xacro (robot description, xacro)
@@ -1,4 +1,4 @@
 <?xml version="1.0"?>
-<robot name="summit_xl" xmlns:xacro="http://www.ros.org/wiki/xacro">
+<robot name="summit_xl" xmlns:xacro="http://wiki.ros.org/xacro">
   <xacro:include filename="$(find summit_xl_description)/urdf/bases/summit_xl_base.gazebo.xacro" />
   <xacro:macro name="summit_xl_base" params="prefix publish_bf hq">

File: summit_xl_description/urdf/bases/summit_xls_base.urdf.xacro (robot description, xacro)
@@ -1,4 +1,4 @@
 <?xml version="1.0"?>
-<robot name="summit_xl" xmlns:xacro="http://www.ros.org/wiki/xacro">
+<robot name="summit_xl" xmlns:xacro="http://wiki.ros.org/xacro">
   <xacro:include filename="$(find summit_xl_description)/urdf/bases/summit_xl_base.gazebo.xacro" />
   <xacro:macro name="summit_xls_base" params="prefix publish_bf hq">

File: summit_xl_description/urdf/wheels/omni_wheel.urdf.xacro (robot description, xacro)
@@ -1,4 +1,4 @@
 <?xml version="1.0"?>
-<robot name="wheel" xmlns:xacro="http://www.ros.org/wiki/xacro">
+<robot name="wheel" xmlns:xacro="http://wiki.ros.org/xacro">
   <xacro:property name="M_PI" value="3.1415926535897931" />
   <!-- Wheels -->

File: summit_xl_description/urdf/wheels/rubber_wheel.urdf.xacro (robot description, xacro)
@@ -1,4 +1,4 @@
 <?xml version="1.0"?>
-<robot name="wheel" xmlns:xacro="http://www.ros.org/wiki/xacro">
+<robot name="wheel" xmlns:xacro="http://wiki.ros.org/xacro">
   <xacro:property name="M_PI" value="3.1415926535897931" />
   <!-- Wheels -->

Commit message: Add ros planar move plugin for skid simulation

File: summit_xl_description/robots/summit_xl_std.urdf.xacro (robot description, xacro)
@@ -80,7 +80,12 @@
    <!-- Gazebo ros control pluggins -->
    <xacro:ros_control/>
-   <xacro:if value="$(arg ros_planar_move_plugin)">
-	   <xacro:omni_steering prefix="$(arg prefix)" publish_tf="false"/>
-   </xacro:if>
+	<xacro:if value="$(arg ros_planar_move_plugin)">
+		<xacro:if value="$(arg omni_wheels)">
+			<xacro:omni_steering prefix="$(arg prefix)" publish_tf="false"/>
+		</xacro:if>
+		<xacro:unless value="$(arg omni_wheels)">
+			<xacro:skid_steering prefix="$(arg prefix)" publish_tf="false"/>
+		</xacro:unless>
+	</xacro:if>
    <xacro:summit_xl prefix="$(arg prefix)" publish_bf="true" hq="true"/>
 </robot>

File: summit_xl_description/urdf/bases/summit_xl_base.gazebo.xacro (robot description, xacro)
@@ -47,4 +47,17 @@
 	  </gazebo>
   </xacro:macro>
+  	<xacro:macro name="skid_steering" params="prefix publish_tf">
+		<gazebo>
+			<plugin name="skid_steering" filename="libgazebo_ros_planar_move.so">
+			<commandTopic>robotnik_base_control/cmd_vel</commandTopic>
+			<odometryTopic>robotnik_base_control/odom</odometryTopic>
+			<odometryFrame>${prefix}odom</odometryFrame>
+			<odometryRate>50.0</odometryRate>
+			<robotBaseFrame>${prefix}base_footprint</robotBaseFrame>
+			<publishTF>${publish_tf}</publishTF>
+			<enableYAxis>false</enableYAxis>
+			</plugin>
+		</gazebo>
+  	</xacro:macro>
   <xacro:macro name="ros_force_based_move" params="publish_tf prefix">
 	  <gazebo>

Commit message: summit_xl_descritpion: Add ros_planar_move_plugin_force_based option for summit_xl_std

File: summit_xl_description/robots/summit_xl_std.urdf.xacro (robot description, xacro)
@@ -21,4 +21,5 @@
 	<xacro:arg name="prefix" default="summit_xl_"/>
 	<xacro:arg name="ros_planar_move_plugin" default="false"/>
+	<xacro:arg name="ros_planar_move_plugin_force_based" default="false"/>
 	<xacro:arg name="omni_wheels" default="false"/>
 	<xacro:arg name="gpu" default="false"/>
@@ -85,8 +86,8 @@
 	<xacro:if value="$(arg ros_planar_move_plugin)">
 		<xacro:if value="$(arg omni_wheels)">
-			<xacro:omni_steering prefix="$(arg prefix)" publish_tf="true"/>
+			<xacro:omni_steering prefix="$(arg prefix)" publish_tf="true" force_based="$(arg ros_planar_move_plugin_force_based)"/>
 		</xacro:if>
 		<xacro:unless value="$(arg omni_wheels)">
-			<xacro:skid_steering prefix="$(arg prefix)" publish_tf="true"/>
+			<xacro:skid_steering prefix="$(arg prefix)" publish_tf="true" force_based="$(arg ros_planar_move_plugin_force_based)"/>
 		</xacro:unless>
 	</xacro:if>

File: summit_xl_description/urdf/bases/summit_xl_base.gazebo.xacro (robot description, xacro)
@@ -34,29 +34,65 @@
     </gazebo>
   </xacro:macro>
-  <xacro:macro name="omni_steering" params="prefix publish_tf">
-		<gazebo>
-	    <plugin name="omni_steering" filename="libgazebo_ros_planar_move.so">
-	      <commandTopic>robotnik_base_control/cmd_vel</commandTopic>
-	      <odometryTopic>robotnik_base_control/odom</odometryTopic>
-	      <odometryFrame>${prefix}odom</odometryFrame>
-	      <odometryRate>50.0</odometryRate>
-	      <robotBaseFrame>${prefix}base_footprint</robotBaseFrame>
-	      <publishTF>${publish_tf}</publishTF>
-	      <enableYAxis>true</enableYAxis>
-	    </plugin>
-	  </gazebo>
+  <xacro:macro name="omni_steering" params="prefix publish_tf force_based">
+		<xacro:if value="${force_based}">
+			<gazebo>
+				<plugin name="ros_force_based_move" filename="librobotnik_force_based_move.so">
+					<commandTopic>robotnik_base_control/cmd_vel</commandTopic>
+					<odometryTopic>robotnik_base_control/odom</odometryTopic>
+					<odometryFrame>${prefix}odom</odometryFrame>
+					<yaw_velocity_p_gain>10000.0</yaw_velocity_p_gain>
+					<x_velocity_p_gain>10000.0</x_velocity_p_gain>
+					<y_velocity_p_gain>10000.0</y_velocity_p_gain>
+					<robotBaseFrame>${prefix}base_footprint</robotBaseFrame>
+					<commandWatchdog>1</commandWatchdog>
+					<odometryRate>50.0</odometryRate>
+					<publishOdometryTf>${publish_tf}</publishOdometryTf>
+				</plugin>
+			</gazebo>
+		</xacro:if>
+		<xacro:unless value="${force_based}">
+			<gazebo>
+				<plugin name="omni_steering" filename="libgazebo_ros_planar_move.so">
+				<commandTopic>robotnik_base_control/cmd_vel</commandTopic>
+				<odometryTopic>robotnik_base_control/odom</odometryTopic>
+				<odometryFrame>${prefix}odom</odometryFrame>
+				<odometryRate>50.0</odometryRate>
+				<robotBaseFrame>${prefix}base_footprint</robotBaseFrame>
+				<publishTF>${publish_tf}</publishTF>
+				<enableYAxis>true</enableYAxis>
+				</plugin>
+			</gazebo>
+		</xacro:unless>
   </xacro:macro>
-  	<xacro:macro name="skid_steering" params="prefix publish_tf">
-		<gazebo>
-			<plugin name="skid_steering" filename="libgazebo_ros_planar_move.so">
-			<commandTopic>robotnik_base_control/cmd_vel</commandTopic>
-			<odometryTopic>robotnik_base_control/odom</odometryTopic>
-			<odometryFrame>${prefix}odom</odometryFrame>
-			<odometryRate>50.0</odometryRate>
-			<robotBaseFrame>${prefix}base_footprint</robotBaseFrame>
-			<publishTF>${publish_tf}</publishTF>
-			<enableYAxis>false</enableYAxis>
-			</plugin>
-		</gazebo>
+  	<xacro:macro name="skid_steering" params="prefix publish_tf force_based">
+		<xacro:if value="${force_based}">
+			<gazebo>
+				<plugin name="ros_force_based_move" filename="librobotnik_force_based_move.so">
+					<commandTopic>robotnik_base_control/cmd_vel</commandTopic>
+					<odometryTopic>robotnik_base_control/odom</odometryTopic>
+					<odometryFrame>${prefix}odom</odometryFrame>
+					<yaw_velocity_p_gain>10000.0</yaw_velocity_p_gain>
+					<x_velocity_p_gain>10000.0</x_velocity_p_gain>
+					<y_velocity_p_gain>0.0</y_velocity_p_gain>
+					<robotBaseFrame>${prefix}base_footprint</robotBaseFrame>
+					<commandWatchdog>1</commandWatchdog>
+					<odometryRate>50.0</odometryRate>
+					<publishOdometryTf>${publish_tf}</publishOdometryTf>
+				</plugin>
+			</gazebo>
+		</xacro:if>
+	  	<xacro:unless value="${force_based}">
+			<gazebo>
+				<plugin name="skid_steering" filename="libgazebo_ros_planar_move.so">
+				<commandTopic>robotnik_base_control/cmd_vel</commandTopic>
+				<odometryTopic>robotnik_base_control/odom</odometryTopic>
+				<odometryFrame>${prefix}odom</odometryFrame>
+				<odometryRate>50.0</odometryRate>
+				<robotBaseFrame>${prefix}base_footprint</robotBaseFrame>
+				<publishTF>${publish_tf}</publishTF>
+				<enableYAxis>false</enableYAxis>
+				</plugin>
+			</gazebo>
+		</xacro:unless>
   	</xacro:macro>
   <xacro:macro name="ros_force_based_move" params="publish_tf prefix">

Commit message: Fixing aresibo urdf

File: summit_xl_description/robots/summit_xl_std.urdf.xacro (robot description, xacro)
@@ -62,10 +62,10 @@
         <!-- IMU -->
 		<xacro:sensor_imu prefix="$(arg prefix)imu" parent="$(arg prefix)base_link">
-			<origin xyz="-0.18 0.0 0.170" rpy="0 0 0"/>
+			<origin xyz="-0.0365 0.132 0.161" rpy="0 0 0"/>
 		</xacro:sensor_imu>
-		<!-- 2d laser -->
-		<xacro:sensor_hokuyo_ust10lx prefix="$(arg prefix)front_laser" parent="$(arg prefix)base_link" prefix_topic="front_laser" gpu="$(arg gpu)">
-			<origin xyz="0.0 0.0 0.33" rpy="0 0 0"/>
-		</xacro:sensor_hokuyo_ust10lx>
+		<!-- Lidar -->
+		<xacro:sensor_rslidar_16 prefix="$(arg prefix)rslidar_16" parent="$(arg prefix)base_link" prefix_topic="rslidar_16" gpu="$(arg gpu)">
+			<origin xyz="-0.018 0.0 0.369" rpy="0 0 0"/>
+		</xacro:sensor_rslidar_16>
 		<!-- ptz camera -->
 		<xacro:sensor_axis prefix="$(arg prefix)front_ptz_camera" parent="$(arg prefix)base_link">
@@ -74,9 +74,9 @@
 	  <!-- RGBD -->
 	  <xacro:sensor_orbbec_astra prefix="$(arg prefix)front_rgbd_camera" parent="$(arg prefix)base_link" prefix_topic="front_rgbd_camera">
-			<origin xyz="0.324 0.012 0.172" rpy="0 0 0"/>
+			<origin xyz="0.028 0.0 0.471" rpy="0 0 0"/>
 		</xacro:sensor_orbbec_astra>
 	  <!-- GPS -->
 	  <xacro:sensor_gps prefix="$(arg prefix)gps" parent="$(arg prefix)base_link" gps_latitude="$(arg gps_latitude)" gps_longitude="$(arg gps_longitude)">
-			<origin xyz="-0.22 0 0.275" rpy="0 0 0"/>
+			<origin xyz="-0.235 0 0.647" rpy="0 0 0"/>
 		</xacro:sensor_gps>
    </xacro:macro>

Commit message: Update std_model: hokuyo ust20, gps_with mast

File: summit_xl_description/robots/summit_xl_std.urdf.xacro (robot description, xacro)
@@ -65,7 +65,7 @@
 		</xacro:sensor_imu>
 		<!-- 2d laser -->
-		<xacro:sensor_hokuyo_ust10lx prefix="$(arg prefix)front_laser" parent="$(arg prefix)base_link" prefix_topic="front_laser" gpu="$(arg gpu)">
-			<origin xyz="0.0 0.0 0.33" rpy="0 0 0"/>
-		</xacro:sensor_hokuyo_ust10lx>
+		<xacro:sensor_hokuyo_ust20lx prefix="$(arg prefix)front_laser" parent="$(arg prefix)base_link" prefix_topic="front_laser" gpu="$(arg gpu)">
+			<origin xyz="0.0 0.0 0.2726" rpy="0 0 0"/>
+		</xacro:sensor_hokuyo_ust20lx>
 		<!-- ptz camera -->
 		<xacro:sensor_axis prefix="$(arg prefix)front_ptz_camera" parent="$(arg prefix)base_link">
@@ -77,7 +77,7 @@
 		</xacro:sensor_orbbec_astra>
 	  <!-- GPS -->
-	  <xacro:sensor_gps prefix="$(arg prefix)gps" parent="$(arg prefix)base_link" gps_latitude="$(arg gps_latitude)" gps_longitude="$(arg gps_longitude)">
+	  <xacro:sensor_gps_with_mast prefix="$(arg prefix)gps" parent="$(arg prefix)base_link" gps_latitude="$(arg gps_latitude)" gps_longitude="$(arg gps_longitude)">
 			<origin xyz="-0.22 0 0.275" rpy="0 0 0"/>
-		</xacro:sensor_gps>
+		</xacro:sensor_gps_with_mast>
    </xacro:macro>
    <!-- Gazebo ros control pluggins -->

Commit message: Add mastil teltonika urdf and mesh for antenna and update summit_xl_std.urdf.xacro antenna position

File: summit_xl_description/robots/summit_xl_std.urdf.xacro (robot description, xacro)
@@ -12,4 +12,6 @@
 	<!-- Import all available sensors -->
 	<xacro:include filename="$(find robotnik_sensors)/urdf/all_sensors.urdf.xacro" />
+	<!-- Import antenna -->
+	<xacro:include filename="$(find summit_xl_description)/urdf/structures/structure_teltonika.urdf.xacro" />
 	<xacro:property name="PI" value="3.1415926535897931"/>
 	<!-- Wheel parameters -->
@@ -65,12 +67,12 @@
 			<origin xyz="-0.18 0.0 0.170" rpy="0 0 0"/>
 		</xacro:sensor_imu>
-		<!-- 2d laser -->
-		<xacro:sensor_hokuyo_ust20lx prefix="$(arg prefix)front_laser" parent="$(arg prefix)base_link" prefix_topic="front_laser" gpu="$(arg gpu)">
-			<origin xyz="0.0 0.0 0.2726" rpy="0 0 0"/>
-		</xacro:sensor_hokuyo_ust20lx>
+		<!-- 3d laser -->
+		<xacro:sensor_rs_helios_16p prefix="$(arg prefix)top_3d_laser" parent="$(arg prefix)base_link" gpu="$(arg gpu)">
+			<origin xyz="-0.11808 0.0 0.38509" rpy="0 0 0"/>
+		</xacro:sensor_rs_helios_16p>
 		<!-- ptz camera -->
-		<xacro:sensor_axis prefix="$(arg prefix)front_ptz_camera" parent="$(arg prefix)base_link">
+		<!--xacro:sensor_axis prefix="$(arg prefix)front_ptz_camera" parent="$(arg prefix)base_link">
 			<origin xyz="0.19 0 0.26" rpy="0 ${15*PI/180} 0"/>
-		</xacro:sensor_axis>
+		</xacro:sensor_axis-->
 	  <!-- RGBD -->
 	  <xacro:sensor_orbbec_astra prefix="$(arg prefix)front_rgbd_camera" parent="$(arg prefix)base_link" prefix_topic="front_rgbd_camera">
@@ -79,6 +81,10 @@
 	  <!-- GPS -->
 	  <xacro:sensor_gps_with_mast prefix="$(arg prefix)gps" parent="$(arg prefix)base_link" gps_latitude="$(arg gps_latitude)" gps_longitude="$(arg gps_longitude)">
-			<origin xyz="-0.22 0 0.275" rpy="0 0 0"/>
+			<origin xyz="-0.22528 0.095 0.275" rpy="0 0 0"/>
 		</xacro:sensor_gps_with_mast>
+	  <!--Antenna-->
+	  	<xacro:structure_mastil_teltonika prefix="$(arg prefix)antenna" parent="$(arg prefix)base_link">
+			<origin xyz="-0.22528 -0.095 0.23325" rpy="0 0 0"/>
+		</xacro:structure_mastil_teltonika>
    </xacro:macro>
    <!-- Gazebo ros control pluggins -->

Commit message: Change the position of the axis camera on SummitXL std

File: summit_xl_description/robots/summit_xl_std.urdf.xacro (robot description, xacro)
@@ -71,5 +71,5 @@
 		<!-- ptz camera -->
 		<xacro:sensor_axis prefix="$(arg prefix)front_ptz_camera" parent="$(arg prefix)base_link">
-			<origin xyz="0.19 0 0.26" rpy="0 ${15*PI/180} 0"/>
+			<origin xyz="0.185 0 0.1967" rpy="0 ${15*PI/180} 0"/>
 		</xacro:sensor_axis>
 	  <!-- RGBD -->
