Commit message: Add prefix

File: summit_xl_description/robots/summit_xl_std.urdf.xacro (robot description, xacro)
@@ -8,4 +8,5 @@
   <xacro:include filename="$(find summit_xl_description)/urdf/wheels/rubber_wheel.urdf.xacro"/>
   <xacro:include filename="$(find summit_xl_description)/urdf/wheels/omni_wheel.urdf.xacro"/>
+  <xacro:include filename="$(find summit_xl_description)/urdf/structures/structure_gps.urdf.xacro"/>
   <!-- Import all available sensors -->
   <xacro:include filename="$(find robotnik_sensors)/urdf/all_sensors.urdf.xacro"/>
@@ -22,4 +23,5 @@
   <xacro:property name="hq" value="true"/>
   <xacro:arg name="robot_id" default="robot"/>
+  <xacro:arg name="prefix" default=""/>
   <xacro:arg name="robot_ns" default="$(arg robot_id)"/>
   <xacro:arg name="omni_wheels" default="false"/>
@@ -28,45 +30,45 @@
   <!-- *************** -->
   <!-- Summit XL -->
-  <xacro:summit_xl_base publish_bf="true" hq="${hq}"/>
+  <xacro:summit_xl_base prefix="$(arg prefix)" publish_bf="true" hq="${hq}"/>
   <!--xacro:gazebo_colors /-->
   <!-- WHEELS -->
   <xacro:unless value="$(arg omni_wheels)">
-    <xacro:rubber_wheel prefix="front_right_" parent="base_link" reflect="false" hq="${hq}">
+    <xacro:rubber_wheel prefix="front_right_" parent="$(arg prefix)base_link" reflect="false" hq="${hq}">
       <origin xyz="${wheel_offset_x} -${wheel_offset_y} ${wheel_offset_z}" rpy="0 0 0"/>
     </xacro:rubber_wheel>
-    <xacro:rubber_wheel prefix="front_left_" parent="base_link" reflect="true" hq="${hq}">
+    <xacro:rubber_wheel prefix="front_left_" parent="$(arg prefix)base_link" reflect="true" hq="${hq}">
       <origin xyz="${wheel_offset_x} ${wheel_offset_y} ${wheel_offset_z}" rpy="0 0 0"/>
     </xacro:rubber_wheel>
-    <xacro:rubber_wheel prefix="rear_left_" parent="base_link" reflect="true" hq="${hq}">
+    <xacro:rubber_wheel prefix="rear_left_" parent="$(arg prefix)base_link" reflect="true" hq="${hq}">
       <origin xyz="-${wheel_offset_x} ${wheel_offset_y} ${wheel_offset_z}" rpy="0 0 0"/>
     </xacro:rubber_wheel>
-    <xacro:rubber_wheel prefix="rear_right_" parent="base_link" reflect="false" hq="${hq}">
+    <xacro:rubber_wheel prefix="rear_right_" parent="$(arg prefix)base_link" reflect="false" hq="${hq}">
       <origin xyz="-${wheel_offset_x} -${wheel_offset_y} ${wheel_offset_z}" rpy="0 0 0"/>
     </xacro:rubber_wheel>
   </xacro:unless>
   <xacro:if value="$(arg omni_wheels)">
-    <xacro:omni_wheel prefix="front_right_" parent="base_link" reflect="false" hq="${hq}">
+    <xacro:omni_wheel prefix="front_right_" parent="$(arg prefix)base_link" reflect="false" hq="${hq}">
       <origin xyz="${wheel_offset_x} -${wheel_offset_y} ${wheel_offset_z}" rpy="0 0 0"/>
     </xacro:omni_wheel>
-    <xacro:omni_wheel prefix="front_left_" parent="base_link" reflect="true" hq="${hq}">
+    <xacro:omni_wheel prefix="front_left_" parent="$(arg prefix)base_link" reflect="true" hq="${hq}">
       <origin xyz="${wheel_offset_x} ${wheel_offset_y} ${wheel_offset_z}" rpy="0 0 0"/>
     </xacro:omni_wheel>
-    <xacro:omni_wheel prefix="back_left_" parent="base_link" reflect="true" hq="${hq}">
+    <xacro:omni_wheel prefix="back_left_" parent="$(arg prefix)base_link" reflect="true" hq="${hq}">
       <origin xyz="-${wheel_offset_x} ${wheel_offset_y} ${wheel_offset_z}" rpy="0 0 0"/>
     </xacro:omni_wheel>
-    <xacro:omni_wheel prefix="back_right_" parent="base_link" reflect="false" hq="${hq}">
+    <xacro:omni_wheel prefix="back_right_" parent="$(arg prefix)base_link" reflect="false" hq="${hq}">
       <origin xyz="-${wheel_offset_x} -${wheel_offset_y} ${wheel_offset_z}" rpy="0 0 0"/>
     </xacro:omni_wheel>
   </xacro:if>
   <!-- SENSORS -->
-  <xacro:sensor_imu_hector ns="$(arg robot_ns)" prefix="imu" parent="base_link">
-    <origin xyz="-0.18 0.0 0.170" rpy="0 0 0"/>
-  </xacro:sensor_imu_hector>
-  <xacro:sensor_hokuyo_ust20lx ns="$(arg robot_ns)" prefix="front_laser" parent="base_link">
-    <origin xyz="0.0 0.0 0.33" rpy="0 0 0"/>
-  </xacro:sensor_hokuyo_ust20lx>
-  <xacro:sensor_orbbec_astra ns="$(arg robot_ns)" prefix="front_rgbd_camera" parent="base_link">
-    <origin xyz="0.324 0.012 0.172" rpy="0 0 0"/>
-  </xacro:sensor_orbbec_astra>
+  <xacro:sensor_robosense_helios node_namespace="$(arg robot_ns)" frame_prefix="$(arg prefix)front_laser_" parent="$(arg prefix)base_link">
+      <origin xyz="-0.11808 0.0 0.38509" rpy="0 0 0"/>
+  </xacro:sensor_robosense_helios>
+  <xacro:sensor_stereolabs_zed2 node_namespace="$(arg robot_ns)" frame_prefix="$(arg prefix)front_camera_" parent="$(arg prefix)base_link">
+      <origin xyz="0.324 0.012 0.172" rpy="0 0 0"/>
+  </xacro:sensor_stereolabs_zed2>
+  <xacro:structure_mastil_gps prefix="$(arg prefix)gps" parent="$(arg prefix)base_link">
+    <origin xyz="-0.24 0.095 0.30" rpy="0 0 0"/>
+  </xacro:structure_mastil_gps>
   <!-- Gazebo ros control plugins -->
   <xacro:arg name="config_controllers" default=""/>

File: summit_xl_description/urdf/bases/summit_xl_base.urdf.xacro (robot description, xacro)
@@ -1,5 +1,5 @@
 <?xml version="1.0"?>
 <robot name="summit_xl" xmlns:xacro="http://wiki.ros.org/xacro">
-  <xacro:macro name="summit_xl_base" params="publish_bf hq">
+  <xacro:macro name="summit_xl_base" params="prefix publish_bf hq">
     <!-- Robot mechanical and motor parameters -->
     <xacro:property name="PI" value="3.1415926535897931"/>
@@ -7,13 +7,13 @@
     <!-- BASE FOOTPRINT -->
     <xacro:if value="${publish_bf}">
-      <link name="base_footprint"/>
+      <link name="${prefix}base_footprint"/>
       <joint name="base_footprint_joint" type="fixed">
         <origin xyz="0 0 ${wheel_radius}" rpy="0 0 0" />
-        <parent link="base_footprint"/>
-        <child link="base_link" />
+        <parent link="${prefix}base_footprint"/>
+        <child link="${prefix}base_link" />
       </joint>
     </xacro:if>
     <!-- BASE_LINK -->
-    <link name="base_link">
+    <link name="${prefix}base_link">
       <inertial>
         <mass value="25.0" />
@@ -40,10 +40,10 @@
     </link>
     <!-- DOCKING -->
-    <joint name="base_docking_joint" type="fixed">
+    <joint name="${prefix}base_docking_joint" type="fixed">
       <origin xyz="0.284 0.012 0.068" rpy="0 0 0 " />
-      <parent link="base_link"/>
-      <child link="base_docking_contact_link" />
+      <parent link="${prefix}base_link"/>
+      <child link="${prefix}base_docking_contact_link" />
     </joint>
-    <link name="base_docking_contact_link" />
+    <link name="${prefix}base_docking_contact_link" />
   </xacro:macro>
 </robot>

Commit message: [ROS2 Humble] Add testing xacro files. (#21)
* Ros2 humble simulation

* Added tests

* Add prefix

File: summit_xl_description/robots/summit_xl_std.urdf.xacro (robot description, xacro)
@@ -1,92 +1,77 @@
 <?xml version="1.0"?>
 <robot name="summit_xl" xmlns:xacro="http://wiki.ros.org/xacro">
-	<!-- ***************** -->
-	<!-- Imported elements -->
-	<!-- ***************** -->
-	<!-- First we import all posible elements defined in the urdf.xacro files. All these elements are defined as macro:xacros -->
-	<!-- Import summit XL base elements -->
-	<xacro:include filename="$(find summit_xl_description)/urdf/bases/summit_xl_base.urdf.xacro" />
-	<!-- Import summit XL wheels -->
-	<xacro:include filename="$(find summit_xl_description)/urdf/wheels/rubber_wheel.urdf.xacro" />
-  <xacro:include filename="$(find summit_xl_description)/urdf/wheels/omni_wheel.urdf.xacro" />
-	<!-- Import all available sensors -->
-	<xacro:include filename="$(find robotnik_sensors)/urdf/all_sensors.urdf.xacro" />
-	<xacro:property name="PI" value="3.1415926535897931"/>
-	<!-- Wheel parameters -->
-	<xacro:property name="wheel_offset_x" value="0.229" />    <!-- x,y,z in translation from base_link to the center of the wheel -->
-	<xacro:property name="wheel_offset_y" value="0.235" />
-	<xacro:property name="wheel_offset_z" value="0.0" />
-	<!-- Flag to select the high or low quality model -->
-	<xacro:property name="hq" value="true" />
-	<xacro:arg name="prefix" default="summit_xl_"/>
-	<xacro:arg name="ros_planar_move_plugin" default="false"/>
-	<xacro:arg name="omni_wheels" default="false"/>
-	<xacro:arg name="gpu" default="false"/>
-    <xacro:macro name="summit_xl" params="prefix publish_bf hq">
-		<!-- *************** -->
-		<!-- Robots Elements -->
-		<!-- *************** -->
-		<!-- Here we create the robot elements using the xacro:macros imported at the beggining of this file -->
-		<!-- Summit XL base -->
-		<xacro:summit_xl_base prefix="$(arg prefix)" publish_bf="true" hq="${hq}" />
-    <xacro:unless value="$(arg omni_wheels)">
-  		<xacro:rubber_wheel prefix="$(arg prefix)front_right" parent="$(arg prefix)base_link" reflect="false" hq="${hq}">
-  			<origin xyz="${wheel_offset_x} -${wheel_offset_y} ${wheel_offset_z}" rpy="0 0 0"/>
-  		</xacro:rubber_wheel>
-  		<xacro:rubber_wheel prefix="$(arg prefix)front_left" parent="$(arg prefix)base_link" reflect="true" hq="${hq}">
-  			<origin xyz="${wheel_offset_x} ${wheel_offset_y} ${wheel_offset_z}" rpy="0 0 0"/>
-  		</xacro:rubber_wheel>
-  		<xacro:rubber_wheel prefix="$(arg prefix)back_left" parent="$(arg prefix)base_link" reflect="true" hq="${hq}">
-  			<origin xyz="-${wheel_offset_x} ${wheel_offset_y} ${wheel_offset_z}" rpy="0 0 0"/>
-  		</xacro:rubber_wheel>
-  		<xacro:rubber_wheel prefix="$(arg prefix)back_right" parent="$(arg prefix)base_link" reflect="false" hq="${hq}">
-  			<origin xyz="-${wheel_offset_x} -${wheel_offset_y} ${wheel_offset_z}" rpy="0 0 0"/>
-  		</xacro:rubber_wheel>
-    </xacro:unless>
-    <xacro:if value="$(arg omni_wheels)">
-  		<xacro:omni_wheel prefix="$(arg prefix)front_right" parent="$(arg prefix)base_link" reflect="false" hq="${hq}">
-  			<origin xyz="${wheel_offset_x} -${wheel_offset_y} ${wheel_offset_z}" rpy="0 0 0"/>
-  		</xacro:omni_wheel>
-  		<xacro:omni_wheel prefix="$(arg prefix)front_left" parent="$(arg prefix)base_link" reflect="true" hq="${hq}">
-  			<origin xyz="${wheel_offset_x} ${wheel_offset_y} ${wheel_offset_z}" rpy="0 0 0"/>
-  		</xacro:omni_wheel>
-  		<xacro:omni_wheel prefix="$(arg prefix)back_left" parent="$(arg prefix)base_link" reflect="true" hq="${hq}">
-  			<origin xyz="-${wheel_offset_x} ${wheel_offset_y} ${wheel_offset_z}" rpy="0 0 0"/>
-  		</xacro:omni_wheel>
-  		<xacro:omni_wheel prefix="$(arg prefix)back_right" parent="$(arg prefix)base_link" reflect="false" hq="${hq}">
-  			<origin xyz="-${wheel_offset_x} -${wheel_offset_y} ${wheel_offset_z}" rpy="0 0 0"/>
-  		</xacro:omni_wheel>
-    </xacro:if>
-        <!-- IMU -->
-		<xacro:sensor_imu prefix="$(arg prefix)imu" parent="$(arg prefix)base_link">
-			<origin xyz="-0.18 0.0 0.170" rpy="0 0 0"/>
-		</xacro:sensor_imu>
-		<!-- 2d laser -->
-		<xacro:sensor_hokuyo_ust10lx prefix="$(arg prefix)front_laser" parent="$(arg prefix)base_link" prefix_topic="front_laser" gpu="$(arg gpu)">
-			<origin xyz="0.0 0.0 0.33" rpy="0 0 0"/>
-		</xacro:sensor_hokuyo_ust10lx>
-		<!-- ptz camera -->
-		<xacro:sensor_axis prefix="$(arg prefix)front_ptz_camera" parent="$(arg prefix)base_link">
-			<origin xyz="0.19 0 0.26" rpy="0 ${15*PI/180} 0"/>
-		</xacro:sensor_axis>
-	  <!-- RGBD -->
-	  <xacro:sensor_orbbec_astra prefix="$(arg prefix)front_rgbd_camera" parent="$(arg prefix)base_link" prefix_topic="front_rgbd_camera">
-			<origin xyz="0.324 0.012 0.172" rpy="0 0 0"/>
-		</xacro:sensor_orbbec_astra>
-	  <!-- GPS -->
-	  <xacro:sensor_gps prefix="$(arg prefix)gps" parent="$(arg prefix)base_link" gps_latitude="$(arg gps_latitude)" gps_longitude="$(arg gps_longitude)">
-			<origin xyz="-0.22 0 0.275" rpy="0 0 0"/>
-		</xacro:sensor_gps>
-   </xacro:macro>
-   <!-- Gazebo ros control pluggins -->
-   <xacro:ros_control/>
-	<xacro:if value="$(arg ros_planar_move_plugin)">
-		<xacro:if value="$(arg omni_wheels)">
-			<xacro:omni_steering prefix="$(arg prefix)" publish_tf="true"/>
-		</xacro:if>
-		<xacro:unless value="$(arg omni_wheels)">
-			<xacro:skid_steering prefix="$(arg prefix)" publish_tf="true"/>
-		</xacro:unless>
-	</xacro:if>
-   <xacro:summit_xl prefix="$(arg prefix)" publish_bf="true" hq="true"/>
+  <!-- ***************** -->
+  <!-- Imported elements -->
+  <!-- ***************** -->
+  <!-- Import RB1 base elements (base + wheels) -->
+  <xacro:include filename="$(find summit_xl_description)/urdf/bases/summit_xl_base.urdf.xacro"/>
+  <xacro:include filename="$(find summit_xl_description)/urdf/wheels/rubber_wheel.urdf.xacro"/>
+  <xacro:include filename="$(find summit_xl_description)/urdf/wheels/omni_wheel.urdf.xacro"/>
+  <xacro:include filename="$(find summit_xl_description)/urdf/structures/structure_gps.urdf.xacro"/>
+  <!-- Import all available sensors -->
+  <xacro:include filename="$(find robotnik_sensors)/urdf/all_sensors.urdf.xacro"/>
+  <!-- ***************** -->
+  <!-- Global parameters -->
+  <!-- ***************** -->
+  <xacro:property name="PI" value="3.1415926535897931"/>
+  <!-- Wheel parameters -->
+  <!-- x,y,z in translation from base_link to the center of the wheel -->
+  <xacro:property name="wheel_offset_x" value="0.218"/>
+  <xacro:property name="wheel_offset_y" value="0.218"/>
+  <xacro:property name="wheel_offset_z" value="0.0512"/>
+  <!-- Flag to select the high or low quality model -->
+  <xacro:property name="hq" value="true"/>
+  <xacro:arg name="robot_id" default="robot"/>
+  <xacro:arg name="prefix" default=""/>
+  <xacro:arg name="robot_ns" default="$(arg robot_id)"/>
+  <xacro:arg name="omni_wheels" default="false"/>
+  <!-- *************** -->
+  <!-- Robots Elements -->
+  <!-- *************** -->
+  <!-- Summit XL -->
+  <xacro:summit_xl_base prefix="$(arg prefix)" publish_bf="true" hq="${hq}"/>
+  <!--xacro:gazebo_colors /-->
+  <!-- WHEELS -->
+  <xacro:unless value="$(arg omni_wheels)">
+    <xacro:rubber_wheel prefix="front_right_" parent="$(arg prefix)base_link" reflect="false" hq="${hq}">
+      <origin xyz="${wheel_offset_x} -${wheel_offset_y} ${wheel_offset_z}" rpy="0 0 0"/>
+    </xacro:rubber_wheel>
+    <xacro:rubber_wheel prefix="front_left_" parent="$(arg prefix)base_link" reflect="true" hq="${hq}">
+      <origin xyz="${wheel_offset_x} ${wheel_offset_y} ${wheel_offset_z}" rpy="0 0 0"/>
+    </xacro:rubber_wheel>
+    <xacro:rubber_wheel prefix="rear_left_" parent="$(arg prefix)base_link" reflect="true" hq="${hq}">
+      <origin xyz="-${wheel_offset_x} ${wheel_offset_y} ${wheel_offset_z}" rpy="0 0 0"/>
+    </xacro:rubber_wheel>
+    <xacro:rubber_wheel prefix="rear_right_" parent="$(arg prefix)base_link" reflect="false" hq="${hq}">
+      <origin xyz="-${wheel_offset_x} -${wheel_offset_y} ${wheel_offset_z}" rpy="0 0 0"/>
+    </xacro:rubber_wheel>
+  </xacro:unless>
+  <xacro:if value="$(arg omni_wheels)">
+    <xacro:omni_wheel prefix="front_right_" parent="$(arg prefix)base_link" reflect="false" hq="${hq}">
+      <origin xyz="${wheel_offset_x} -${wheel_offset_y} ${wheel_offset_z}" rpy="0 0 0"/>
+    </xacro:omni_wheel>
+    <xacro:omni_wheel prefix="front_left_" parent="$(arg prefix)base_link" reflect="true" hq="${hq}">
+      <origin xyz="${wheel_offset_x} ${wheel_offset_y} ${wheel_offset_z}" rpy="0 0 0"/>
+    </xacro:omni_wheel>
+    <xacro:omni_wheel prefix="back_left_" parent="$(arg prefix)base_link" reflect="true" hq="${hq}">
+      <origin xyz="-${wheel_offset_x} ${wheel_offset_y} ${wheel_offset_z}" rpy="0 0 0"/>
+    </xacro:omni_wheel>
+    <xacro:omni_wheel prefix="back_right_" parent="$(arg prefix)base_link" reflect="false" hq="${hq}">
+      <origin xyz="-${wheel_offset_x} -${wheel_offset_y} ${wheel_offset_z}" rpy="0 0 0"/>
+    </xacro:omni_wheel>
+  </xacro:if>
+  <!-- SENSORS -->
+  <xacro:sensor_robosense_helios node_namespace="$(arg robot_ns)" frame_prefix="$(arg prefix)front_laser_" parent="$(arg prefix)base_link">
+      <origin xyz="-0.11808 0.0 0.38509" rpy="0 0 0"/>
+  </xacro:sensor_robosense_helios>
+  <xacro:sensor_stereolabs_zed2 node_namespace="$(arg robot_ns)" frame_prefix="$(arg prefix)front_camera_" parent="$(arg prefix)base_link">
+      <origin xyz="0.324 0.012 0.172" rpy="0 0 0"/>
+  </xacro:sensor_stereolabs_zed2>
+  <xacro:structure_mastil_gps prefix="$(arg prefix)gps" parent="$(arg prefix)base_link">
+    <origin xyz="-0.24 0.095 0.30" rpy="0 0 0"/>
+  </xacro:structure_mastil_gps>
+  <!-- Gazebo ros control plugins -->
+  <xacro:arg name="config_controllers" default=""/>
+  <xacro:include filename="$(find summit_xl_description)/urdf/ros2_control.urdf.xacro"/>
+  <xacro:ros2_control/>
 </robot>

File: summit_xl_description/urdf/bases/summit_xl_base.urdf.xacro (robot description, xacro)
@@ -1,63 +1,49 @@
 <?xml version="1.0"?>
 <robot name="summit_xl" xmlns:xacro="http://wiki.ros.org/xacro">
-  <xacro:include filename="$(find summit_xl_description)/urdf/bases/summit_xl_base.gazebo.xacro" />
   <xacro:macro name="summit_xl_base" params="prefix publish_bf hq">
-	  <!-- Robot mechanical and motor parameters -->
-	  <xacro:property name="PI" value="3.1415926535897931"/>
-	  <xacro:property name="wheel_radius" value="0.11"/>
-	  <!-- BASE FOOTPRINT -->
-	  <xacro:if value="${publish_bf}">
-		<link name="${prefix}base_footprint">
-		  <visual>
-			  <origin xyz="0 0 0" rpy="0 0 0" />
-			  <geometry>
-				 <box size="0.001 0.001 0.001" />
-			  </geometry>
-		  </visual>
-		</link>
-		<joint name="${prefix}base_footprint_joint" type="fixed">
-		  <origin xyz="0 0 ${wheel_radius}" rpy="0 0 0" /> <!-- ${wheel_radius} property must be defined inside wheel description -->
-		  <parent link="${prefix}base_footprint"/>
-		  <child link="${prefix}base_link" />
-		</joint>
-	  </xacro:if>
-	  <!-- BASE_LINK -->
-	  <link name="${prefix}base_link">
-		<inertial>
-		  <mass value="25.0" />
-		  <origin xyz="0 0 0" />
-		  <inertia  ixx="1.391" ixy="0.004"  ixz="0.0"  iyy="6.853"  iyz="0.0"  izz="6.125" />
-		</inertial>
-		<visual>
-		   <origin xyz="0 0 0" rpy="0 0 0" />
-		   <xacro:if value="${hq}">
-		   <geometry>
-			 <mesh filename="package://summit_xl_description/meshes/bases/summit_xl_chassis.dae"/>
-		   </geometry>
-		   </xacro:if>
-		   <xacro:unless value="${hq}">
-		   <geometry>
-			 <mesh filename="package://summit_xl_description/meshes/bases/summit_xl_chassis_simple.stl"/>
-		   </geometry>
-		   </xacro:unless>
-		   <material name="darkgrey">
-			 <color rgba="0.1 0.1 0.1 1"/>
-		   </material>
-		</visual>
-		<collision>
-		   <origin xyz="0 0 0" rpy="0 0 0 " />
-		   <geometry>
-			 <mesh filename="package://summit_xl_description/meshes/bases/summit_xl_chassis_collision.dae"/>
-		   </geometry>
-		</collision>
-	  </link>
-		<!-- DOCKING CONTACTS -->
-		<joint name="${prefix}base_docking_joint" type="fixed">
-			<origin xyz="0.284 0.012 0.068" rpy="0 0 0 " />
-			<parent link="${prefix}base_link"/>
-			<child link="${prefix}base_docking_contact_link" />
-		</joint>
-		<!-- DOCKING LINK -->
-		<link name="${prefix}base_docking_contact_link" />
+    <!-- Robot mechanical and motor parameters -->
+    <xacro:property name="PI" value="3.1415926535897931"/>
+    <xacro:property name="wheel_radius" value="0.11"/>
+    <!-- BASE FOOTPRINT -->
+    <xacro:if value="${publish_bf}">
+      <link name="${prefix}base_footprint"/>
+      <joint name="base_footprint_joint" type="fixed">
+        <origin xyz="0 0 ${wheel_radius}" rpy="0 0 0" />
+        <parent link="${prefix}base_footprint"/>
+        <child link="${prefix}base_link" />
+      </joint>
+    </xacro:if>
+    <!-- BASE_LINK -->
+    <link name="${prefix}base_link">
+      <inertial>
+        <mass value="25.0" />
+        <origin xyz="0 0 0" />
+        <inertia  ixx="1.391" ixy="0.004"  ixz="0.0"  iyy="6.853"  iyz="0.0"  izz="6.125" />
+      </inertial>
+      <visual>
+        <origin xyz="0 0 0" rpy="0 0 0" />
+        <geometry>
+          <xacro:if value="${hq}">
+            <mesh filename="file://$(find summit_xl_description)/meshes/bases/summit_xl_chassis.dae"/>
+          </xacro:if>
+          <xacro:unless value="${hq}">
+            <mesh filename="file://$(find summit_xl_description)/meshes/bases/summit_xl_chassis_simple.stl"/>
+          </xacro:unless>
+        </geometry>
+      </visual>
+      <collision>
+        <origin xyz="0 0 0" rpy="0 0 0 " />
+        <geometry>
+          <mesh filename="file://$(find summit_xl_description)/meshes/bases/summit_xl_chassis_collision.dae"/>
+        </geometry>
+      </collision>
+    </link>
+    <!-- DOCKING -->
+    <joint name="${prefix}base_docking_joint" type="fixed">
+      <origin xyz="0.284 0.012 0.068" rpy="0 0 0 " />
+      <parent link="${prefix}base_link"/>
+      <child link="${prefix}base_docking_contact_link" />
+    </joint>
+    <link name="${prefix}base_docking_contact_link" />
   </xacro:macro>
 </robot>

Commit message: Fix antenna position

File: summit_xl_description/robots/summit_xl_std.urdf.xacro (robot description, xacro)
@@ -12,6 +12,4 @@
 	<!-- Import all available sensors -->
 	<xacro:include filename="$(find robotnik_sensors)/urdf/all_sensors.urdf.xacro" />
-	<!-- Import antenna -->
-	<xacro:include filename="$(find summit_xl_description)/urdf/structures/structure_teltonika.urdf.xacro" />
 	<!-- Import antenna -->
 	<xacro:include filename="$(find summit_xl_description)/urdf/structures/structure_teltonika.urdf.xacro" />
@@ -85,4 +83,8 @@
 			<origin xyz="-0.22528 0.095 0.275" rpy="0 0 0"/>
 		</xacro:sensor_gps_with_mast>
+	  <!--Antenna-->
+	  <xacro:structure_mastil_teltonika prefix="$(arg prefix)antenna" parent="$(arg prefix)base_link">
+			<origin xyz="-0.22528 -0.095 0.23325" rpy="0 0 0"/>
+		</xacro:structure_mastil_teltonika>
 	  <!-- Gazebo ros control pluggins -->
       <xacro:ros_control/>

Commit message: Add IMU new position

File: summit_xl_description/robots/summit_xl_std.urdf.xacro (robot description, xacro)
@@ -65,5 +65,5 @@
         <!-- IMU -->
 		<xacro:sensor_imu prefix="$(arg prefix)imu" parent="$(arg prefix)base_link" topic="imu/data_raw">
-			<origin xyz="-0.18 0.0 0.170" rpy="0 0 0"/>
+			<origin xyz="0.0385 0.132 0.158" rpy="0 0 0"/>
 		</xacro:sensor_imu>
 		<!-- 3d laser -->
