Commit message: added transmission to pan-tilt urdf

File: summit_xl_description/urdf/pan_tilt/pan_tilt.urdf.xacro (robot description, xacro)
@@ -132,4 +132,15 @@
 		<dynamics damping="${joint_damping}" friction="${joint_friction}"/>
 	</joint>
+    <transmission name="j1_trans">
+	 <type>transmission_interface/SimpleTransmission</type>
+     <joint name="${name}_joint_1">
+        <hardwareInterface>EffortJointInterface</hardwareInterface>
+     </joint>
+     <actuator name="j1_motor">
+	    <hardwareInterface>EffortJointInterface</hardwareInterface>
+        <mechanicalReduction>${j1_mechanical_reduction}</mechanicalReduction>
+		<motorTorqueConstant>${j1_motor_torque_constant}</motorTorqueConstant>
+	 </actuator>
+    </transmission>
     <!-- LINK S2 Fixed -->
 	<link name="${name}_link_s2">
@@ -208,4 +219,15 @@
 		<dynamics damping="${joint_damping}" friction="${joint_friction}"/>
 	</joint>
+    <transmission name="j2_trans">
+	 <type>transmission_interface/SimpleTransmission</type>
+     <joint name="${name}_joint_2">
+        <hardwareInterface>EffortJointInterface</hardwareInterface>
+     </joint>
+     <actuator name="j2_motor">
+	    <hardwareInterface>EffortJointInterface</hardwareInterface>
+        <mechanicalReduction>${j2_mechanical_reduction}</mechanicalReduction>
+		<motorTorqueConstant>${j2_motor_torque_constant}</motorTorqueConstant>
+	 </actuator>
+    </transmission>
   </xacro:macro>
 </robot>

Commit message: updated sign of ptu, added state launch

File: summit_xl_description/urdf/pan_tilt/pan_tilt.urdf.xacro (robot description, xacro)
@@ -128,5 +128,5 @@
 		<parent link="${name}_link_base" />
 		<child link="${name}_link_1" />
-		<axis xyz="0 0 -1" />
+		<axis xyz="0 0 1" />
 		<limit effort="${joint_effort_limit}" velocity="${joint_velocity_limit}" upper="${j1_upper_limit}" lower="${j1_lower_limit}"/>
 		<dynamics damping="${joint_damping}" friction="${joint_friction}"/>
@@ -215,5 +215,5 @@
 		<parent link="${name}_link_1" />
 		<child link="${name}_link_2" />
-		<axis xyz="0 1 0" />
+		<axis xyz="0 -1 0" />
 		<limit effort="${joint_effort_limit}" velocity="${joint_velocity_limit}" upper="${j2_upper_limit}" lower="${j2_lower_limit}"/>
 		<dynamics damping="${joint_damping}" friction="${joint_friction}"/>

Commit message: ptu range limits

File: summit_xl_description/urdf/pan_tilt/pan_tilt.urdf.xacro (robot description, xacro)
@@ -12,6 +12,8 @@
   <xacro:property name="j1_lower_limit" value="-3.13"/>
   <xacro:property name="j1_upper_limit" value="3.13"/>
-  <xacro:property name="j2_lower_limit" value="-1.5708"/>
-  <xacro:property name="j2_upper_limit" value="1.5708"/>
+  <!-- xacro:property name="j2_lower_limit" value="-1.5708"/>
+  <xacro:property name="j2_upper_limit" value="1.5708"/-->
+  <xacro:property name="j2_lower_limit" value="-1.60"/>
+  <xacro:property name="j2_upper_limit" value="1.60"/>
   <xacro:property name="joint_effort_limit" value="2.0"/>
   <xacro:property name="joint_velocity_limit" value="2.9217"/>
