Commit message: description: updating steel model to the new configuration in Kinetic

File: summit_xl_description/urdf/bases/summit_xl_hls_base.urdf.xacro (robot description, xacro)
@@ -3,23 +3,23 @@
   <xacro:include filename="$(find summit_xl_description)/urdf/bases/summit_xl_base.gazebo.xacro" />
   <xacro:macro name="summit_xl_hls_base" params="prefix publish_bf hq">
-  <!-- Robot mechanical and motor parameters -->
-  <xacro:property name="PI" value="3.1415926535897931"/>
-  <!-- xacro:property name="wheel_width" value="0.175" / -->
-  <!-- BASE FOOTPRINT -->
-  <xacro:if value="${publish_bf}">
-    <link name="${prefix}base_footprint">
-      <visual>
-          <origin xyz="0 0 0" rpy="0 0 0" />
-          <geometry>
-             <box size="0.001 0.001 0.001" />
-          </geometry>
-      </visual>
-    </link>
-    <joint name="${prefix}base_footprint_joint" type="fixed">
-      <origin xyz="0 0 ${wheel_radius}" rpy="0 0 0" /> <!-- ${wheel_radius} property must be defined inside wheel description -->
-      <parent link="${prefix}base_footprint"/>
-      <child link="${prefix}base_link" />
-    </joint>
-  </xacro:if>
+	  <!-- Robot mechanical and motor parameters -->
+	  <xacro:property name="PI" value="3.1415926535897931"/>
+	  <xacro:property name="wheel_width" value="0.175" />
+	<!-- BASE FOOTPRINT -->
+	  <xacro:if value="${publish_bf}">
+		<link name="${prefix}base_footprint">
+		  <visual>
+			  <origin xyz="0 0 0" rpy="0 0 0" />
+			  <geometry>
+				 <box size="0.001 0.001 0.001" />
+			  </geometry>
+		  </visual>
+		</link>
+		<joint name="${prefix}base_footprint_joint" type="fixed">
+		  <origin xyz="0 0 ${wheel_radius}" rpy="0 0 0" /> <!-- ${wheel_radius} property must be defined inside wheel description -->
+		  <parent link="${prefix}base_footprint"/>
+		  <child link="${prefix}base_link" />
+		</joint>
+	  </xacro:if>
   <!-- BASE_LINK -->
   <link name="${prefix}base_link">

File: summit_xl_description/urdf/structures/structure_hokuyo.urdf.xacro (robot description, xacro)
@@ -1,5 +1,5 @@
 <?xml version="1.0"?>
 <robot name="structure" xmlns:xacro="http://www.ros.org/wiki/xacro">
-  <xacro:macro name="structure" params="prefix parent *origin">
+  <xacro:macro name="structure_laser" params="prefix parent *origin">
 	  <joint name="${prefix}_joint" type="fixed">
 	    <axis xyz="0 1 0"/>

File: summit_xl_description/urdf/structures/structure_ptz_rgbd_gps.urdf.xacro (robot description, xacro)
@@ -1,5 +1,5 @@
 <?xml version="1.0"?>
 <robot name="structure" xmlns:xacro="http://ros.org/wiki/xacro">
-  <xacro:macro name="structure" params="prefix parent *origin">
+  <xacro:macro name="structure_ptz" params="prefix parent *origin">
 	  <joint name="${prefix}_joint" type="fixed">
 	    <axis xyz="0 1 0"/>

Commit message: description: increasing mass of XL Steel

File: summit_xl_description/urdf/bases/summit_xl_hls_base.urdf.xacro (robot description, xacro)
@@ -25,5 +25,5 @@
   <link name="${prefix}base_link">
     <inertial>
-      <mass value="25.0" />
+      <mass value="125.0" />
       <origin xyz="0 0 0" />
       <inertia  ixx="1.391" ixy="0.004"  ixz="0.0"  iyy="6.853"  iyz="0.0"  izz="6.125" />
