Commit message: added a standard steel model to rviz launch

File: summit_xl_description/urdf/bases/summit_xl_steel_base.urdf.xacro (robot description, xacro)
@@ -2,5 +2,5 @@
 <robot name="summit_xl" xmlns:xacro="http://www.ros.org/wiki/xacro">
   <xacro:include filename="$(find summit_xl_description)/urdf/bases/summit_xl_base.gazebo.xacro" />
-  <xacro:macro name="summit_xl_hls_base" params="name publish_bf hq">
+  <xacro:macro name="summit_xl_steel_base" params="name publish_bf hq">
   <!-- Robot mechanical and motor parameters -->
   <xacro:property name="PI" value="3.1415926535897931"/>
@@ -33,10 +33,10 @@
        <xacro:if value="${hq}">
        <geometry>
-	     <mesh filename="package://summit_xl_description/meshes/bases/hls/v2017/chasis_box.stl"/>
+	     <mesh filename="package://summit_xl_description/meshes/bases/hls/v2017/chassis_box.stl"/>
        </geometry>
        </xacro:if>
        <xacro:unless value="${hq}">
        <geometry>
-	     <mesh filename="package://summit_xl_description/meshes/bases/hls/v2017/chasis.dae"/>
+	     <mesh filename="package://summit_xl_description/meshes/bases/hls/v2017/chassis_box.dae"/>
        </geometry>
        </xacro:unless>
@@ -48,5 +48,5 @@
        <origin xyz="0 0 0" rpy="0 0 0 " />
        <geometry>
-         <mesh filename="package://summit_xl_description/meshes/bases/hls/v2017/chasis.dae"/>
+         <mesh filename="package://summit_xl_description/meshes/bases/hls/v2017/chassis_box.dae"/>
        </geometry>
     </collision>

Commit message: added meshes with robotnik logo for steel

File: summit_xl_description/urdf/bases/summit_xl_steel_base.urdf.xacro (robot description, xacro)
@@ -33,10 +33,10 @@
        <xacro:if value="${hq}">
        <geometry>
-	     <mesh filename="package://summit_xl_description/meshes/bases/hls/v2017/chassis_box.stl"/>
+	     <mesh filename="package://summit_xl_description/meshes/bases/hls/v2017/chassis_box.dae"/>
        </geometry>
        </xacro:if>
        <xacro:unless value="${hq}">
        <geometry>
-	     <mesh filename="package://summit_xl_description/meshes/bases/hls/v2017/chassis_box.dae"/>
+	     <mesh filename="package://summit_xl_description/meshes/bases/hls/v2017/chassis_box.stl"/>
        </geometry>
        </xacro:unless>
