Commit message: summit_xl_description:: Added docking_contact link to URDF. Added robots version

File: summit_xl_description/urdf/bases/summit_xl_base.urdf.xacro (robot description, xacro)
@@ -52,4 +52,12 @@
 		</collision>
 	  </link>
+		<!-- DOCKING CONTACTS -->
+		<joint name="${prefix}base_docking_joint" type="fixed">
+			<origin xyz="0.282 0.0 0.078" rpy="0 0 0 " />
+			<parent link="${prefix}base_link"/>
+			<child link="${prefix}base_docking_contact_link" />
+		</joint>
+		<!-- DOCKING LINK -->
+	<link name="${prefix}base_docking_contact_link" />
   </xacro:macro>
 </robot>

Commit message: description: added docking_contact_link to the base urdf

File: summit_xl_description/urdf/bases/summit_xl_base.urdf.xacro (robot description, xacro)
@@ -52,4 +52,12 @@
 		</collision>
 	  </link>
+		<!-- DOCKING CONTACTS -->
+		<joint name="${prefix}base_docking_joint" type="fixed">
+			<origin xyz="0.284 0.012 0.068" rpy="0 0 0 " />
+			<parent link="${prefix}base_link"/>
+			<child link="${prefix}base_docking_contact_link" />
+		</joint>
+		<!-- DOCKING LINK -->
+		<link name="${prefix}base_docking_contact_link" />
   </xacro:macro>
 </robot>
