Commit message: description: setting new position (+5 cm) for the docking contacts for the new steel model

File: summit_xl_description/urdf/bases/summit_xls_base.urdf.xacro (robot description, xacro)
@@ -56,5 +56,5 @@
     </link>
     <joint name="${prefix}base_docking_joint" type="fixed">
-      <origin xyz="0.30 0 0.09" rpy="0 0 0" />
+      <origin xyz="0.35 0 0.09" rpy="0 0 0" />
       <parent link="${prefix}base_link"/>
       <child link="${prefix}base_docking_contact" />

Commit message: Update summit_xls_base.urdf.xacro

File: summit_xl_description/urdf/bases/summit_xls_base.urdf.xacro (robot description, xacro)
@@ -148,4 +148,16 @@
       <child link="${prefix}base_docking_contact" />
     </joint>
+  <xacro:include filename="$(find roas_bringup)/urdf/roas.urdf.xacro"/>
+  <xacro:include filename="$(find ur_e_description)/urdf/ur5e_robot.urdf.xacro"/>
+  <joint name="top_structure_joint" type="fixed">
+    <origin xyz="0.0 0 0.0" rpy="0 0 0" />
+    <parent link="${prefix}base_chapa"/>
+    <child link="top_structure" />
+  </joint>
+  <joint name="${prefix}ur5e_joint" type="fixed">
+    <parent link="${prefix}base_link" />
+    <child link ="ur5e_base_link" />
+    <origin xyz="0.255 0 0.4" rpy="0 0 -1.5708" />
+  </joint>
   </xacro:macro>
 </robot>

Commit message: put it back the original ur5e base configuration

File: summit_xl_description/urdf/bases/summit_xls_base.urdf.xacro (robot description, xacro)
@@ -159,6 +159,5 @@
     <parent link="${prefix}base_link" />
     <child link ="ur5e_base_link" />
-    <origin xyz="0.255 0 0.4" rpy="0 0 0" />
-    <!-- <origin xyz="0.255 0 0.4" rpy="0 0 -1.5708" /> -->
+    <origin xyz="0.255 0 0.4" rpy="0 0 -1.5708" />
   </joint>
   </xacro:macro>
