Commit message: description: renames from oem to plus

File: summit_xl_description/urdf/bases/summit_xlsk_base_plus.urdf.xacro (robot description, xacro)
@@ -33,10 +33,10 @@
       <xacro:if value="${hq}">
       <geometry>
-      <mesh filename="package://summit_xl_description/meshes/bases/xls/summit_xlsk_oem.stl"/>
+      <mesh filename="package://summit_xl_description/meshes/bases/xls/summit_xlsk_plus.stl"/>
       </geometry>
       </xacro:if>
       <xacro:unless value="${hq}">
       <geometry>
-      <mesh filename="package://summit_xl_description/meshes/bases/xls/summit_xlsk_oem.dae"/>
+      <mesh filename="package://summit_xl_description/meshes/bases/xls/summit_xlsk_plus.dae"/>
       </geometry>
       </xacro:unless>
@@ -48,5 +48,5 @@
        <origin xyz="0 0 0" rpy="0 0 0 " />
        <geometry>
-         <mesh filename="package://summit_xl_description/meshes/bases/xls/summit_xlsk_oem.dae"/>
+         <mesh filename="package://summit_xl_description/meshes/bases/xls/summit_xlsk_plus.dae"/>
        </geometry>
     </collision>

Commit message: description: Several changes
- From oem to plus
- Adds laser support
- Fixes plates and logos positions

File: summit_xl_description/urdf/bases/summit_xlsk_base_plus.urdf.xacro (robot description, xacro)
@@ -2,5 +2,6 @@
 <robot name="summit_xl" xmlns:xacro="http://wiki.ros.org/xacro">
   <xacro:include filename="$(find summit_xl_description)/urdf/bases/summit_xl_base.gazebo.xacro" />
-  <xacro:macro name="summit_xls_base" params="prefix publish_bf hq">
+  <xacro:include filename="$(find summit_xl_description)/urdf/structures/sick_microscan3_support.urdf.xacro" />
+  <xacro:macro name="summit_xls_base" params="prefix publish_bf hq laser_support:=true">
   <!-- Robot mechanical and motor parameters -->
   <xacro:property name="PI" value="3.1415926535897931"/>
@@ -33,10 +34,10 @@
       <xacro:if value="${hq}">
       <geometry>
-      <mesh filename="package://summit_xl_description/meshes/bases/xls/summit_xlsk_oem.stl"/>
+      <mesh filename="package://summit_xl_description/meshes/bases/xls/summit_xlsk_plus.stl"/>
       </geometry>
       </xacro:if>
       <xacro:unless value="${hq}">
       <geometry>
-      <mesh filename="package://summit_xl_description/meshes/bases/xls/summit_xlsk_oem.dae"/>
+      <mesh filename="package://summit_xl_description/meshes/bases/xls/summit_xlsk_plus.dae"/>
       </geometry>
       </xacro:unless>
@@ -48,11 +49,6 @@
        <origin xyz="0 0 0" rpy="0 0 0 " />
        <geometry>
-         <mesh filename="package://summit_xl_description/meshes/bases/xls/summit_xlsk_oem.dae"/>
+         <mesh filename="package://summit_xl_description/meshes/bases/xls/summit_xlsk_plus.dae"/>
        </geometry>
-       <!-- better a box than a mesh for collision -->
-      <!--<origin xyz="0 0 0.381" rpy="0 0 0"/>-->
-      <!--<geometry>-->
-        <!--<box size="0.719 0.578 0.363"/>-->
-      <!--</geometry>-->
     </collision>
   </link>
@@ -73,5 +69,5 @@
   </link>
   <joint name="${prefix}base_tapa_joint" type="fixed">
-    <origin xyz="0.0 0 0.38062" rpy="0 0 0" />
+    <origin xyz="0.0 0 0.56162" rpy="0 0 0" />
     <parent link="${prefix}base_link"/>
     <child link="${prefix}base_chapa" />
@@ -90,5 +86,5 @@
   </link>
   <joint name="${prefix}base_logo_left_joint" type="fixed">
-    <origin xyz="0.0 0.28931 0.29062" rpy="0 0 0" />
+    <origin xyz="0.0 0.2894 0.35562" rpy="0 0 0" />
     <parent link="${prefix}base_link"/>
     <child link="${prefix}base_logo_left" />
@@ -107,5 +103,5 @@
   </link>
   <joint name="${prefix}base_logo_right_joint" type="fixed">
-    <origin xyz="0.0 -0.28931 0.29062" rpy="0 0 ${PI}" />
+    <origin xyz="0.0 -0.28931 0.35562" rpy="0 0 ${PI}" />
     <parent link="${prefix}base_link"/>
     <child link="${prefix}base_logo_right" />
@@ -153,4 +149,12 @@
       <child link="${prefix}base_docking_contact" />
     </joint>
+  <xacro:if value="${laser_support}">
+    <sick_microscan3_support prefix="${prefix}front_laser" parent="${prefix}base_link" >
+      <origin xyz="0.28704 -0.22255 0.20212" rpy="0 0 -0.645772" />
+    </sick_microscan3_support>
+    <sick_microscan3_support prefix="${prefix}rear_laser" parent="${prefix}base_link" >
+      <origin xyz="-0.28704 +0.22255 0.20212" rpy="0 0 2.496" />
+    </sick_microscan3_support>
+  </xacro:if>
   </xacro:macro>
 </robot>
