Commit message: Transmission modified with new style.

File: summit_xl_description/urdf/bases/summit_xl_base.gazebo.xacro (robot description, xacro)
@@ -2,5 +2,5 @@
 <robot xmlns:xacro="http://ros.org/wiki/xacro">
   <!-- ros control plugin -->
-  <!-- xacro:macro name="ros_control">
+  <xacro:macro name="ros_control">
     <gazebo>
       <plugin name="ros_control" filename="libgazebo_ros_control.so">
@@ -11,10 +11,10 @@
       </plugin>
     </gazebo>
-	</xacro:macro -->
+	</xacro:macro>
 	<!-- skid steering plugin -->
 	<xacro:macro name="skid_steering" params="broadcastOdomTF">
     <gazebo>
       <plugin name="skid_steer_drive_controller" filename="libgazebo_ros_skid_steer_drive.so">
-				<robotNamespace>/summit_xl</robotNamespace>
+			<robotNamespace>/summit_xl</robotNamespace>
 		    <updateRate>100.0</updateRate>
 		    <leftFrontJoint>joint_front_left_wheel</leftFrontJoint>

File: summit_xl_description/urdf/bases/summit_xl_base.urdf.xacro (robot description, xacro)
@@ -1,5 +1,5 @@
 <?xml version="1.0"?>
 <robot name="summit_xl" xmlns:xacro="http://www.ros.org/wiki/xacro">
-	<xacro:include filename="$(find summit_xl_description)/urdf/bases/summit_xl_base.gazebo.xacro" />
+  <xacro:include filename="$(find summit_xl_description)/urdf/bases/summit_xl_base.gazebo.xacro" />
   <xacro:macro name="summit_xl_base" params="name publish_bf hq">
   <!-- Robot mechanical and motor parameters -->

File: summit_xl_description/urdf/bases/summit_xl_hl_base.urdf.xacro (robot description, xacro)
@@ -38,5 +38,5 @@
        <xacro:unless value="${hq}">
        <geometry>
-	     <mesh filename="package://summit_xl_description/meshes/bases/summit_xl_hl_chassis_simple.stl"/>
+	     <mesh filename="package://summit_xl_description/meshes/bases/summit_xl_hl_chassis.dae"/>
        </geometry>
        </xacro:unless>
@@ -48,5 +48,5 @@
        <origin xyz="0 0 0" rpy="0 0 0 " />
        <geometry>
-         <mesh filename="package://summit_xl_description/meshes/bases/summit_xl_hl_chassis_collision.dae"/>
+         <mesh filename="package://summit_xl_description/meshes/bases/summit_xl_hl_chassis.dae"/>
        </geometry>
     </collision>

File: summit_xl_description/urdf/wheels/omni_wheel.urdf.xacro (robot description, xacro)
@@ -71,8 +71,9 @@
     <transmission name="${name}_wheel_joint_trans">
       <type>transmission_interface/SimpleTransmission</type>
-      <joint name="joint_${name}_wheel" />
+      <joint name="joint_${name}_wheel" >
+         <hardwareInterface>EffortJointInterface</hardwareInterface>
+      </joint>
       <actuator name="${name}_wheel_joint_motor">
-        <hardwareInterface>EffortJointInterface</hardwareInterface>
-        <mechanicalReduction>1</mechanicalReduction>
+         <mechanicalReduction>1</mechanicalReduction>
       </actuator>
     </transmission>

File: summit_xl_description/urdf/wheels/rubber_wheel.urdf.xacro (robot description, xacro)
@@ -58,13 +58,14 @@
     <transmission name="${name}_wheel_joint_trans">
       <type>transmission_interface/SimpleTransmission</type>
-      <joint name="joint_${name}_wheel" />
+      <joint name="joint_${name}_wheel">
+		<hardwareInterface>EffortJointInterface</hardwareInterface>
+      </joint>
       <actuator name="${name}_wheel_joint_motor">
-        <hardwareInterface>EffortJointInterface</hardwareInterface>
         <mechanicalReduction>1</mechanicalReduction>
       </actuator>
-    </transmission>
+     </transmission>
     <gazebo reference="${name}_wheel">
-			<mu1 value="5.0"/>
-			<mu2 value="0.5"/>
+			<mu1 value="1.0"/>
+			<mu2 value="1.0"/>
 			<kp value="10000000.0" />
 			<kd value="1.0" />

Commit message: remove sliding of robot through gazebo plugin

File: summit_xl_description/urdf/bases/summit_xl_base.gazebo.xacro (robot description, xacro)
@@ -62,5 +62,5 @@
   <xacro:macro name="ros_force_based_move" params="publish_tf prefix">
 	  <gazebo>
-		 <plugin name="ros_force_based_move" filename="libgazebo_ros_force_based_move.so">
+		 <plugin name="ros_force_based_move" filename="librobotnik_force_based_move.so">
 			 <commandTopic>robotnik_base_control/cmd_vel</commandTopic>
 			 <odometryTopic>robotnik_base_control/odom</odometryTopic>
@@ -70,4 +70,5 @@
 			 <y_velocity_p_gain>10000.0</y_velocity_p_gain>
 			 <robotBaseFrame>${prefix}base_footprint</robotBaseFrame>
+			 <commandWatchdog>1</commandWatchdog>
 			 <odometryRate>50.0</odometryRate>
 			 <publishOdometryTf>${publish_tf}</publishOdometryTf>

File: summit_xl_description/urdf/bases/summit_xlsk_base_oem.urdf.xacro (robot description, xacro)
@@ -50,4 +50,9 @@
          <mesh filename="package://summit_xl_description/meshes/bases/xls/summit_xlsk_oem.dae"/>
        </geometry>
+       <!-- better a box than a mesh for collision -->
+      <!--<origin xyz="0 0 0.381" rpy="0 0 0"/>-->
+      <!--<geometry>-->
+        <!--<box size="0.719 0.578 0.363"/>-->
+      <!--</geometry>-->
     </collision>
   </link>

File: summit_xl_description/urdf/wheels/omni_wheel.urdf.xacro (robot description, xacro)
@@ -58,4 +58,5 @@
 -->
 					<cylinder length="${omni_wheel_height}" radius="${omni_wheel_radius}" />
+					<!-- sphere radius="${omni_wheel_radius}"/-->
         </geometry>
       </collision>

Commit message: summit_xl_descritpion: Sets force_based param to false by default

File: summit_xl_description/urdf/bases/summit_xl_base.gazebo.xacro (robot description, xacro)
@@ -34,5 +34,5 @@
     </gazebo>
   </xacro:macro>
-  <xacro:macro name="omni_steering" params="prefix publish_tf force_based">
+  <xacro:macro name="omni_steering" params="prefix publish_tf force_based:=false">
 		<xacro:if value="${force_based}">
 			<gazebo>
