Commit message: versions: updated rgbd camera offset

File: summit_xl_description/robots/versions/SXLS0-180704AA.urdf.xacro (robot description, xacro)
@@ -34,7 +34,7 @@
 	<xacro:property name="imu_offset_y" value="-0.15"/>
 	<xacro:property name="imu_offset_z" value="0.18"/>
-	<xacro:property name="front_rgbd_camera_offset_x" value="0.324"/>
+	<xacro:property name="front_rgbd_camera_offset_x" value="0.374"/>
 	<xacro:property name="front_rgbd_camera_offset_y" value="0.012"/>
-	<xacro:property name="front_rgbd_camera_offset_z" value="0.230"/>
+	<xacro:property name="front_rgbd_camera_offset_z" value="0.295"/>
 	<xacro:property name="gps_offset_x" value="-0.365"/>
 	<xacro:property name="gps_offset_y" value="-0.167"/>
