Commit message: description: Add model version SHL00-181120AC

File: summit_xl_description/robots/versions/SHL00-181120AC.urdf.xacro (robot description, xacro)
@@ -54,7 +54,7 @@
 		</xacro:sensor_orbbec_astra>
 	    <!-- GPS -->
-	    <!--xacro:sensor_gps prefix="$(arg prefix)gps" parent="$(arg prefix)base_link">
-			<origin xyz="-0.22 0 0.275" rpy="0 0 0"/>
-		</xacro:sensor_gps-->
+	    <xacro:sensor_gps prefix="$(arg prefix)gps" parent="$(arg prefix)base_link">
+			<origin xyz="-0.0 0.0 0.37" rpy="0 0 0"/>
+		</xacro:sensor_gps>
    </xacro:macro>
    <!-- Gazebo ros control pluggins -->
