Commit message: summit_xl_description: Update summit_xl with kinova gen urdf

File: summit_xl_description/robots/versions/SXL00-200505AA.urdf.xacro (robot description, xacro)
@@ -74,7 +74,7 @@
 		</xacro:sensor_hokuyo_ust10lx-->
 		<!-- 3d laser -->
-		<!--xacro:sensor_rslidar_mems prefix="$(arg prefix)top_3d_laser" parent="$(arg prefix)base_link">
+		<xacro:sensor_rslidar_mems prefix="$(arg prefix)top_3d_laser" parent="$(arg prefix)base_link">
 			<origin xyz="0.3134 0 0.2424" rpy="0 0 0"/>
-		</xacro:sensor_rslidar_mems-->
+		</xacro:sensor_rslidar_mems>
 		<!-- ptz camera -->
 		<!--xacro:sensor_axis prefix="$(arg prefix)front_ptz_camera" parent="$(arg prefix)base_link">
@@ -86,7 +86,7 @@
 		</xacro:sensor_orbbec_astra-->
 	  <!-- GPS -->
-	  <!--xacro:sensor_gps prefix="$(arg prefix)gps" parent="$(arg prefix)base_link">
-			<origin xyz="-0.28 0 0.6676" rpy="0 0 0"/>
-		</xacro:sensor_gps-->
+	  <xacro:sensor_gps_with_mast prefix="$(arg prefix)gps" parent="$(arg prefix)base_link">
+		<origin xyz="-0.28 0 0.4176" rpy="0 0 0"/>
+	</xacro:sensor_gps_with_mast>
     <!-- Instance jaco arm -->
     <joint name="$(arg prefix)arm_base_joint" type="fixed">

Commit message: description: Update version 200505AA with basic wheels

File: summit_xl_description/robots/versions/SXL00-200505AA.urdf.xacro (robot description, xacro)
@@ -8,6 +8,5 @@
 	<xacro:include filename="$(find summit_xl_description)/urdf/bases/summit_xl_base.urdf.xacro" />
 	<!-- Import summit XL wheels -->
-	<xacro:include filename="$(find summit_xl_description)/urdf/wheels/rubber_wheel.urdf.xacro" />
-  <xacro:include filename="$(find summit_xl_description)/urdf/wheels/omni_wheel.urdf.xacro" />
+	<xacro:include filename="$(find summit_xl_description)/urdf/wheels/basic_wheel.urdf.xacro" />
 	<!-- Import all available sensors -->
 	<xacro:include filename="$(find robotnik_sensors)/urdf/all_sensors.urdf.xacro" />
@@ -18,4 +17,7 @@
 	<xacro:property name="wheel_offset_y" value="0.235" />
 	<xacro:property name="wheel_offset_z" value="0.0" />
+	<xacro:property name="wheel_radius" value="0.1025" />
+	<xacro:property name="wheel_height" value="0.14" />
+	<xacro:property name="wheel_mass" value="0.5" />
   <xacro:property name="arm_offset_x" value="0.204" />    <!-- x,y,z in translation from base_link to the center of the arm -->
 	<xacro:property name="arm_offset_y" value="0.0" />
@@ -37,76 +39,48 @@
 		<!-- Summit XL base -->
 		<xacro:summit_xl_base prefix="$(arg prefix)" publish_bf="true" hq="${hq}" />
-    <xacro:unless value="$(arg omni_wheels)">
-  		<xacro:rubber_wheel prefix="$(arg prefix)front_right" parent="$(arg prefix)base_link" reflect="false" hq="${hq}">
+  		<xacro:basic_wheel prefix="$(arg prefix)front_right" parent="$(arg prefix)base_link" radius="${wheel_radius}" height="${wheel_height}" mass="${wheel_height}">
   			<origin xyz="${wheel_offset_x} -${wheel_offset_y} ${wheel_offset_z}" rpy="0 0 0"/>
-  		</xacro:rubber_wheel>
-  		<xacro:rubber_wheel prefix="$(arg prefix)front_left" parent="$(arg prefix)base_link" reflect="true" hq="${hq}">
+  		</xacro:basic_wheel>
+  		<xacro:basic_wheel prefix="$(arg prefix)front_left" parent="$(arg prefix)base_link" radius="${wheel_radius}" height="${wheel_height}" mass="${wheel_height}">
   			<origin xyz="${wheel_offset_x} ${wheel_offset_y} ${wheel_offset_z}" rpy="0 0 0"/>
-  		</xacro:rubber_wheel>
-  		<xacro:rubber_wheel prefix="$(arg prefix)back_left" parent="$(arg prefix)base_link" reflect="true" hq="${hq}">
+  		</xacro:basic_wheel>
+  		<xacro:basic_wheel prefix="$(arg prefix)back_left" parent="$(arg prefix)base_link" radius="${wheel_radius}" height="${wheel_height}" mass="${wheel_height}">
   			<origin xyz="-${wheel_offset_x} ${wheel_offset_y} ${wheel_offset_z}" rpy="0 0 0"/>
-  		</xacro:rubber_wheel>
-  		<xacro:rubber_wheel prefix="$(arg prefix)back_right" parent="$(arg prefix)base_link" reflect="false" hq="${hq}">
+  		</xacro:basic_wheel>
+  		<xacro:basic_wheel prefix="$(arg prefix)back_right" parent="$(arg prefix)base_link" radius="${wheel_radius}" height="${wheel_height}" mass="${wheel_height}">
   			<origin xyz="-${wheel_offset_x} -${wheel_offset_y} ${wheel_offset_z}" rpy="0 0 0"/>
-  		</xacro:rubber_wheel>
-    </xacro:unless>
-    <xacro:if value="$(arg omni_wheels)">
-  		<xacro:omni_wheel prefix="$(arg prefix)front_right" parent="$(arg prefix)base_link" reflect="false" hq="${hq}">
-  			<origin xyz="${wheel_offset_x} -${wheel_offset_y} ${wheel_offset_z}" rpy="0 0 0"/>
-  		</xacro:omni_wheel>
-  		<xacro:omni_wheel prefix="$(arg prefix)front_left" parent="$(arg prefix)base_link" reflect="true" hq="${hq}">
-  			<origin xyz="${wheel_offset_x} ${wheel_offset_y} ${wheel_offset_z}" rpy="0 0 0"/>
-  		</xacro:omni_wheel>
-  		<xacro:omni_wheel prefix="$(arg prefix)back_left" parent="$(arg prefix)base_link" reflect="true" hq="${hq}">
-  			<origin xyz="-${wheel_offset_x} ${wheel_offset_y} ${wheel_offset_z}" rpy="0 0 0"/>
-  		</xacro:omni_wheel>
-  		<xacro:omni_wheel prefix="$(arg prefix)back_right" parent="$(arg prefix)base_link" reflect="false" hq="${hq}">
-  			<origin xyz="-${wheel_offset_x} -${wheel_offset_y} ${wheel_offset_z}" rpy="0 0 0"/>
-  		</xacro:omni_wheel>
+  		</xacro:basic_wheel>
+        <!-- IMU -->
+      <xacro:sensor_imu prefix="$(arg prefix)imu" parent="$(arg prefix)base_link">
+        <origin xyz="-0.18 0.0 0.170" rpy="0 0 0"/>
+      </xacro:sensor_imu>
+      <!-- 3d laser -->
+      <xacro:sensor_rslidar_mems prefix="$(arg prefix)top_3d_laser" parent="$(arg prefix)base_link">
+        <origin xyz="0.3134 0 0.2424" rpy="0 0 0"/>
+      </xacro:sensor_rslidar_mems>
+      <!-- GPS -->
+      <xacro:sensor_gps_with_mast prefix="$(arg prefix)gps" parent="$(arg prefix)base_link">
+        <origin xyz="-0.28 0 0.4176" rpy="0 0 0"/>
+      </xacro:sensor_gps_with_mast>
+      <!-- Instance jaco arm -->
+      <joint name="$(arg prefix)arm_base_joint" type="fixed">
+        <origin xyz="${arm_offset_x} ${arm_offset_y} ${arm_offset_z}" rpy="${arm_offset_roll} ${arm_offset_pitch} ${arm_offset_yaw}" />
+        <parent link="$(arg prefix)base_link" />
+        <child link="$(arg prefix)arm_base_link" />
+        <axis xyz="0 0 0" />
+      </joint>
+      <link name="$(arg prefix)arm_base_link" />
+      <xacro:j2s7s300 base_parent="$(arg prefix)arm_base_link" prefix="$(arg prefix)j2s7s300"/>
+    </xacro:macro>
+   <!-- Gazebo ros control pluggins -->
+    <xacro:ros_control/>
+    <xacro:if value="$(arg ros_planar_move_plugin)">
+      <xacro:if value="$(arg omni_wheels)">
+        <xacro:omni_steering prefix="$(arg prefix)" publish_tf="true"/>
+      </xacro:if>
+      <xacro:unless value="$(arg omni_wheels)">
+        <xacro:skid_steering prefix="$(arg prefix)" publish_tf="true"/>
+      </xacro:unless>
     </xacro:if>
-        <!-- IMU -->
-		<xacro:sensor_imu prefix="$(arg prefix)imu" parent="$(arg prefix)base_link">
-			<origin xyz="-0.18 0.0 0.170" rpy="0 0 0"/>
-		</xacro:sensor_imu>
-		<!-- 2d laser -->
-		<!--xacro:sensor_hokuyo_ust10lx prefix="$(arg prefix)front_laser" parent="$(arg prefix)base_link" prefix_topic="front_laser" gpu="$(arg gpu)">
-			<origin xyz="0.0 0.0 0.33" rpy="0 0 0"/>
-		</xacro:sensor_hokuyo_ust10lx-->
-		<!-- 3d laser -->
-		<xacro:sensor_rslidar_mems prefix="$(arg prefix)top_3d_laser" parent="$(arg prefix)base_link">
-			<origin xyz="0.3134 0 0.2424" rpy="0 0 0"/>
-		</xacro:sensor_rslidar_mems>
-		<!-- ptz camera -->
-		<!--xacro:sensor_axis prefix="$(arg prefix)front_ptz_camera" parent="$(arg prefix)base_link">
-			<origin xyz="0.19 0 0.26" rpy="0 ${15*PI/180} 0"/>
-		</xacro:sensor_axis-->
-	  <!-- RGBD -->
-	  <!--xacro:sensor_orbbec_astra prefix="$(arg prefix)front_rgbd_camera" parent="$(arg prefix)base_link" prefix_topic="front_rgbd_camera">
-			<origin xyz="0.324 0.012 0.172" rpy="0 0 0"/>
-		</xacro:sensor_orbbec_astra-->
-	  <!-- GPS -->
-	  <xacro:sensor_gps_with_mast prefix="$(arg prefix)gps" parent="$(arg prefix)base_link">
-		<origin xyz="-0.28 0 0.4176" rpy="0 0 0"/>
-	</xacro:sensor_gps_with_mast>
-    <!-- Instance jaco arm -->
-    <joint name="$(arg prefix)arm_base_joint" type="fixed">
-      <origin xyz="${arm_offset_x} ${arm_offset_y} ${arm_offset_z}" rpy="${arm_offset_roll} ${arm_offset_pitch} ${arm_offset_yaw}" />
-      <parent link="$(arg prefix)base_link" />
-      <child link="$(arg prefix)arm_base_link" />
-      <axis xyz="0 0 0" />
-    </joint>
-    <link name="$(arg prefix)arm_base_link" />
-    <xacro:j2s7s300 base_parent="$(arg prefix)arm_base_link" prefix="$(arg prefix)j2s7s300"/>
-   </xacro:macro>
-   <!-- Gazebo ros control pluggins -->
-   <xacro:ros_control/>
-	<xacro:if value="$(arg ros_planar_move_plugin)">
-		<xacro:if value="$(arg omni_wheels)">
-			<xacro:omni_steering prefix="$(arg prefix)" publish_tf="true"/>
-		</xacro:if>
-		<xacro:unless value="$(arg omni_wheels)">
-			<xacro:skid_steering prefix="$(arg prefix)" publish_tf="true"/>
-		</xacro:unless>
-	</xacro:if>
-   <xacro:summit_xl_gen prefix="$(arg prefix)" publish_bf="true" hq="true"/>
+    <xacro:summit_xl_gen prefix="$(arg prefix)" publish_bf="true" hq="true"/>
 </robot>
