Commit message: Update urdf to common ones

File: summit_xl_description/robots/versions/summit_xl_gen_j2s7s300.urdf.xacro (robot description, xacro)
@@ -12,5 +12,5 @@
     <!-- Import all available sensors -->
     <xacro:include filename="$(find robotnik_sensors)/urdf/all_sensors.urdf.xacro" />
-    <xacro:include filename="$(find summit_xl_description)/urdf/arms/kinova/j2s6s300.xacro" />
+    <xacro:include filename="$(find summit_xl_description)/urdf/arms/kinova/j2s7s300.xacro" />
     <xacro:property name="PI" value="3.1415926535897931"/>
     <!-- Wheel parameters -->
@@ -18,5 +18,4 @@
     <xacro:property name="wheel_offset_y" value="0.235" />
     <xacro:property name="wheel_offset_z" value="0.0" />
-    -
     <xacro:property name="arm_offset_x" value="0.204" />    <!-- x,y,z in translation from base_link to the center of the arm -->
     <xacro:property name="arm_offset_y" value="0.0" />
@@ -71,43 +70,11 @@
         </xacro:sensor_imu>
         <!-- 2d laser -->
-        <xacro:sensor_hokuyo_utm30lx prefix="$(arg prefix)front_laser" parent="$(arg prefix)base_link" prefix_topic="front_laser" gpu="$(arg gpu)">
-            <origin xyz="0.290 0.0 0.235" rpy="0 0 0"/>
-        </xacro:sensor_hokuyo_utm30lx>
-        <!-- MAST OF THE ANTENNA GPS -->
-	  <joint name="$(arg prefix)mast_base_joint" type="fixed">
-	    <origin xyz="-0.2776 0 0.44"/>
-	    <parent link="$(arg prefix)base_link"/>
-	    <child link="$(arg prefix)mast_base_link"/>
-	  </joint>
-	  <link name="$(arg prefix)mast_base_link">
-	    <inertial>
-	      <mass value="0.001"/>
-	      <origin rpy="0 0 0" xyz="0 0 0"/>
-	      <inertia ixx="0.0001" ixy="0" ixz="0" iyy="0.000001" iyz="0" izz="0.0001"/>
-	    </inertial>
-	    <visual>
-	      <origin rpy="0 0 0" xyz="0 0 0"/>
-	      <material name="mast_color">
-	    <color rgba="0.1 0.1 0.1 1"/>
-	  </material>
-	      <geometry>
-		<cylinder length="0.629" radius="0.02" />
-	      </geometry>
-	    </visual>
-	    <collision>
-	      <origin rpy="0 0 0" xyz="0 0 0"/>
-	      <geometry>
-		<cylinder length="0.629" radius="0.02" />
-	      </geometry>
-	    </collision>
-	  </link>
-	  <gazebo reference="$(arg prefix)mast_base_link">
-	    <material>Gazebo/Black</material>
-	    <gravity>true</gravity>
-	  </gazebo>
+        <!--xacro:sensor_hokuyo_ust10lx prefix="$(arg prefix)front_laser" parent="$(arg prefix)base_link" prefix_topic="front_laser" gpu="$(arg gpu)">
+            <origin xyz="0.0 0.0 0.33" rpy="0 0 0"/>
+        </xacro:sensor_hokuyo_ust10lx-->
         <!-- 3d laser -->
-        <xacro:sensor_rslidar_16 prefix="$(arg prefix)top_3d_laser" parent="$(arg prefix)base_link">
-            <origin xyz="-0.2776 0 0.629" rpy="0 0 0"/>
-        </xacro:sensor_rslidar_16>
+        <!--xacro:sensor_rslidar_mems prefix="$(arg prefix)top_3d_laser" parent="$(arg prefix)base_link">
+            <origin xyz="0.3134 0 0.2424" rpy="0 0 0"/>
+        </xacro:sensor_rslidar_mems-->
         <!-- ptz camera -->
         <!--xacro:sensor_axis prefix="$(arg prefix)front_ptz_camera" parent="$(arg prefix)base_link">
@@ -115,11 +82,11 @@
         </xacro:sensor_axis-->
         <!-- RGBD -->
-        <xacro:sensor_orbbec_astra prefix="$(arg prefix)front_rgbd_camera" parent="$(arg prefix)base_link" prefix_topic="front_rgbd_camera">
+        <!--xacro:sensor_orbbec_astra prefix="$(arg prefix)front_rgbd_camera" parent="$(arg prefix)base_link" prefix_topic="front_rgbd_camera">
                 <origin xyz="0.324 0.012 0.172" rpy="0 0 0"/>
-            </xacro:sensor_orbbec_astra>
+            </xacro:sensor_orbbec_astra-->
         <!-- GPS -->
-        <xacro:sensor_gps prefix="$(arg prefix)gps" parent="$(arg prefix)base_link">
-            <origin xyz="-0.2776 0 0.732" rpy="0 0 0"/>
-        </xacro:sensor_gps>
+        <!--xacro:sensor_gps prefix="$(arg prefix)gps" parent="$(arg prefix)base_link">
+            <origin xyz="-0.28 0 0.6676" rpy="0 0 0"/>
+        </xacro:sensor_gps-->
         <!-- Instance jaco arm -->
         <joint name="$(arg prefix)arm_base_joint" type="fixed">
@@ -130,5 +97,5 @@
         </joint>
         <link name="$(arg prefix)arm_base_link" />
-        <xacro:j2s6s300 base_parent="$(arg prefix)arm_base_link" prefix="$(arg prefix)j2s6s300"/>
+        <xacro:j2s7s300 base_parent="$(arg prefix)arm_base_link" prefix="$(arg prefix)j2s7s300"/>
     </xacro:macro>
     <!-- Gazebo ros control pluggins -->
