Commit message: corrected bug in joint name

File: summit_xl_description/urdf/wheels/omni_wheel.urdf.xacro (robot description, xacro)
@@ -71,5 +71,5 @@
     <transmission name="${name}_wheel_joint_trans">
       <type>transmission_interface/SimpleTransmission</type>
-      <joint name="joint_${name}_wheel" >
+      <joint name="${name}_wheel_joint" >
         <hardwareInterface>VelocityJointInterface</hardwareInterface>
       </joint>

Commit message: description: Update wheels properties
- rename radius,height and mass properties for each wheel to avoid conflicts
- Omni wheel uses again Sphere for collision model

File: summit_xl_description/urdf/wheels/omni_wheel.urdf.xacro (robot description, xacro)
@@ -3,7 +3,7 @@
   <xacro:property name="M_PI" value="3.1415926535897931" />
   <!-- Wheels -->
-  <xacro:property name="wheel_radius" value="0.127" />
-  <xacro:property name="wheel_height" value="0.087" />
-  <xacro:property name="wheel_mass" value="6.5" /> <!-- in kg-->
+  <xacro:property name="omni_wheel_radius" value="0.127" />
+  <xacro:property name="omni_wheel_height" value="0.087" />
+  <xacro:property name="omni_wheel_mass" value="6.5" /> <!-- in kg-->
   <xacro:macro name="cylinder_inertia" params="m r h">
     <inertia  ixx="${m*(3*r*r+h*h)/12}" ixy = "0" ixz = "0"
@@ -38,5 +38,5 @@
           <origin xyz="0 0 0" rpy="0 0 0" />
           <geometry>
-            <sphere radius="${wheel_radius}" />
+            <sphere radius="${omni_wheel_radius}" />
           </geometry>
         </xacro:unless>
@@ -48,7 +48,5 @@
 				<origin xyz="0 0 0" rpy="${PI/2} 0 0" />
         <geometry>
-<!--
-          <sphere radius="${wheel_radius}" />
--->
+          <sphere radius="${omni_wheel_radius}" />
 <!--
           <xacro:if value="${reflect}">
@@ -59,11 +57,11 @@
 					</xacro:unless>
 -->
-					<cylinder length="${wheel_height}" radius="${wheel_radius}" />
+					<!--cylinder length="${omni_wheel_height}" radius="${omni_wheel_radius}" /-->
         </geometry>
       </collision>
       <inertial>
-        <mass value="${wheel_mass}" />
+        <mass value="${omni_wheel_mass}" />
         <origin xyz="0 0 0" />
-        <cylinder_inertia  m="${wheel_mass}" r="${wheel_radius}" h="${wheel_height}" />
+        <cylinder_inertia  m="${omni_wheel_mass}" r="${omni_wheel_radius}" h="${omni_wheel_height}" />
       </inertial>
     </link>

File: summit_xl_description/urdf/wheels/rubber_wheel.urdf.xacro (robot description, xacro)
@@ -3,7 +3,7 @@
   <xacro:property name="M_PI" value="3.1415926535897931" />
   <!-- Wheels -->
-  <xacro:property name="wheel_radius" value="0.125" />
-  <xacro:property name="wheel_height" value="0.14" /> <!-- really is the wheel width -->
-  <xacro:property name="wheel_mass" value="6.5" /> <!-- in kg-->
+  <xacro:property name="rubber_wheel_radius" value="0.11" />
+  <xacro:property name="rubber_wheel_height" value="0.15" /> <!-- really is the wheel width -->
+  <xacro:property name="rubber_wheel_mass" value="6.5" /> <!-- in kg-->
   <xacro:macro name="cylinder_inertia" params="m r h">
     <inertia  ixx="${m*(3*r*r+h*h)/12}" ixy = "0" ixz = "0"
@@ -39,5 +39,5 @@
           <origin xyz="0 0 0" rpy="${M_PI/2} 0 0" />
           <geometry>
-            <cylinder length="${wheel_height}" radius="${wheel_radius}" />
+            <cylinder length="${rubber_wheel_height}" radius="${rubber_wheel_radius}" />
           </geometry>
         </xacro:unless>
@@ -46,11 +46,11 @@
 				<origin xyz="0 0 0" rpy="${M_PI/2} 0 0" />
         <geometry>
-          <cylinder length="${wheel_height}" radius="${wheel_radius}" />
+          <cylinder length="${rubber_wheel_height}" radius="${rubber_wheel_radius}" />
         </geometry>
       </collision>
       <inertial>
-        <mass value="${wheel_mass}" />
+        <mass value="${rubber_wheel_mass}" />
         <origin xyz="0 0 0" />
-        <cylinder_inertia  m="${wheel_mass}" r="${wheel_radius}" h="${wheel_height}" />
+        <cylinder_inertia  m="${rubber_wheel_mass}" r="${rubber_wheel_radius}" h="${rubber_wheel_height}" />
       </inertial>
     </link>
