Commit message: description:Use the rubber wheel model for collision to improve adherence

File: summit_xl_description/urdf/wheels/rubber_wheel.urdf.xacro (robot description, xacro)
@@ -44,7 +44,9 @@
       </visual>
       <collision>
-				<origin xyz="0 0 0" rpy="${M_PI/2} 0 0" />
+				<!--origin xyz="0 0 0" rpy="${M_PI/2} 0 0" /-->
+        <origin xyz="0 0 0" rpy="0 0 0" />
         <geometry>
-          <cylinder length="${rubber_wheel_height}" radius="${rubber_wheel_radius}" />
+          <!--cylinder length="${rubber_wheel_height}" radius="${rubber_wheel_radius}" /-->
+          <mesh filename="package://summit_xl_description/meshes/wheels/rubber_wheel_right.dae" />
         </geometry>
       </collision>
@@ -66,5 +68,5 @@
       </actuator>
      </transmission>
-    <gazebo reference="${prefix}_wheel">
+    <!--gazebo reference="${prefix}_wheel">
 			<mu1 value="1.0"/>
 			<mu2 value="1.0"/>
@@ -73,5 +75,5 @@
 			<fdir1 value="1 0 0"/>
       <turnGravityOff>false</turnGravityOff>
-    </gazebo>
+    </gazebo-->
   </xacro:macro>
 </robot>
